File: cad/kicad/PWR-SELECT/PowerSelector.kicad_sch (KiCad schematic)
At the start: 104 parts, among them J101 PANEL_24V_HARNESS, J202 LEMO_EGG.0B.302.CLL_13V_TO_16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, J203 GOLD_MOUNT_10V_TO_16V8, J204 PANEL_POWER_SWITCH_HARNESS, J301 RAW_OUT_TO_LM5176, J401 STATUS_TO_CARRIER_3V3_PULLUPS, J402 POWER_TELEMETRY_TO_CARRIER, Q101 PSMN4R2-80YSE, Q102 PSMN4R2-80YSE, Q201 PSMN4R2-80YSE, Q202 PSMN4R2-80YSE, Q501 SiR5607DP-T1-RE3, Q502 SiR5607DP-T1-RE3, Q503 SiR5607DP-T1-RE3, Q504 SiR5607DP-T1-RE3, U101 LTC4421IUHE#PBF, U201 LTC4418IUF#PBF, U301 TPS3842A015DRLRQ1, U601 INA228AIDGSR, U602 INA228AIDGSR, U603 INA228AIDGSR

Commit message: Lock compact QRC-GOLD battery bracket
Other:
- note added: "J203 QRC-GOLD 8375-0094 DOCK 10.0-16.8 V"
- note removed: "J203 QR-GOLD DOCK 10.0-16.8 V"
Changed lines of the file:
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@@
 		)
 	)
-	(text "J203  QR-GOLD DOCK 10.0-16.8 V"
+	(text "J203  QRC-GOLD 8375-0094 DOCK 10.0-16.8 V"
 		(exclude_from_sim no)
 		(at 28 349 0.0000)

Commit message: Clarify panel-mounted battery dock interface
Other:
- note added: "J203 FROM PANEL QRC-GOLD 8375-0094 HARNESS 10.0-16.8 V"
- note removed: "J203 QRC-GOLD 8375-0094 DOCK 10.0-16.8 V"
Changed lines of the file:
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@@
 		)
 	)
-	(text "J203  QRC-GOLD 8375-0094 DOCK 10.0-16.8 V"
+	(text "J203  FROM PANEL QRC-GOLD 8375-0094 HARNESS 10.0-16.8 V"
 		(exclude_from_sim no)
 		(at 28 349 0.0000)

Commit message: Define bottom PSU harness interfaces
Parts:
- J101: value PANEL_24V_HARNESS -> PSU_24V_HARNESS; footprint Connector_Molex:Molex_Micro-Fit_3.0_43045-0412_2x02_P3.00mm_Vertical -> Connector_Molex:Molex_Mega-Fit_76825-0002_2x01_P5.70mm_Horizontal; symbol Connector_Generic:Conn_02x02_Odd_Even -> Connector_Generic:Conn_01x02; MPN 43045-0412 -> 76825-0002
Connections:
- net GND: now also J101.2 (Pin_2); no longer J101.3 (Pin_3), J101.4 (Pin_4)
- net V24_IN: no longer J101.2 (Pin_2)
Other:
- note added: "H01: RPS-400 CN3 +V to J101-1; CN2 -V to J101-2; 14 AWG."
- note added: "J101 BOTTOM-PSU 24 V HARNESS"
- note added: "Priority: internal PSU 24 V, then D-Tap, then Gold Mount. No source paralleling."
- note removed: "J101 REAR 24 V INLET HARNESS"
- note removed: "Priority: rear 24 V, then D-Tap, then Gold Mount. No source paralleling."
- note removed: "Rear KPJX-4S-S inlet: R7B pins 1/4 = +24 V; pins 2/3 = return."
Changed lines of the file:
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@@
 	(title_block
 		(title "Radxa CM5 ProComm 24 V / Battery Seamless Power Selector")
-		(date "2026-08-15")
+		(date "2026-08-16")
 		(rev "A1")
 		(company "ProComm")
-		(comment 1 "Fixed priority: rear 24 V, then D-Tap, then Gold Mount dock")
+		(comment 1 "Fixed priority: internal PSU 24 V, then D-Tap, then Gold Mount dock")
 		(comment 2 "RAW_OUT_LOAD feeds the protected CM5-CARRIER regulator input")
 		(comment 3 "Battery inputs use LTC4418 plus back-to-back P-MOS reverse-polarity blocking")
@@
 	)
 	(symbol
-		(lib_id "Connector_Generic:Conn_02x02_Odd_Even")
+		(lib_id "Connector_Generic:Conn_01x02")
 		(at 27.94 43.18 0)
 		(unit 1)
@@
 		(fields_autoplaced no)
 		(property "Reference" "J101"
-			(at 29.21 45.72 0.0000)
+			(at 27.94 45.72 0.0000)
 			(effects
 				(font
@@
 			)
 		)
-		(property "Value" "PANEL_24V_HARNESS"
-			(at 29.21 38.1 0.0000)
+		(property "Value" "PSU_24V_HARNESS"
+			(at 27.94 38.1 0.0000)
 			(effects
 				(font
@@
 			)
 		)
-		(property "Footprint" "Connector_Molex:Molex_Micro-Fit_3.0_43045-0412_2x02_P3.00mm_Vertical"
+		(property "Footprint" "Connector_Molex:Molex_Mega-Fit_76825-0002_2x01_P5.70mm_Horizontal"
 			(at 27.94 43.18 0.0000)
 			(effects
@@
 			)
 		)
-		(property "MPN" "43045-0412"
+		(property "MPN" "76825-0002"
 			(at 30.48 48.2599 0)
 			(effects
@@
 			)
 		)
+		(property "Datasheet" "https://www.molex.com/en-us/products/part-detail/768250002"
+			(at 27.94 43.18 0)
+			(effects
+				(font
+					(size 1.27 1.27)
+				)
+				(hide yes)
+			)
+		)
 		(pin "1"
 		)
 		(pin "2"
 		)
-		(pin "3"
-		)
-		(pin "4"
-		)
 		(instances
 			(project "PowerSelector"
@@
 		)
 	)
-	(label "V24_IN"
-		(at 35.56 43.18 0)
-		(effects
-			(font
-				(size 1 1)
-			)
-			(justify left bottom)
-		)
-	)
 	(label "GND"
 		(at 22.86 45.72 0)
@@
 		)
 	)
-	(label "GND"
-		(at 35.56 45.72 0)
-		(effects
-			(font
-				(size 1 1)
-			)
-			(justify left bottom)
-		)
-	)
 	(label "V24_IN"
 		(at 48.26 43.18 0)
@@
 		)
 	)
-	(text "Rear KPJX-4S-S inlet: R7B pins 1/4 = +24 V; pins 2/3 = return."
+	(text "H01: RPS-400 CN3 +V to J101-1; CN2 -V to J101-2; 14 AWG."
 		(exclude_from_sim no)
 		(at 80 26 0.0000)
@@
 		)
 	)
-	(text "J101  REAR 24 V INLET HARNESS"
+	(text "J101  BOTTOM-PSU 24 V HARNESS"
 		(exclude_from_sim no)
 		(at 28 34 0.0000)
@@
 		)
 	)
-	(text "Priority: rear 24 V, then D-Tap, then Gold Mount. No source paralleling."
+	(text "Priority: internal PSU 24 V, then D-Tap, then Gold Mount. No source paralleling."
 		(exclude_from_sim no)
 		(at 330 392 0.0000)

Commit message: Complete A1 detailed carrier and audio capture
Parts:
- removed C532: 1nF C0G, Capacitor_SMD:C_0603_1608Metric, symbol Device:C
- removed R101: 18.2k 0.1%, Resistor_SMD:R_0603_1608Metric, symbol Device:R
- removed R102: 9.10k 0.1%, Resistor_SMD:R_0603_1608Metric, symbol Device:R
- removed R103: 3.01k 0.1%, Resistor_SMD:R_0603_1608Metric, symbol Device:R
- removed R104: 1.06M 0.1%, Resistor_SMD:R_0603_1608Metric, symbol Device:R
- removed R301: 176k 0.1%, Resistor_SMD:R_0603_1608Metric, symbol Device:R
- removed R502: 26.1k 0.1%, Resistor_SMD:R_0603_1608Metric, symbol Device:R
- removed R503: 919k 0.1%, Resistor_SMD:R_0603_1608Metric, symbol Device:R
- added C307, C308, C309: 6800uF 50V, Capacitor_THT:CP_Radial_D30.0mm_P10.00mm_SnapIn, symbol Device:C_Polarized
- added J401: STATUS_TO_CARRIER_3V3_PULLUPS, Connector_Molex:Molex_PicoBlade_53047-0810_1x08_P1.25mm_Vertical, symbol Connector_Generic:Conn_01x08
- added R201: 28.0k 0.1%, Resistor_SMD:R_0603_1608Metric, symbol Device:R
- added R202: 15.8k 0.1%, Resistor_SMD:R_0603_1608Metric, symbol Device:R
- added R203: 4.22k 0.1%, Resistor_SMD:R_0603_1608Metric, symbol Device:R
- added R204: 965k 0.1%, Resistor_SMD:R_0603_1608Metric, symbol Device:R
- added R311: 1.00mR 1% 1W, Resistor_SMD:R_Shunt_Vishay_WSK2512_6332Metric_T2.21mm, symbol Device:R_Shunt
- added R501: 55.6k 0.1%, Resistor_SMD:R_0603_1608Metric, symbol Device:R
- added R504: 56.2k 0.1%, Resistor_SMD:R_0603_1608Metric, symbol Device:R
- added R505: 31.6k 0.1%, Resistor_SMD:R_0603_1608Metric, symbol Device:R
- C306: renamed from R311; value 1.00mR 1% 1W -> 6800uF 50V; footprint Resistor_SMD:R_Shunt_Vishay_WSK2512_6332Metric_T2.21mm -> Capacitor_THT:CP_Radial_D30.0mm_P10.00mm_SnapIn; symbol Device:R_Shunt -> Device:C_Polarized; MPN WSK25121L000FEA -> LGU1H682MELB; Manufacturer Vishay -> Nichicon; Mechanical (none) -> 30 mm diameter x 35 mm; retain with tray-supported clamp
- C532: renamed from R501; value 55.6k 0.1% -> 1nF C0G; footprint Resistor_SMD:R_0603_1608Metric -> Capacitor_SMD:C_0603_1608Metric; symbol Device:R -> Device:C
- R101: renamed from R201; value 28.0k 0.1% -> 18.2k 0.1%
- R102: renamed from R202; value 15.8k 0.1% -> 9.10k 0.1%
- R103: renamed from R203; value 4.22k 0.1% -> 3.01k 0.1%
- R104: renamed from R204; value 965k 0.1% -> 1.06M 0.1%
- R301: renamed from J401; value STATUS_TO_CARRIER_3V3_PULLUPS -> 176k 0.1%; footprint Connector_Molex:Molex_PicoBlade_53047-0810_1x08_P1.25mm_Vertical -> Resistor_SMD:R_0603_1608Metric; symbol Connector_Generic:Conn_01x08 -> Device:R; MPN 53047-0810 -> (none); Manufacturer Molex -> (none)
- R502: renamed from R504; value 56.2k 0.1% -> 26.1k 0.1%
- R503: renamed from R505; value 31.6k 0.1% -> 919k 0.1%
Connections:
- net BAT_FUSED: now also R301.1, R204.1; no longer R104.1
- net BAT_LOW_N: now also J401.6 (Pin_6); no longer R301.6 (Pin_6)
- net BAT_MON: now also R301.2
- net CH_24V_N: now also J401.2 (Pin_2); no longer R301.2 (Pin_2)
- net CH_BAT_N: now also J401.3 (Pin_3); no longer R301.3 (Pin_3)
- net DTAP_FUSED: now also R503.1
- net GND: now also C306.2, C307.2, C308.2, C309.2, J401.1 (Pin_1), R201.2, R501.2, R504.2; no longer R301.1 (Pin_1), R502.2
- net OV_24: now also R101.1, R102.2
- net OV_BAT: now also R201.1, R202.2; no longer R101.1, R102.2
- net OV_DTAP: now also R502.2, R501.1; no longer C532.1
- net OV_GOLD: now also R504.1, R505.2; no longer R502.1, R503.2
- net RAW_OUT: now also C307.1, C308.1, C309.1, R311.1, R311.2; no longer C306.2
- net RAW_OUT_LOAD: now also R311.3, R311.4; no longer C306.3, C306.4
- net TMR_PRE: now also C532.1
- net UVF_24: now also R103.1, R104.2
- net UVF_BAT: now also R203.1, R204.2; no longer R103.1, R104.2
- net UVR_24: now also R102.1, R103.2
- net UVR_BAT: now also R202.1, R203.2; no longer R102.1, R103.2
- net UV_DTAP: now also R502.1, R503.2
- net UV_GOLD: now also R505.1; no longer R503.1
- net V24_FUSED: now also R104.1
- net VALID_24V_N: now also J401.4 (Pin_4); no longer R301.4 (Pin_4)
- net VALID_BAT_N: now also J401.5 (Pin_5); no longer R301.5 (Pin_5)
- net VALID_DTAP_N: now also J401.7 (Pin_7); no longer R301.7 (Pin_7)
- net VALID_GOLD_N: now also J401.8 (Pin_8); no longer R301.8 (Pin_8)
Other:
- note added: "30 x 35 mm cans require a tray-supported clamp; board outline and dock clearance remain A2 sample gates."
- note added: "At -20% capacitance the total provides about 25.4 ms ideal hold-up at 184.2 W from 24.0 V to 12.5 V."
- note added: "Both selectors are break-before-make; C301-C309 provide continuous energy to the carrier input."
- note added: "C306"
- note added: "C306-C309: 4 x 6800 uF = 27.2 mF; total with C301-C303 is 27.86 mF nominal."
- note added: "C307"
- note added: "C308"
- note added: "C309"
- note removed: "660 uF nominal (528 uF at -20%): approximately 0.33 V worst-case transfer droop at 10 A / 15 us."
- note removed: "Both selectors are break-before-make; C301-C303 provide continuous energy to the LM5176 input."
- note removed: "RAW_OUT remains within the downstream LM5176 input range during 24 V to battery transfer."

Commit message: Lock CM5 power and radio interfaces before routing
Parts:
- added R106: 107k 0.1%, Resistor_SMD:R_0603_1608Metric, symbol Device:R
- added R206: 12.1k 0.1%, Resistor_SMD:R_0603_1608Metric, symbol Device:R
- added R507: 10.0k 0.1%, Resistor_SMD:R_0603_1608Metric, symbol Device:R
- C101, C201, C304: MPN (none) -> GRM32RR71H105KA01L; Manufacturer (none) -> Murata
- C105, C202, C203, C205: MPN (none) -> GRM32ER71H106KA12L; Manufacturer (none) -> Murata
- C110, C210, C511, C521: MPN (none) -> GRM188R71H473KA61D; Manufacturer (none) -> Murata
- C120, C121: MPN (none) -> GRM188R71E105KA12D; Manufacturer (none) -> Murata
- C122, C311, C532: MPN (none) -> GRM1885C1H102JA01D; Manufacturer (none) -> Murata
- C123, C223, C310, C531, C601, C603, C611, C613, C621, C623: MPN (none) -> GRM188R71E104KA01D; Manufacturer (none) -> Murata
- C305: MPN (none) -> GRM188R71H104KA93D; Manufacturer (none) -> Murata
- C512, C522: MPN (none) -> GRM188R71H474KA12D; Manufacturer (none) -> Murata
- C533: value 100uF 35V -> 100uF 63V; MPN (none) -> EEEFK1J101L; Manufacturer (none) -> Panasonic
- C602, C612, C622: MPN (none) -> GRM188R72A103KA01D; Manufacturer (none) -> Murata
- C630: MPN (none) -> GRM188R71A105KA61D; Manufacturer (none) -> Murata
- R101: MPN (none) -> ERA3AEB1822V; Manufacturer (none) -> Panasonic
- R102: MPN (none) -> ERA3AEB9101V; Manufacturer (none) -> Panasonic
- R103: MPN (none) -> ERA3AEB3011V; Manufacturer (none) -> Panasonic
- R104: value 1.06M 0.1% -> 953k 0.1%; MPN (none) -> ERA3AEB9533V; Manufacturer (none) -> Panasonic
- R105: MPN (none) -> RC0603FR-072R4L; Manufacturer (none) -> Yageo
- R131, R231: MPN (none) -> RC0603FR-07100KL; Manufacturer (none) -> Yageo
- R201: MPN (none) -> ERA3AEB2802V; Manufacturer (none) -> Panasonic
- R202: MPN (none) -> ERA3AEB1582V; Manufacturer (none) -> Panasonic
- R203: MPN (none) -> ERA3AEB4221V; Manufacturer (none) -> Panasonic
- R204: value 965k 0.1% -> 953k 0.1%; MPN (none) -> ERA3AEB9533V; Manufacturer (none) -> Panasonic
- R205: MPN (none) -> RC0603FR-071R69L; Manufacturer (none) -> Yageo
- R301: MPN (none) -> ERA3AEB1763V; Manufacturer (none) -> Panasonic
- R302: MPN (none) -> ERA3AEB1002V; Manufacturer (none) -> Panasonic
- R501: MPN (none) -> ERA3AEB5562V; Manufacturer (none) -> Panasonic
- R502: MPN (none) -> ERA3AEB2612V; Manufacturer (none) -> Panasonic
- R503: value 919k 0.1% -> 909k 0.1%; MPN (none) -> ERA3AEB9093V; Manufacturer (none) -> Panasonic
- R504: MPN (none) -> ERA3AEB5622V; Manufacturer (none) -> Panasonic
- R505: MPN (none) -> ERA3AEB3162V; Manufacturer (none) -> Panasonic
- R506: MPN (none) -> ERA3AEB9093V; Manufacturer (none) -> Panasonic
- R511, R521: MPN (none) -> RC0603FR-076K81L; Manufacturer (none) -> Yageo
- R541, R542: MPN (none) -> RC0603FR-0747KL; Manufacturer (none) -> Yageo
- R601, R602, R611, R612, R621, R622: MPN (none) -> RC0603FR-0710RL; Manufacturer (none) -> Yageo
- R603, R613, R623: MPN (none) -> RC0603FR-07100RL; Manufacturer (none) -> Yageo
Connections:
- net UVF_24: now also R106.2; no longer R104.2
- net UVF_BAT: now also R206.2; no longer R204.2
- net UV_DTAP: now also R507.2; no longer R503.2
- new net BAT_RTOP_MID: R204.2, R206.1
- new net DTAP_RTOP_MID: R503.2, R507.1
- new net V24_RTOP_MID: R104.2, R106.1
Other:
- note added: "R104 953k 0.1%"
- note added: "R106 107k 0.1%"
- note added: "R204 953k 0.1%"
- note added: "R206 12.1k 0.1%"
- note added: "R503 909k 0.1%"
- note added: "R507 10.0k 0.1%"
- note removed: "R104 1.06M 0.1%"
- note removed: "R204 965k 0.1%"
- note removed: "R503 919k 0.1%"
