File: cad/kicad/PWR-SELECT/PowerSelector.kicad_pcb (KiCad board)
At the start: 6 copper layers, 116 x 80 mm, 111 parts, among them J101 PSU_24V_HARNESS, J202 LEMO_EGG.0B.302.CLL_13V_TO_16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, J203 GOLD_MOUNT_10V_TO_16V8, J204 PANEL_POWER_SWITCH_HARNESS, J301 RAW_OUT_TO_LM5176, J401 STATUS_TO_CARRIER_3V3_PULLUPS, J402 POWER_TELEMETRY_TO_CARRIER, Q101 PSMN4R2-80YSE, Q102 PSMN4R2-80YSE, Q201 PSMN4R2-80YSE, Q202 PSMN4R2-80YSE, Q501 SiR5607DP-T1-RE3, Q502 SiR5607DP-T1-RE3, Q503 SiR5607DP-T1-RE3, Q504 SiR5607DP-T1-RE3, U101 LTC4421IUHE#PBF, U201 LTC4418IUF#PBF, U301 TPS3842A015DRLRQ1, U601 INA228AIDGSR, U602 INA228AIDGSR, U603 INA228AIDGSR

Commit message: Fix PCB-A1 in-board 3D placement
Parts:
- C101, C105, C110, C120, C121, C122, C123, C201, C202, C203, C205, C210, C223, C304, C305, C310, C311, C511, C512, C521, C522, C531, C532, C601, C602, C603, C611, C612, C613, C621, C622, C623, C630, D101, D201, D202, D203, D511, D521, F101, F201, F202, F203, Q101, Q102, Q201, Q202, Q501, Q502, Q503, Q504, R101, R102, R103, R104, R105, R106, R111, R131, R201, R202, R203, R204, R205, R206, R211, R231, R301, R302, R311, R501, R502, R503, R504, R505, R506, R507, R511, R521, R541, R542, R601, R602, R603, R611, R612, R613, R621, R622, R623, U301, U601, U602, U603: moved to B.Cu
- moved R501 404.8 mm to (15.5, 22.8)
- moved C309 400.6 mm to (12.3, 49.3)
- moved R311 385.0 mm to (28.4, 10.9)
- moved R503 363.7 mm to (70.8, 24.5), turned to 90 degrees
- moved R502 360.5 mm to (67.0, 23.8)
- moved R206 343.2 mm to (26.0, 22.3)
- moved C310 339.2 mm to (97.8, 17.5), turned to 90 degrees
- moved R301 332.7 mm to (62.5, 22.3)
- moved R201 330.9 mm to (3.52, 21.8)
- moved R231 330.2 mm to (58.0, 22.3)
- moved J204 318.0 mm to (106.1, 43.0)
- moved J203 316.3 mm to (93.6, 43.0)
- moved J202 314.6 mm to (81.1, 37.0)
- moved R203 312.7 mm to (36.0, 21.8)
- moved R202 310.2 mm to (31.5, 21.8)
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Other:
- board text added: "F.Cu POWER HARDWARE / B.Cu CONTROL; MOUNT DATUM PENDING"
- board text added: "PWR-SELECT PCB-A1"
- board text removed: "BOTTOM-TRAY MOUNT HOLES NOT RELEASED - NONE GUESSED"
- board text removed: "PWR-SELECT PCB-A0"
- board text removed: "UNPLACED / UNVERIFIED PCB FOOTPRINT STAGING - NOT BOARD GEOMETRY"
