File: cad/kicad/AUDIO-8X8/AK4458-DAC.kicad_sch (KiCad schematic)
At the start: 23 parts, among them U301 AK4458VN

Commit message: Audit schematic logic against controlled datasheets
Parts:
- C361, C362, C363, C364: value 100uF 6.3V polymer -> 220uF 6.3V polymer; footprint Capacitor_SMD:CP_Elec_6.3x5.8 -> Capacitor_SMD:CP_Elec_8x6.9; MPN 6SVP100M -> 6SVP220MX
- C373, C375: value 4.7uF -> 10uF; footprint Capacitor_SMD:C_0805_2012Metric -> Capacitor_SMD:C_0603_1608Metric; MPN GRM21BR71A475KA73L -> GRM188R71A106KA73D
- R351, R352, R353, R354: value 20R -> 10R; MPN RC0603FR-0720RL -> RC0603FR-0710RL
Connections:
- net AUD_DAC_MUTE_N renamed AUDIO_SAFE_UNMUTE_N
Other:
- note added: "Each VREFH branch uses the AK4458 optional 10 ohm / 220 uF low-impedance filter. Place AVDD, TVDD, and VDD18 bypass parts at their pins."
- note removed: "Place each 100 nF at its corresponding supply/reference pin pair; VDD18 1 uF must have the shortest return to DVSS/EP."

Commit message: Implement direct socketed dual-SIM daughterboard
Parts:
- removed C371: 1uF, Capacitor_SMD:C_0603_1608Metric, symbol Device:C
- removed C372: 100nF, Capacitor_SMD:C_0402_1005Metric, symbol Device:C
- removed R321, R322: 10k 0.1%, Resistor_SMD:R_0603_1608Metric, symbol Device:R
- added C351, C374: 100nF, Capacitor_SMD:C_0402_1005Metric, symbol Device:C
- added C375: 10uF, Capacitor_SMD:C_0603_1608Metric, symbol Device:C
- added R351: 10R, Resistor_SMD:R_0603_1608Metric, symbol Device:R
- C371: renamed from C374; value 100nF -> 1uF; footprint Capacitor_SMD:C_0402_1005Metric -> Capacitor_SMD:C_0603_1608Metric; MPN C1005X7R1H104K050BB -> GRM188R71A105KA61D; Manufacturer TDK -> Murata
- C372: renamed from C375; value 10uF -> 100nF; footprint Capacitor_SMD:C_0603_1608Metric -> Capacitor_SMD:C_0402_1005Metric; MPN GRM188R71A106KA73D -> C1005X7R1H104K050BB; Manufacturer Murata -> TDK
- R331: renamed from R351; value 10R -> 10k 0.1%; MPN RC0603FR-0710RL -> RC0603FR-0710KL
- R332: renamed from C351; value 100nF -> 10k 0.1%; footprint Capacitor_SMD:C_0402_1005Metric -> Resistor_SMD:R_0603_1608Metric; symbol Device:C -> Device:R; MPN C1005X7R1H104K050BB -> RC0603FR-0710KL; Manufacturer TDK -> Yageo
- renumbered R331 to R321, R332 to R322
Connections:
- net AGND: now also R331.2, C351.2, C374.2, C375.2; no longer R321.2, R322.2
- net AKM_3V3_D: now also R321.1, R322.1, C374.1, C375.1; no longer C371.1, C372.1
- net DAC_5V_A: now also C372.1, R351.1; no longer R331.1
- net DAC_CAD1: now also R331.1; no longer R321.1
- net DAC_I2C_MODE: now also R321.2
- net DAC_LDOE: now also R322.2
- net DAC_PS: now also R332.1; no longer R322.1
- net DAC_VDD18: now also C371.1
- net DAC_VREFH1: now also C351.1, R351.2; no longer R331.2, R332.1
Other:
- moved on the sheet: C371, C372, R321, R322, R331
Changed lines of the file:
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@@
 		(instances
 			(project "AK4458-DAC"
-				(path "/0b2d4537-d5e9-5bc3-991f-7ffe1832510b"
+				(path "/5177fae7-57f8-5346-9fdd-c38c950c7bf0"
 					(reference "U301")
 					(unit 1)
@@
 		(instances
 			(project "AK4458-DAC"
-				(path "/0b2d4537-d5e9-5bc3-991f-7ffe1832510b"
+				(path "/5177fae7-57f8-5346-9fdd-c38c950c7bf0"
 					(reference "R321")
 					(unit 1)
@@
 		(instances
 			(project "AK4458-DAC"
-				(path "/0b2d4537-d5e9-5bc3-991f-7ffe1832510b"
+				(path "/5177fae7-57f8-5346-9fdd-c38c950c7bf0"
 					(reference "R322")
 					(unit 1)
@@
 		(instances
 			(project "AK4458-DAC"
-				(path "/0b2d4537-d5e9-5bc3-991f-7ffe1832510b"
+				(path "/5177fae7-57f8-5346-9fdd-c38c950c7bf0"
 					(reference "R323")
 					(unit 1)
@@
 		(instances
 			(project "AK4458-DAC"
-				(path "/0b2d4537-d5e9-5bc3-991f-7ffe1832510b"
+				(path "/5177fae7-57f8-5346-9fdd-c38c950c7bf0"
 					(reference "R331")
 					(unit 1)
@@
 		(instances
 			(project "AK4458-DAC"
-				(path "/0b2d4537-d5e9-5bc3-991f-7ffe1832510b"
+				(path "/5177fae7-57f8-5346-9fdd-c38c950c7bf0"
 					(reference "R332")
 					(unit 1)
@@
 		(instances
 			(project "AK4458-DAC"
-				(path "/0b2d4537-d5e9-5bc3-991f-7ffe1832510b"
+				(path "/5177fae7-57f8-5346-9fdd-c38c950c7bf0"
 					(reference "R351")
 					(unit 1)
@@
 		(instances
 			(project "AK4458-DAC"
-				(path "/0b2d4537-d5e9-5bc3-991f-7ffe1832510b"
+				(path "/5177fae7-57f8-5346-9fdd-c38c950c7bf0"
 					(reference "C351")
 					(unit 1)
@@
 		(instances
 			(project "AK4458-DAC"
-				(path "/0b2d4537-d5e9-5bc3-991f-7ffe1832510b"
+				(path "/5177fae7-57f8-5346-9fdd-c38c950c7bf0"
 					(reference "C361")
 					(unit 1)
@@
 		(instances
 			(project "AK4458-DAC"
-				(path "/0b2d4537-d5e9-5bc3-991f-7ffe1832510b"
+				(path "/5177fae7-57f8-5346-9fdd-c38c950c7bf0"
 					(reference "R352")
 					(unit 1)
@@
 		(instances
 			(project "AK4458-DAC"
-				(path "/0b2d4537-d5e9-5bc3-991f-7ffe1832510b"
+				(path "/5177fae7-57f8-5346-9fdd-c38c950c7bf0"
 					(reference "C352")
 					(unit 1)
@@
 		(instances
 			(project "AK4458-DAC"
-				(path "/0b2d4537-d5e9-5bc3-991f-7ffe1832510b"
+				(path "/5177fae7-57f8-5346-9fdd-c38c950c7bf0"
 					(reference "C362")
 					(unit 1)
@@
 		(instances
 			(project "AK4458-DAC"
-				(path "/0b2d4537-d5e9-5bc3-991f-7ffe1832510b"
+				(path "/5177fae7-57f8-5346-9fdd-c38c950c7bf0"
 					(reference "R353")
 					(unit 1)
@@
 		(instances
 			(project "AK4458-DAC"
-				(path "/0b2d4537-d5e9-5bc3-991f-7ffe1832510b"
+				(path "/5177fae7-57f8-5346-9fdd-c38c950c7bf0"
 					(reference "C353")
 					(unit 1)
@@
 		(instances
 			(project "AK4458-DAC"
-				(path "/0b2d4537-d5e9-5bc3-991f-7ffe1832510b"
+				(path "/5177fae7-57f8-5346-9fdd-c38c950c7bf0"
 					(reference "C363")
 					(unit 1)
@@
 		(instances
 			(project "AK4458-DAC"
-				(path "/0b2d4537-d5e9-5bc3-991f-7ffe1832510b"
+				(path "/5177fae7-57f8-5346-9fdd-c38c950c7bf0"
 					(reference "R354")
 					(unit 1)
@@
 		(instances
 			(project "AK4458-DAC"
-				(path "/0b2d4537-d5e9-5bc3-991f-7ffe1832510b"
+				(path "/5177fae7-57f8-5346-9fdd-c38c950c7bf0"
 					(reference "C354")
 					(unit 1)
@@
 		(instances
 			(project "AK4458-DAC"
-				(path "/0b2d4537-d5e9-5bc3-991f-7ffe1832510b"
+				(path "/5177fae7-57f8-5346-9fdd-c38c950c7bf0"
 					(reference "C364")
 					(unit 1)
@@
 		(instances
 			(project "AK4458-DAC"
-				(path "/0b2d4537-d5e9-5bc3-991f-7ffe1832510b"
+				(path "/5177fae7-57f8-5346-9fdd-c38c950c7bf0"
 					(reference "C371")
 					(unit 1)
@@
 		(instances
 			(project "AK4458-DAC"
-				(path "/0b2d4537-d5e9-5bc3-991f-7ffe1832510b"
+				(path "/5177fae7-57f8-5346-9fdd-c38c950c7bf0"
 					(reference "C372")
 					(unit 1)
@@
 		(instances
 			(project "AK4458-DAC"
-				(path "/0b2d4537-d5e9-5bc3-991f-7ffe1832510b"
+				(path "/5177fae7-57f8-5346-9fdd-c38c950c7bf0"
 					(reference "C373")
 					(unit 1)
@@
 		(instances
 			(project "AK4458-DAC"
-				(path "/0b2d4537-d5e9-5bc3-991f-7ffe1832510b"
+				(path "/5177fae7-57f8-5346-9fdd-c38c950c7bf0"
 					(reference "C374")
 					(unit 1)
@@
 		(instances
 			(project "AK4458-DAC"
-				(path "/0b2d4537-d5e9-5bc3-991f-7ffe1832510b"
+				(path "/5177fae7-57f8-5346-9fdd-c38c950c7bf0"
 					(reference "C375")
 					(unit 1)
