File: cad/kicad/AUDIO-8X8/AK5558-ADC.kicad_sch (KiCad schematic)
At the start: 36 parts, among them U201 AK5558VN

Commit message: Audit schematic logic against controlled datasheets
Parts:
- added C286: 100nF, Capacitor_SMD:C_0402_1005Metric, symbol Device:C
- added C287: 10uF, Capacitor_SMD:C_0603_1608Metric, symbol Device:C
- C281: value 1uF -> 4.7uF; footprint Capacitor_SMD:C_0603_1608Metric -> Capacitor_SMD:C_0805_2012Metric; MPN GRM188R71A105KA61D -> GRM21BR71A475KA73L
- C283, C285: value 4.7uF -> 10uF; footprint Capacitor_SMD:C_0805_2012Metric -> Capacitor_SMD:C_0603_1608Metric; MPN GRM21BR71A475KA73L -> GRM188R71A106KA73D
Connections:
- net ADC_5V_A: now also C286.1, C287.1
- net AGND: now also C286.2, C287.2
- net ADC_DSDOL4_NC: no longer names the net of U201.40 (DSDOL4)
- net ADC_DSDOR4_NC: no longer names the net of U201.41 (DSDOR4)
- net ADC_SDTO2_NC: no longer names the net of U201.37 (SDTO2/DSDOR2)
- net ADC_SDTO3_NC: no longer names the net of U201.38 (SDTO3/DSDOL3)
- net ADC_SDTO4_NC: no longer names the net of U201.39 (SDTO4/DSDOR3)
- no-connect marks 0 -> 5
Other:
- note added: "Place C282/C283 at AVDD1, C286/C287 at AVDD2, and C284/C285 at TVDD. C281 is the required 4.7 uF VDD18 stabilizer."
- note removed: "Place each 100 nF at its corresponding supply/reference pin pair; VDD18 1 uF must have the shortest return to DVSS/EP."

Commit message: Implement direct socketed dual-SIM daughterboard
Parts:
- removed C281: 4.7uF, Capacitor_SMD:C_0805_2012Metric, symbol Device:C
- removed C282: 100nF, Capacitor_SMD:C_0402_1005Metric, symbol Device:C
- removed C283: 10uF, Capacitor_SMD:C_0603_1608Metric, symbol Device:C
- removed R221, R222, R223: 10k 0.1%, Resistor_SMD:R_0603_1608Metric, symbol Device:R
- added C285, C287: 10uF, Capacitor_SMD:C_0603_1608Metric, symbol Device:C
- added C286: 100nF, Capacitor_SMD:C_0402_1005Metric, symbol Device:C
- added R248, R249, R250: 10k 0.1%, Resistor_SMD:R_0603_1608Metric, symbol Device:R
- C281: renamed from C284; value 100nF -> 4.7uF; footprint Capacitor_SMD:C_0402_1005Metric -> Capacitor_SMD:C_0805_2012Metric; MPN C1005X7R1H104K050BB -> GRM21BR71A475KA73L; Manufacturer TDK -> Murata
- C282: renamed from C285; value 10uF -> 100nF; footprint Capacitor_SMD:C_0603_1608Metric -> Capacitor_SMD:C_0402_1005Metric; MPN GRM188R71A106KA73D -> C1005X7R1H104K050BB; Manufacturer Murata -> TDK
- C283: renamed from C286; value 100nF -> 10uF; footprint Capacitor_SMD:C_0402_1005Metric -> Capacitor_SMD:C_0603_1608Metric; MPN C1005X7R1H104K050BB -> GRM188R71A106KA73D; Manufacturer TDK -> Murata
- C284: renamed from C287; value 10uF -> 100nF; footprint Capacitor_SMD:C_0603_1608Metric -> Capacitor_SMD:C_0402_1005Metric; MPN GRM188R71A106KA73D -> C1005X7R1H104K050BB; Manufacturer Murata -> TDK
- renumbered R224 to R221, R225 to R222, R226 to R223, R227 to R224, R228 to R225, R241 to R226, R242 to R227, R243 to R228, R244 to R241, R245 to R242, R246 to R243, R247 to R244, R248 to R245, R249 to R246, R250 to R247
Connections:
- net ADC_5V_A: now also C282.1, C286.1, C287.1; no longer C284.1
- net ADC_CAD0: now also R242.1; no longer R227.1
- net ADC_CAD1: now also R243.1; no longer R228.1
- net ADC_DIF0: now also R224.2; no longer R221.2
- net ADC_DIF1: now also R225.2; no longer R222.2
- net ADC_DP: now also R248.1; no longer R245.1
- net ADC_HPFE: now also R249.1; no longer R246.1
- net ADC_I2C_MODE: now also R227.2; no longer R224.2
- net ADC_LDOE: now also R228.2; no longer R225.2
- net ADC_MSN: now also R241.1; no longer R226.1
- net ADC_ODP: now also R250.1; no longer R247.1
- net ADC_PSN: now also R247.1; no longer R244.1
- net ADC_PW0: now also R221.2
- net ADC_PW1: now also R222.2
- net ADC_PW2: now also R223.2
- net ADC_SD_PMOD: now also R245.1; no longer R242.1
- net ADC_SLOW: now also R244.1; no longer R241.1
- net ADC_TDM0: now also R246.1; no longer R243.1
- net ADC_TDM1: now also R226.2; no longer R223.2
- net ADC_VDD18: now also C281.1
- net AGND: now also C285.2, C286.2, C287.2, R248.2, R249.2, R250.2; no longer R226.2, R227.2, R228.2
- net AKM_3V3_D: now also C284.1, R226.1, R227.1, R228.1, C285.1; no longer C281.1, C282.1
Other:
- moved on the sheet: C281, C282, C283, C284, R221, R222, R223, R224, R225, R226, R227, R228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
Changed lines of the file:
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@@
 		(instances
 			(project "AK5558-ADC"
-				(path "/b111be58-5b18-5e09-a452-181893b11c74"
+				(path "/7d8bfbf7-e7f4-539c-a742-574ff9ec8fc2"
 					(reference "U201")
 					(unit 1)
@@
 		(instances
 			(project "AK5558-ADC"
-				(path "/b111be58-5b18-5e09-a452-181893b11c74"
+				(path "/7d8bfbf7-e7f4-539c-a742-574ff9ec8fc2"
 					(reference "R221")
 					(unit 1)
@@
 		(instances
 			(project "AK5558-ADC"
-				(path "/b111be58-5b18-5e09-a452-181893b11c74"
+				(path "/7d8bfbf7-e7f4-539c-a742-574ff9ec8fc2"
 					(reference "R222")
 					(unit 1)
@@
 		(instances
 			(project "AK5558-ADC"
-				(path "/b111be58-5b18-5e09-a452-181893b11c74"
+				(path "/7d8bfbf7-e7f4-539c-a742-574ff9ec8fc2"
 					(reference "R223")
 					(unit 1)
@@
 		(instances
 			(project "AK5558-ADC"
-				(path "/b111be58-5b18-5e09-a452-181893b11c74"
+				(path "/7d8bfbf7-e7f4-539c-a742-574ff9ec8fc2"
 					(reference "R224")
 					(unit 1)
@@
 		(instances
 			(project "AK5558-ADC"
-				(path "/b111be58-5b18-5e09-a452-181893b11c74"
+				(path "/7d8bfbf7-e7f4-539c-a742-574ff9ec8fc2"
 					(reference "R225")
 					(unit 1)
@@
 		(instances
 			(project "AK5558-ADC"
-				(path "/b111be58-5b18-5e09-a452-181893b11c74"
+				(path "/7d8bfbf7-e7f4-539c-a742-574ff9ec8fc2"
 					(reference "R226")
 					(unit 1)
@@
 		(instances
 			(project "AK5558-ADC"
-				(path "/b111be58-5b18-5e09-a452-181893b11c74"
+				(path "/7d8bfbf7-e7f4-539c-a742-574ff9ec8fc2"
 					(reference "R227")
 					(unit 1)
@@
 		(instances
 			(project "AK5558-ADC"
-				(path "/b111be58-5b18-5e09-a452-181893b11c74"
+				(path "/7d8bfbf7-e7f4-539c-a742-574ff9ec8fc2"
 					(reference "R228")
 					(unit 1)
@@
 		(instances
 			(project "AK5558-ADC"
-				(path "/b111be58-5b18-5e09-a452-181893b11c74"
+				(path "/7d8bfbf7-e7f4-539c-a742-574ff9ec8fc2"
 					(reference "R241")
 					(unit 1)
@@
 		(instances
 			(project "AK5558-ADC"
-				(path "/b111be58-5b18-5e09-a452-181893b11c74"
+				(path "/7d8bfbf7-e7f4-539c-a742-574ff9ec8fc2"
 					(reference "R242")
 					(unit 1)
@@
 		(instances
 			(project "AK5558-ADC"
-				(path "/b111be58-5b18-5e09-a452-181893b11c74"
+				(path "/7d8bfbf7-e7f4-539c-a742-574ff9ec8fc2"
 					(reference "R243")
 					(unit 1)
@@
 		(instances
 			(project "AK5558-ADC"
-				(path "/b111be58-5b18-5e09-a452-181893b11c74"
+				(path "/7d8bfbf7-e7f4-539c-a742-574ff9ec8fc2"
 					(reference "R244")
 					(unit 1)
@@
 		(instances
 			(project "AK5558-ADC"
-				(path "/b111be58-5b18-5e09-a452-181893b11c74"
+				(path "/7d8bfbf7-e7f4-539c-a742-574ff9ec8fc2"
 					(reference "R245")
 					(unit 1)
@@
 		(instances
 			(project "AK5558-ADC"
-				(path "/b111be58-5b18-5e09-a452-181893b11c74"
+				(path "/7d8bfbf7-e7f4-539c-a742-574ff9ec8fc2"
 					(reference "R246")
 					(unit 1)
@@
 		(instances
 			(project "AK5558-ADC"
-				(path "/b111be58-5b18-5e09-a452-181893b11c74"
+				(path "/7d8bfbf7-e7f4-539c-a742-574ff9ec8fc2"
 					(reference "R247")
 					(unit 1)
@@
 		(instances
 			(project "AK5558-ADC"
-				(path "/b111be58-5b18-5e09-a452-181893b11c74"
+				(path "/7d8bfbf7-e7f4-539c-a742-574ff9ec8fc2"
 					(reference "R248")
 					(unit 1)
@@
 		(instances
 			(project "AK5558-ADC"
-				(path "/b111be58-5b18-5e09-a452-181893b11c74"
+				(path "/7d8bfbf7-e7f4-539c-a742-574ff9ec8fc2"
 					(reference "R249")
 					(unit 1)
@@
 		(instances
 			(project "AK5558-ADC"
-				(path "/b111be58-5b18-5e09-a452-181893b11c74"
+				(path "/7d8bfbf7-e7f4-539c-a742-574ff9ec8fc2"
 					(reference "R250")
 					(unit 1)
@@
 		(instances
 			(project "AK5558-ADC"
-				(path "/b111be58-5b18-5e09-a452-181893b11c74"
+				(path "/7d8bfbf7-e7f4-539c-a742-574ff9ec8fc2"
 					(reference "R261")
 					(unit 1)
@@
 		(instances
 			(project "AK5558-ADC"
-				(path "/b111be58-5b18-5e09-a452-181893b11c74"
+				(path "/7d8bfbf7-e7f4-539c-a742-574ff9ec8fc2"
 					(reference "C261")
 					(unit 1)
@@
 		(instances
 			(project "AK5558-ADC"
-				(path "/b111be58-5b18-5e09-a452-181893b11c74"
+				(path "/7d8bfbf7-e7f4-539c-a742-574ff9ec8fc2"
 					(reference "C271")
 					(unit 1)
@@
 		(instances
 			(project "AK5558-ADC"
-				(path "/b111be58-5b18-5e09-a452-181893b11c74"
+				(path "/7d8bfbf7-e7f4-539c-a742-574ff9ec8fc2"
 					(reference "R262")
 					(unit 1)
@@
 		(instances
 			(project "AK5558-ADC"
-				(path "/b111be58-5b18-5e09-a452-181893b11c74"
+				(path "/7d8bfbf7-e7f4-539c-a742-574ff9ec8fc2"
 					(reference "C262")
 					(unit 1)
@@
 		(instances
 			(project "AK5558-ADC"
-				(path "/b111be58-5b18-5e09-a452-181893b11c74"
+				(path "/7d8bfbf7-e7f4-539c-a742-574ff9ec8fc2"
 					(reference "C272")
 					(unit 1)
@@
 		(instances
 			(project "AK5558-ADC"
-				(path "/b111be58-5b18-5e09-a452-181893b11c74"
+				(path "/7d8bfbf7-e7f4-539c-a742-574ff9ec8fc2"
 					(reference "R263")
 					(unit 1)
@@
 		(instances
 			(project "AK5558-ADC"
-				(path "/b111be58-5b18-5e09-a452-181893b11c74"
+				(path "/7d8bfbf7-e7f4-539c-a742-574ff9ec8fc2"
 					(reference "C263")
 					(unit 1)
@@
 		(instances
 			(project "AK5558-ADC"
-				(path "/b111be58-5b18-5e09-a452-181893b11c74"
+				(path "/7d8bfbf7-e7f4-539c-a742-574ff9ec8fc2"
 					(reference "C273")
 					(unit 1)
@@
 		(instances
 			(project "AK5558-ADC"
-				(path "/b111be58-5b18-5e09-a452-181893b11c74"
+				(path "/7d8bfbf7-e7f4-539c-a742-574ff9ec8fc2"
 					(reference "R264")
 					(unit 1)
@@
 		(instances
 			(project "AK5558-ADC"
-				(path "/b111be58-5b18-5e09-a452-181893b11c74"
+				(path "/7d8bfbf7-e7f4-539c-a742-574ff9ec8fc2"
 					(reference "C264")
 					(unit 1)
@@
 		(instances
 			(project "AK5558-ADC"
-				(path "/b111be58-5b18-5e09-a452-181893b11c74"
+				(path "/7d8bfbf7-e7f4-539c-a742-574ff9ec8fc2"
 					(reference "C274")
 					(unit 1)
@@
 		(instances
 			(project "AK5558-ADC"
-				(path "/b111be58-5b18-5e09-a452-181893b11c74"
+				(path "/7d8bfbf7-e7f4-539c-a742-574ff9ec8fc2"
 					(reference "C281")
 					(unit 1)
@@
 		(instances
 			(project "AK5558-ADC"
-				(path "/b111be58-5b18-5e09-a452-181893b11c74"
+				(path "/7d8bfbf7-e7f4-539c-a742-574ff9ec8fc2"
 					(reference "C282")
 					(unit 1)
@@
 		(instances
 			(project "AK5558-ADC"
-				(path "/b111be58-5b18-5e09-a452-181893b11c74"
+				(path "/7d8bfbf7-e7f4-539c-a742-574ff9ec8fc2"
 					(reference "C283")
 					(unit 1)
@@
 		(instances
 			(project "AK5558-ADC"
-				(path "/b111be58-5b18-5e09-a452-181893b11c74"
+				(path "/7d8bfbf7-e7f4-539c-a742-574ff9ec8fc2"
 					(reference "C284")
 					(unit 1)
@@
 		(instances
 			(project "AK5558-ADC"
-				(path "/b111be58-5b18-5e09-a452-181893b11c74"
+				(path "/7d8bfbf7-e7f4-539c-a742-574ff9ec8fc2"
 					(reference "C285")
 					(unit 1)
@@
 		(instances
 			(project "AK5558-ADC"
-				(path "/b111be58-5b18-5e09-a452-181893b11c74"
+				(path "/7d8bfbf7-e7f4-539c-a742-574ff9ec8fc2"
 					(reference "C286")
 					(unit 1)
@@
 		(instances
 			(project "AK5558-ADC"
-				(path "/b111be58-5b18-5e09-a452-181893b11c74"
+				(path "/7d8bfbf7-e7f4-539c-a742-574ff9ec8fc2"
 					(reference "C287")
 					(unit 1)
