File: cad/kicad/AUDIO-8X8/Audio-8x8.kicad_pcb (KiCad board)
At the start: 6 copper layers, 78 x 268 mm, 578 parts, among them J101 AUDIO_TDM_CONTROL, J102 AUDIO_12V_POWER, J201 NC3MAV, J202 NC3MAV, J203 NC3MAV, J204 NC3MAV, J205 NC3MAV, J206 NC3MAV, J207 NC3MAV, J208 NC3MAV, J301 NC3FAV, J302 NC3FAV, J303 NC3FAV, J304 NC3FAV, J305 NC3FAV, J306 NC3FAV, J307 NC3FAV, J308 NC3FAV, J901 CHASSIS_BOND_TEST, K501 TQ2-12V, K502 TQ2-12V, K503 TQ2-12V, K504 TQ2-12V, K505 TQ2-12V, K506 TQ2-12V, K507 TQ2-12V, K508 TQ2-12V, Q501 2N7002K, Q502 2N7002K, Q503 2N7002K, Q504 2N7002K, Q505 2N7002K, Q506 2N7002K, Q507 2N7002K, Q508 2N7002K, U101 SN65LVDT2D, U102 SN65LVDT2D, U103 SN65LVDT2D, U104 SN65LVDT2D, U105 SN65LVDS1D, U106 SN74LVC1G11DBVR, U201 AK5558VN, U301 AK4458VN, U401 THAT1206S08-U, U402 THAT1206S08-U, U403 THAT1206S08-U, U404 THAT1206S08-U, U405 THAT1206S08-U, U406 THAT1206S08-U, U407 THAT1206S08-U, U408 THAT1206S08-U, U421 OPA1652AIDR, U422 OPA1652AIDR, U423 OPA1652AIDR, U424 OPA1652AIDR, U425 OPA1652AIDR, U426 OPA1652AIDR, U427 OPA1652AIDR, U428 OPA1652AIDR, U501 OPA1652AIDR, U502 OPA1652AIDR, U503 OPA1652AIDR, U504 OPA1652AIDR, U505 OPA1652AIDR, U506 OPA1652AIDR, U507 OPA1652AIDR, U508 OPA1652AIDR, U521 THAT1646S08-U, U522 THAT1646S08-U, U523 THAT1646S08-U, U524 THAT1646S08-U, U525 THAT1646S08-U, U526 THAT1646S08-U, U527 THAT1646S08-U, U528 THAT1646S08-U, U601 TRI 20-1223, U602 TPS62913RPU, U603 LT3045IMSE, U604 LT3045IMSE, U605 TPS7A2033PDBVR

Commit message: Fix PCB-A1 in-board 3D placement
Parts:
- C101, C102, C103, C104, C105, C106, C107, C261, C262, C263, C264, C271, C272, C273, C274, C281, C282, C283, C284, C285, C286, C287, C351, C352, C353, C354, C361, C362, C363, C364, C371, C372, C373, C374, C375, C4030, C4031, C4032, C4033, C4034, C4035, C4036, C4037, C4060, C4061, C4062, C4063, C4064, C4065, C4066, C4067, C4090, C4091, C4092, C4093, C4094, C4095, C4096, C4097, C4120, C4121, C4122, C4123, C4124, C4125, C4126, C4127, C4150, C4151, C4152, C4153, C4154, C4155, C4156, C4157, C4180, C4181, C4182, C4183, C4184, C4185, C4186, C4187, C4210, C4211, C4212, C4213, C4214, C4215, C4216, C4217, C4240, C4241, C4242, C4243, C4244, C4245, C4246, C4247, C5040, C5041, C5042, C5043, C5044, C5045, C5046, C5047, C5048, C5049, C5050, C5080, C5081, C5082, C5083, C5084, C5085, C5086, C5087, C5088, C5089, C5090, C5120, C5121, C5122, C5123, C5124, C5125, C5126, C5127, C5128, C5129, C5130, C5160, C5161, C5162, C5163, C5164, C5165, C5166, C5167, C5168, C5169, C5170, C5200, C5201, C5202, C5203, C5204, C5205, C5206, C5207, C5208, C5209, C5210, C5240, C5241, C5242, C5243, C5244, C5245, C5246, C5247, C5248, C5249, C5250, C5280, C5281, C5282, C5283, C5284, C5285, C5286, C5287, C5288, C5289, C5290, C5320, C5321, C5322, C5323, C5324, C5325, C5326, C5327, C5328, C5329, C5330, C601, C602, C603, C610, C611, C612, C613, C620, C621, C622, C623, C624, C630, C631, C632, C650, C651, C652, C670, C671, C672, C673, C901, D4030, D4031, D4032, D4033, D4034, D4035, D4060, D4061, D4062, D4063, D4064, D4065, D4090, D4091, D4092, D4093, D4094, D4095, D4120, D4121, D4122, D4123, D4124, D4125, D4150, D4151, D4152, D4153, D4154, D4155, D4180, D4181, D4182, D4183, D4184, D4185, D4210, D4211, D4212, D4213, D4214, D4215, D4240, D4241, D4242, D4243, D4244, D4245, D5040, D5041, D5042, D5043, D5044, D5080, D5081, D5082, D5083, D5084, D5120, D5121, D5122, D5123, D5124, D5160, D5161, D5162, D5163, D5164, D5200, D5201, D5202, D5203, D5204, D5240, D5241, D5242, D5243, D5244, D5280, D5281, D5282, D5283, D5284, D5320, D5321, D5322, D5323, D5324, F601, J101, J102, J901, K501, K502, K503, K504, K505, K506, K507, K508, L5040, L5041, L5080, L5081, L5120, L5121, L5160, L5161, L5200, L5201, L5240, L5241, L5280, L5281, L5320, L5321, L601, Q501, Q502, Q503, Q504, Q505, Q506, Q507, Q508, R111, R112, R113, R114, R115, R116, R117, R221, R222, R223, R224, R225, R226, R227, R228, R241, R242, R243, R244, R245, R246, R247, R248, R249, R250, R261, R262, R263, R264, R321, R322, R323, R331, R332, R351, R352, R353, R354, R4030, R4031, R4036, R4037, R4038, R4039, R4040, R4041, R4060, R4061, R4066, R4067, R4068, R4069, R4070, R4071, R4090, R4091, R4096, R4097, R4098, R4099, R4100, R4101, R4120, R4121, R4126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: moved to B.Cu
- moved C624 417.9 mm to (11.3, 210.5), turned to 90 degrees
- moved C623 406.6 mm to (15.0, 206.8)
- moved C4180 386.7 mm to (30.0, 154.8), turned to 90 degrees
- moved C374 384.3 mm to (5.21, 35.3)
- moved C375 382.0 mm to (14.3, 12.5)
- moved L5241 377.6 mm to (11.1, 146.0), turned to 90 degrees
- moved R321 377.5 mm to (15.3, 31.5)
- moved D5120 376.6 mm to (5.95, 152.1), turned to 90 degrees
- moved R264 374.8 mm to (11.3, 30.5)
- moved D4125 374.4 mm to (15.1, 142.4)
- moved C372 372.9 mm to (2.71, 35.3)
- moved D4124 372.1 mm to (9.64, 142.4)
- moved R263 371.8 mm to (7.28, 30.5)
- moved C5084 371.7 mm to (16.5, 105.5)
- moved C5083 369.6 mm to (10.0, 105.5)
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Other:
- board text added: "AUDIO-8X8 PCB-A1"
- board text added: "B.Cu BALANCED CHANNEL STAGES"
- board text added: "B.Cu DIGITAL / AKM"
- board text added: "B.Cu ISOLATED AUDIO POWER"
- board text removed: "AUDIO QUIET ZONE: NO PWM / SWITCH NODES"
- board text removed: "AUDIO-8X8 PCB-A0"
- board text removed: "UNPLACED / UNVERIFIED PCB FOOTPRINT STAGING - NOT BOARD GEOMETRY"
