File: cad/kicad/AUDIO-8X8/Audio-8x8.kicad_sch (KiCad schematic)
At the start: 21 parts, among them J101 AUDIO_TDM_CONTROL, J102 AUDIO_12V_POWER, J201 NC3MAV, J202 NC3MAV, J203 NC3MAV, J204 NC3MAV, J205 NC3MAV, J206 NC3MAV, J207 NC3MAV, J208 NC3MAV, J301 NC3FAV, J302 NC3FAV, J303 NC3FAV, J304 NC3FAV, J305 NC3FAV, J306 NC3FAV, J307 NC3FAV, J308 NC3FAV, J901 CHASSIS_BOND_TEST

Commit message: Audit schematic logic against controlled datasheets
Parts:
- removed J101: AUDIO_TDM_CONTROL, Connector_Molex_Milligrid:Molex_8783230xx_2x15_P2.0mm_Header_Vertical_Polarized_MountingPegs, symbol Connector_Generic:Conn_02x15_Odd_Even
- removed J102: AUDIO_12V_POWER, Connector_Molex:Molex_Micro-Fit_3.0_43045-0412_2x02_P3.00mm_Vertical, symbol Connector_Generic:Conn_02x02_Odd_Even
- added J9901: AUDIO_TDM_CONTROL, Connector_Molex_Milligrid:Molex_8783230xx_2x15_P2.0mm_Header_Vertical_Polarized_MountingPegs, symbol Connector_Generic:Conn_02x15_Odd_Even
- added J9902: AUDIO_12V_POWER, Connector_Molex:Molex_Micro-Fit_3.0_43045-0412_2x02_P3.00mm_Vertical, symbol Connector_Generic:Conn_02x02_Odd_Even
Connections:
- net AUDIO_12V: now also J9902.1 (Pin_1), J9902.2 (Pin_2)
- net AUDIO_ENABLE: now also J9901.24 (Pin_24)
- net AUDIO_PRESENT_N: now also J9901.23 (Pin_23)
- net AUD_ADC_RST_N: now also J9901.19 (Pin_19)
- net AUD_ADC_SDOUT_N: now also J9901.14 (Pin_14)
- net AUD_ADC_SDOUT_P: now also J9901.13 (Pin_13)
- net AUD_BCLK_N: now also J9901.6 (Pin_6)
- net AUD_BCLK_P: now also J9901.5 (Pin_5)
- net AUD_DAC_RST_N: now also J9901.20 (Pin_20)
- net AUD_DAC_SDIN_N: now also J9901.12 (Pin_12)
- net AUD_DAC_SDIN_P: now also J9901.11 (Pin_11)
- net AUD_FSYNC_N: now also J9901.8 (Pin_8)
- net AUD_FSYNC_P: now also J9901.7 (Pin_7)
- net AUD_I2C_SCL: now also J9901.17 (Pin_17)
- net AUD_I2C_SDA: now also J9901.18 (Pin_18)
- net AUD_IRQ_N: now also J9901.22 (Pin_22)
- net AUD_MCLK_N: now also J9901.2 (Pin_2)
- net AUD_MCLK_P: now also J9901.1 (Pin_1)
- net GND: now also J9901.10 (Pin_10), J9901.15 (Pin_15), J9901.16 (Pin_16), J9901.26 (Pin_26), J9901.29 (Pin_29), J9901.3 (Pin_3), J9901.30 (Pin_30), J9901.4 (Pin_4), J9901.9 (Pin_9), J9902.3 (Pin_3), J9902.4 (Pin_4)
- net LOGIC_3V3: now also J9901.25 (Pin_25)
- net TDM_SPARE_1: now also J9901.27 (Pin_27)
- net TDM_SPARE_2: now also J9901.28 (Pin_28)
- new net AUD_DAC_MUTE_CMD_N: J9901.21 (Pin_21)
Other:
- added sheet AK4458VN DAC (AK4458-DAC.kicad_sch)
- added sheet AK5558VN ADC (AK5558-ADC.kicad_sch)
- added sheet Audio Power (Audio-Power.kicad_sch)
- added sheet Balanced Inputs 1-8 (Audio-Inputs.kicad_sch)
- added sheet Balanced Outputs 1-8 (Audio-Outputs.kicad_sch)
- added sheet TDM / Clock / Control (Audio-TDM-Clock.kicad_sch)
- note added: "G. CONNECTED AUDIO-8X8 HIERARCHY"
- note added: "Root J9901/J9902 are interface-only duplicates; detailed J101/J102 own the production footprints."

Commit message: Implement direct socketed dual-SIM daughterboard
Parts:
- removed J301, J302, J303, J304, J305, J306, J307: NC3FAV, Connector_Audio:Jack_XLR_Neutrik_NC3FAV_Vertical, symbol Connector_Audio:NC3FAV
- added J202, J203, J204, J205, J206, J207, J208: NC3MAV, Connector_Audio:Jack_XLR_Neutrik_NC3MAV_Vertical, symbol Connector_Audio:NC3MAV
- J301: renamed from J202; value NC3MAV -> NC3FAV; footprint Connector_Audio:Jack_XLR_Neutrik_NC3MAV_Vertical -> Connector_Audio:Jack_XLR_Neutrik_NC3FAV_Vertical; symbol Connector_Audio:NC3MAV -> Connector_Audio:NC3FAV; MPN NC3MAV -> NC3FAV
- J302: renamed from J203; value NC3MAV -> NC3FAV; footprint Connector_Audio:Jack_XLR_Neutrik_NC3MAV_Vertical -> Connector_Audio:Jack_XLR_Neutrik_NC3FAV_Vertical; symbol Connector_Audio:NC3MAV -> Connector_Audio:NC3FAV; MPN NC3MAV -> NC3FAV
- J303: renamed from J204; value NC3MAV -> NC3FAV; footprint Connector_Audio:Jack_XLR_Neutrik_NC3MAV_Vertical -> Connector_Audio:Jack_XLR_Neutrik_NC3FAV_Vertical; symbol Connector_Audio:NC3MAV -> Connector_Audio:NC3FAV; MPN NC3MAV -> NC3FAV
- J304: renamed from J205; value NC3MAV -> NC3FAV; footprint Connector_Audio:Jack_XLR_Neutrik_NC3MAV_Vertical -> Connector_Audio:Jack_XLR_Neutrik_NC3FAV_Vertical; symbol Connector_Audio:NC3MAV -> Connector_Audio:NC3FAV; MPN NC3MAV -> NC3FAV
- J305: renamed from J206; value NC3MAV -> NC3FAV; footprint Connector_Audio:Jack_XLR_Neutrik_NC3MAV_Vertical -> Connector_Audio:Jack_XLR_Neutrik_NC3FAV_Vertical; symbol Connector_Audio:NC3MAV -> Connector_Audio:NC3FAV; MPN NC3MAV -> NC3FAV
- J306: renamed from J207; value NC3MAV -> NC3FAV; footprint Connector_Audio:Jack_XLR_Neutrik_NC3MAV_Vertical -> Connector_Audio:Jack_XLR_Neutrik_NC3FAV_Vertical; symbol Connector_Audio:NC3MAV -> Connector_Audio:NC3FAV; MPN NC3MAV -> NC3FAV
- J307: renamed from J208; value NC3MAV -> NC3FAV; footprint Connector_Audio:Jack_XLR_Neutrik_NC3MAV_Vertical -> Connector_Audio:Jack_XLR_Neutrik_NC3FAV_Vertical; symbol Connector_Audio:NC3MAV -> Connector_Audio:NC3FAV; MPN NC3MAV -> NC3FAV
Connections:
- net AIN_CH1_COLD: now also J301.3
- net AIN_CH1_HOT: now also J301.2
- net AIN_CH2_COLD: now also J302.3
- net AIN_CH2_HOT: now also J302.2
- net AIN_CH3_COLD: now also J303.3
- net AIN_CH3_HOT: now also J303.2
- net AIN_CH4_COLD: now also J304.3
- net AIN_CH4_HOT: now also J304.2
- net AIN_CH5_COLD: now also J305.3
- net AIN_CH5_HOT: now also J305.2
- net AIN_CH6_COLD: now also J306.3
- net AIN_CH6_HOT: now also J306.2
- net AIN_CH7_COLD: now also J307.3
- net AIN_CH7_HOT: now also J307.2
- net AOUT_CH2_COLD: now also J202.3; no longer J301.3
- net AOUT_CH2_HOT: now also J202.2; no longer J301.2
- net AOUT_CH3_COLD: now also J203.3; no longer J302.3
- net AOUT_CH3_HOT: now also J203.2; no longer J302.2
- net AOUT_CH4_COLD: now also J204.3; no longer J303.3
- net AOUT_CH4_HOT: now also J204.2; no longer J303.2
- net AOUT_CH5_COLD: now also J205.3; no longer J304.3
- net AOUT_CH5_HOT: now also J205.2; no longer J304.2
- net AOUT_CH6_COLD: now also J206.3; no longer J305.3
- net AOUT_CH6_HOT: now also J206.2; no longer J305.2
- net AOUT_CH7_COLD: now also J207.3; no longer J306.3
- net AOUT_CH7_HOT: now also J207.2; no longer J306.2
- net AOUT_CH8_COLD: now also J208.3; no longer J307.3
- net AOUT_CH8_HOT: now also J208.2; no longer J307.2
- net XLR_CHASSIS: now also J202.1, J202.G, J203.1, J203.G, J204.1, J204.G, J205.1, J205.G, J206.1, J206.G, J207.1, J207.G, J208.1, J208.G; no longer J301.G, J302.G, J303.G, J304.G, J305.G, J306.G, J307.G
Changed lines of the file:
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@@
 		(instances
 			(project "Audio-8x8"
-				(path "/a75e3689-a56f-5477-b683-87fede7d173d"
+				(path "/50e961a1-39e0-51e2-b65b-51977bd39aec"
 					(reference "J201")
 					(unit 1)
@@
 		(instances
 			(project "Audio-8x8"
-				(path "/a75e3689-a56f-5477-b683-87fede7d173d"
+				(path "/50e961a1-39e0-51e2-b65b-51977bd39aec"
 					(reference "J301")
 					(unit 1)
@@
 		(instances
 			(project "Audio-8x8"
-				(path "/a75e3689-a56f-5477-b683-87fede7d173d"
+				(path "/50e961a1-39e0-51e2-b65b-51977bd39aec"
 					(reference "J202")
 					(unit 1)
@@
 		(instances
 			(project "Audio-8x8"
-				(path "/a75e3689-a56f-5477-b683-87fede7d173d"
+				(path "/50e961a1-39e0-51e2-b65b-51977bd39aec"
 					(reference "J302")
 					(unit 1)
@@
 		(instances
 			(project "Audio-8x8"
-				(path "/a75e3689-a56f-5477-b683-87fede7d173d"
+				(path "/50e961a1-39e0-51e2-b65b-51977bd39aec"
 					(reference "J203")
 					(unit 1)
@@
 		(instances
 			(project "Audio-8x8"
-				(path "/a75e3689-a56f-5477-b683-87fede7d173d"
+				(path "/50e961a1-39e0-51e2-b65b-51977bd39aec"
 					(reference "J303")
 					(unit 1)
@@
 		(instances
 			(project "Audio-8x8"
-				(path "/a75e3689-a56f-5477-b683-87fede7d173d"
+				(path "/50e961a1-39e0-51e2-b65b-51977bd39aec"
 					(reference "J204")
 					(unit 1)
@@
 		(instances
 			(project "Audio-8x8"
-				(path "/a75e3689-a56f-5477-b683-87fede7d173d"
+				(path "/50e961a1-39e0-51e2-b65b-51977bd39aec"
 					(reference "J304")
 					(unit 1)
@@
 		(instances
 			(project "Audio-8x8"
-				(path "/a75e3689-a56f-5477-b683-87fede7d173d"
+				(path "/50e961a1-39e0-51e2-b65b-51977bd39aec"
 					(reference "J205")
 					(unit 1)
@@
 		(instances
 			(project "Audio-8x8"
-				(path "/a75e3689-a56f-5477-b683-87fede7d173d"
+				(path "/50e961a1-39e0-51e2-b65b-51977bd39aec"
 					(reference "J305")
 					(unit 1)
@@
 		(instances
 			(project "Audio-8x8"
-				(path "/a75e3689-a56f-5477-b683-87fede7d173d"
+				(path "/50e961a1-39e0-51e2-b65b-51977bd39aec"
 					(reference "J206")
 					(unit 1)
@@
 		(instances
 			(project "Audio-8x8"
-				(path "/a75e3689-a56f-5477-b683-87fede7d173d"
+				(path "/50e961a1-39e0-51e2-b65b-51977bd39aec"
 					(reference "J306")
 					(unit 1)
@@
 		(instances
 			(project "Audio-8x8"
-				(path "/a75e3689-a56f-5477-b683-87fede7d173d"
+				(path "/50e961a1-39e0-51e2-b65b-51977bd39aec"
 					(reference "J207")
 					(unit 1)
@@
 		(instances
 			(project "Audio-8x8"
-				(path "/a75e3689-a56f-5477-b683-87fede7d173d"
+				(path "/50e961a1-39e0-51e2-b65b-51977bd39aec"
 					(reference "J307")
 					(unit 1)
@@
 		(instances
 			(project "Audio-8x8"
-				(path "/a75e3689-a56f-5477-b683-87fede7d173d"
+				(path "/50e961a1-39e0-51e2-b65b-51977bd39aec"
 					(reference "J208")
 					(unit 1)
@@
 		(instances
 			(project "Audio-8x8"
-				(path "/a75e3689-a56f-5477-b683-87fede7d173d"
+				(path "/50e961a1-39e0-51e2-b65b-51977bd39aec"
 					(reference "J308")
 					(unit 1)
@@
 		(instances
 			(project "Audio-8x8"
-				(path "/a75e3689-a56f-5477-b683-87fede7d173d"
+				(path "/50e961a1-39e0-51e2-b65b-51977bd39aec"
 					(reference "J9901")
 					(unit 1)
@@
 		(instances
 			(project "Audio-8x8"
-				(path "/a75e3689-a56f-5477-b683-87fede7d173d"
+				(path "/50e961a1-39e0-51e2-b65b-51977bd39aec"
 					(reference "J9902")
 					(unit 1)
@@
 		(instances
 			(project "Audio-8x8"
-				(path "/a75e3689-a56f-5477-b683-87fede7d173d"
+				(path "/50e961a1-39e0-51e2-b65b-51977bd39aec"
 					(reference "R901")
 					(unit 1)
@@
 		(instances
 			(project "Audio-8x8"
-				(path "/a75e3689-a56f-5477-b683-87fede7d173d"
+				(path "/50e961a1-39e0-51e2-b65b-51977bd39aec"
 					(reference "C901")
 					(unit 1)
@@
 		(instances
 			(project "Audio-8x8"
-				(path "/a75e3689-a56f-5477-b683-87fede7d173d"
+				(path "/50e961a1-39e0-51e2-b65b-51977bd39aec"
 					(reference "J901")
 					(unit 1)
@@
 		(instances
 			(project "Audio-8x8"
-				(path "/a75e3689-a56f-5477-b683-87fede7d173d"
+				(path "/50e961a1-39e0-51e2-b65b-51977bd39aec"
 					(page "2")
 				)
@@
 		(instances
 			(project "Audio-8x8"
-				(path "/a75e3689-a56f-5477-b683-87fede7d173d"
+				(path "/50e961a1-39e0-51e2-b65b-51977bd39aec"
 					(page "3")
 				)
@@
 		(instances
 			(project "Audio-8x8"
-				(path "/a75e3689-a56f-5477-b683-87fede7d173d"
+				(path "/50e961a1-39e0-51e2-b65b-51977bd39aec"
 					(page "4")
 				)
@@
 		(instances
 			(project "Audio-8x8"
-				(path "/a75e3689-a56f-5477-b683-87fede7d173d"
+				(path "/50e961a1-39e0-51e2-b65b-51977bd39aec"
 					(page "5")
 				)
@@
 		(instances
 			(project "Audio-8x8"
-				(path "/a75e3689-a56f-5477-b683-87fede7d173d"
+				(path "/50e961a1-39e0-51e2-b65b-51977bd39aec"
 					(page "6")
 				)
@@
 		(instances
 			(project "Audio-8x8"
-				(path "/a75e3689-a56f-5477-b683-87fede7d173d"
+				(path "/50e961a1-39e0-51e2-b65b-51977bd39aec"
 					(page "7")
 				)
