File: cad/kicad/AUDIO-8X8/Audio-Inputs.kicad_sch (KiCad schematic)
At the start: 176 parts, among them U401 THAT1206S08-U, U402 THAT1206S08-U, U403 THAT1206S08-U, U404 THAT1206S08-U, U405 THAT1206S08-U, U406 THAT1206S08-U, U407 THAT1206S08-U, U408 THAT1206S08-U, U421 OPA1652AIDR, U422 OPA1652AIDR, U423 OPA1652AIDR, U424 OPA1652AIDR, U425 OPA1652AIDR, U426 OPA1652AIDR, U427 OPA1652AIDR, U428 OPA1652AIDR

Commit message: Audit schematic logic against controlled datasheets
Parts:
- added C4036, C4037, C4066, C4067, C4096, C4097, C4126, C4127, C4156, C4157, C4186, C4187, C4216, C4217, C4246, C4247: 100nF, Capacitor_SMD:C_0402_1005Metric, symbol Device:C
Connections:
- net AGND: now also C4036.2, C4037.2, C4066.2, C4067.2, C4096.2, C4097.2, C4126.2, C4127.2, C4156.2, C4157.2, C4186.2, C4187.2, C4216.2, C4217.2, C4246.2, C4247.2
- net AUDIO_N15V: now also C4037.1, C4067.1, C4097.1, C4127.1, C4157.1, C4187.1, C4217.1, C4247.1
- net AUDIO_P15V: now also C4036.1, C4066.1, C4096.1, C4126.1, C4156.1, C4186.1, C4216.1, C4246.1

Commit message: Implement direct socketed dual-SIM daughterboard
Parts:
- removed C4030, C4060, C4090, C4120, C4150, C4180, C4210, C4240: 470pF C0G, Capacitor_SMD:C_0603_1608Metric, symbol Device:C
- removed C4033, C4063, C4093, C4123, C4153, C4183, C4213, C4243: 10uF bipolar, Capacitor_THT:CP_Radial_D5.0mm_P2.00mm, symbol Device:C
- removed C4034, C4064, C4094, C4124, C4154, C4184, C4214: 3.3nF C0G, Capacitor_SMD:C_0603_1608Metric, symbol Device:C
- removed C4037, C4067, C4097, C4127, C4157, C4187, C4217, C4247: 100nF, Capacitor_SMD:C_0402_1005Metric, symbol Device:C
- removed R4030, R4031: 100R, Resistor_SMD:R_0603_1608Metric, symbol Device:R
- added C4245: 100nF, Capacitor_SMD:C_0402_1005Metric, symbol Device:C
- added D4034, D4035, D4064, D4065, D4094, D4095, D4124, D4125, D4154, D4155, D4184, D4185, D4214, D4215, D4244, D4245: 12V zener, Diode_SMD:D_SOD-123, symbol Device:D_Zener
- added R4038, R4068, R4098, R4128, R4158, R4188, R4218, R4248: 13k 0.1%, Resistor_SMD:R_0603_1608Metric, symbol Device:R
- added R4039, R4069, R4099, R4129, R4159, R4189, R4219, R4249: 1k 0.1%, Resistor_SMD:R_0603_1608Metric, symbol Device:R
- C4030: renamed from D4030; value 1N4148W -> 470pF C0G; footprint Diode_SMD:D_SOD-123 -> Capacitor_SMD:C_0603_1608Metric; symbol Device:D -> Device:C; MPN 1N4148W-7-F -> GRM1885C1H471JA01D; Manufacturer Diodes Incorporated -> Murata
- C4031: renamed from D4031; value 1N4148W -> 470pF C0G; footprint Diode_SMD:D_SOD-123 -> Capacitor_SMD:C_0603_1608Metric; symbol Device:D -> Device:C; MPN 1N4148W-7-F -> GRM1885C1H471JA01D; Manufacturer Diodes Incorporated -> Murata
- C4032: renamed from D4032; value 1N4148W -> 100pF C0G; footprint Diode_SMD:D_SOD-123 -> Capacitor_SMD:C_0603_1608Metric; symbol Device:D -> Device:C; MPN 1N4148W-7-F -> GRM1885C1H101JA01D; Manufacturer Diodes Incorporated -> Murata
- C4033: renamed from R4038; value 13k 0.1% -> 10uF bipolar; footprint Resistor_SMD:R_0603_1608Metric -> Capacitor_THT:CP_Radial_D5.0mm_P2.00mm; symbol Device:R -> Device:C; MPN RC0603FR-0713KL -> UES1H100MDM1TD; Manufacturer Yageo -> Nichicon
- C4034: renamed from R4060; value 100R -> 3.3nF C0G; footprint Resistor_SMD:R_0603_1608Metric -> Capacitor_SMD:C_0603_1608Metric; symbol Device:R -> Device:C; MPN RC0603FR-07100RL -> GRM1885C1H332JA01D; Manufacturer Yageo -> Murata
- C4035: renamed from R4061; value 100R -> 100nF; footprint Resistor_SMD:R_0603_1608Metric -> Capacitor_SMD:C_0402_1005Metric; symbol Device:R -> Device:C; MPN RC0603FR-07100RL -> C1005X7R1H104K050BB; Manufacturer Yageo -> TDK
- C4036: renamed from R4036; value 13k 0.1% -> 100nF; footprint Resistor_SMD:R_0603_1608Metric -> Capacitor_SMD:C_0402_1005Metric; symbol Device:R -> Device:C; MPN RC0603FR-0713KL -> C1005X7R1H104K050BB; Manufacturer Yageo -> TDK
- C4037: renamed from R4037; value 1k 0.1% -> 100nF; footprint Resistor_SMD:R_0603_1608Metric -> Capacitor_SMD:C_0402_1005Metric; symbol Device:R -> Device:C; MPN TNPW06031K00BEEA -> C1005X7R1H104K050BB; Manufacturer Vishay -> TDK
- C4060: renamed from D4060; value 1N4148W -> 470pF C0G; footprint Diode_SMD:D_SOD-123 -> Capacitor_SMD:C_0603_1608Metric; symbol Device:D -> Device:C; MPN 1N4148W-7-F -> GRM1885C1H471JA01D; Manufacturer Diodes Incorporated -> Murata
- C4061: renamed from D4061; value 1N4148W -> 470pF C0G; footprint Diode_SMD:D_SOD-123 -> Capacitor_SMD:C_0603_1608Metric; symbol Device:D -> Device:C; MPN 1N4148W-7-F -> GRM1885C1H471JA01D; Manufacturer Diodes Incorporated -> Murata
- C4062: renamed from D4062; value 1N4148W -> 100pF C0G; footprint Diode_SMD:D_SOD-123 -> Capacitor_SMD:C_0603_1608Metric; symbol Device:D -> Device:C; MPN 1N4148W-7-F -> GRM1885C1H101JA01D; Manufacturer Diodes Incorporated -> Murata
- C4063: renamed from R4068; value 13k 0.1% -> 10uF bipolar; footprint Resistor_SMD:R_0603_1608Metric -> Capacitor_THT:CP_Radial_D5.0mm_P2.00mm; symbol Device:R -> Device:C; MPN RC0603FR-0713KL -> UES1H100MDM1TD; Manufacturer Yageo -> Nichicon
- C4064: renamed from R4090; value 100R -> 3.3nF C0G; footprint Resistor_SMD:R_0603_1608Metric -> Capacitor_SMD:C_0603_1608Metric; symbol Device:R -> Device:C; MPN RC0603FR-07100RL -> GRM1885C1H332JA01D; Manufacturer Yageo -> Murata
- C4065: renamed from R4091; value 100R -> 100nF; footprint Resistor_SMD:R_0603_1608Metric -> Capacitor_SMD:C_0402_1005Metric; symbol Device:R -> Device:C; MPN RC0603FR-07100RL -> C1005X7R1H104K050BB; Manufacturer Yageo -> TDK
- C4066: renamed from R4066; value 13k 0.1% -> 100nF; footprint Resistor_SMD:R_0603_1608Metric -> Capacitor_SMD:C_0402_1005Metric; symbol Device:R -> Device:C; MPN RC0603FR-0713KL -> C1005X7R1H104K050BB; Manufacturer Yageo -> TDK
- C4067: renamed from R4067; value 1k 0.1% -> 100nF; footprint Resistor_SMD:R_0603_1608Metric -> Capacitor_SMD:C_0402_1005Metric; symbol Device:R -> Device:C; MPN TNPW06031K00BEEA -> C1005X7R1H104K050BB; Manufacturer Vishay -> TDK
- C4090: renamed from D4090; value 1N4148W -> 470pF C0G; footprint Diode_SMD:D_SOD-123 -> Capacitor_SMD:C_0603_1608Metric; symbol Device:D -> Device:C; MPN 1N4148W-7-F -> GRM1885C1H471JA01D; Manufacturer Diodes Incorporated -> Murata
- C4091: renamed from D4091; value 1N4148W -> 470pF C0G; footprint Diode_SMD:D_SOD-123 -> Capacitor_SMD:C_0603_1608Metric; symbol Device:D -> Device:C; MPN 1N4148W-7-F -> GRM1885C1H471JA01D; Manufacturer Diodes Incorporated -> Murata
- C4092: renamed from D4092; value 1N4148W -> 100pF C0G; footprint Diode_SMD:D_SOD-123 -> Capacitor_SMD:C_0603_1608Metric; symbol Device:D -> Device:C; MPN 1N4148W-7-F -> GRM1885C1H101JA01D; Manufacturer Diodes Incorporated -> Murata
- C4093: renamed from R4098; value 13k 0.1% -> 10uF bipolar; footprint Resistor_SMD:R_0603_1608Metric -> Capacitor_THT:CP_Radial_D5.0mm_P2.00mm; symbol Device:R -> Device:C; MPN RC0603FR-0713KL -> UES1H100MDM1TD; Manufacturer Yageo -> Nichicon
- C4094: renamed from R4120; value 100R -> 3.3nF C0G; footprint Resistor_SMD:R_0603_1608Metric -> Capacitor_SMD:C_0603_1608Metric; symbol Device:R -> Device:C; MPN RC0603FR-07100RL -> GRM1885C1H332JA01D; Manufacturer Yageo -> Murata
- C4095: renamed from R4121; value 100R -> 100nF; footprint Resistor_SMD:R_0603_1608Metric -> Capacitor_SMD:C_0402_1005Metric; symbol Device:R -> Device:C; MPN RC0603FR-07100RL -> C1005X7R1H104K050BB; Manufacturer Yageo -> TDK
- C4096: renamed from R4096; value 13k 0.1% -> 100nF; footprint Resistor_SMD:R_0603_1608Metric -> Capacitor_SMD:C_0402_1005Metric; symbol Device:R -> Device:C; MPN RC0603FR-0713KL -> C1005X7R1H104K050BB; Manufacturer Yageo -> TDK
- C4097: renamed from R4097; value 1k 0.1% -> 100nF; footprint Resistor_SMD:R_0603_1608Metric -> Capacitor_SMD:C_0402_1005Metric; symbol Device:R -> Device:C; MPN TNPW06031K00BEEA -> C1005X7R1H104K050BB; Manufacturer Vishay -> TDK
- C4120: renamed from D4120; value 1N4148W -> 470pF C0G; footprint Diode_SMD:D_SOD-123 -> Capacitor_SMD:C_0603_1608Metric; symbol Device:D -> Device:C; MPN 1N4148W-7-F -> GRM1885C1H471JA01D; Manufacturer Diodes Incorporated -> Murata
- C4121: renamed from D4121; value 1N4148W -> 470pF C0G; footprint Diode_SMD:D_SOD-123 -> Capacitor_SMD:C_0603_1608Metric; symbol Device:D -> Device:C; MPN 1N4148W-7-F -> GRM1885C1H471JA01D; Manufacturer Diodes Incorporated -> Murata
- C4122: renamed from D4122; value 1N4148W -> 100pF C0G; footprint Diode_SMD:D_SOD-123 -> Capacitor_SMD:C_0603_1608Metric; symbol Device:D -> Device:C; MPN 1N4148W-7-F -> GRM1885C1H101JA01D; Manufacturer Diodes Incorporated -> Murata
- C4123: renamed from R4128; value 13k 0.1% -> 10uF bipolar; footprint Resistor_SMD:R_0603_1608Metric -> Capacitor_THT:CP_Radial_D5.0mm_P2.00mm; symbol Device:R -> Device:C; MPN RC0603FR-0713KL -> UES1H100MDM1TD; Manufacturer Yageo -> Nichicon
- C4124: renamed from R4150; value 100R -> 3.3nF C0G; footprint Resistor_SMD:R_0603_1608Metric -> Capacitor_SMD:C_0603_1608Metric; symbol Device:R -> Device:C; MPN RC0603FR-07100RL -> GRM1885C1H332JA01D; Manufacturer Yageo -> Murata
- C4125: renamed from R4151; value 100R -> 100nF; footprint Resistor_SMD:R_0603_1608Metric -> Capacitor_SMD:C_0402_1005Metric; symbol Device:R -> Device:C; MPN RC0603FR-07100RL -> C1005X7R1H104K050BB; Manufacturer Yageo -> TDK
- C4126: renamed from R4126; value 13k 0.1% -> 100nF; footprint Resistor_SMD:R_0603_1608Metric -> Capacitor_SMD:C_0402_1005Metric; symbol Device:R -> Device:C; MPN RC0603FR-0713KL -> C1005X7R1H104K050BB; Manufacturer Yageo -> TDK
- C4127: renamed from R4127; value 1k 0.1% -> 100nF; footprint Resistor_SMD:R_0603_1608Metric -> Capacitor_SMD:C_0402_1005Metric; symbol Device:R -> Device:C; MPN TNPW06031K00BEEA -> C1005X7R1H104K050BB; Manufacturer Vishay -> TDK
- C4150: renamed from D4150; value 1N4148W -> 470pF C0G; footprint Diode_SMD:D_SOD-123 -> Capacitor_SMD:C_0603_1608Metric; symbol Device:D -> Device:C; MPN 1N4148W-7-F -> GRM1885C1H471JA01D; Manufacturer Diodes Incorporated -> Murata
- C4151: renamed from D4151; value 1N4148W -> 470pF C0G; footprint Diode_SMD:D_SOD-123 -> Capacitor_SMD:C_0603_1608Metric; symbol Device:D -> Device:C; MPN 1N4148W-7-F -> GRM1885C1H471JA01D; Manufacturer Diodes Incorporated -> Murata
- C4152: renamed from D4152; value 1N4148W -> 100pF C0G; footprint Diode_SMD:D_SOD-123 -> Capacitor_SMD:C_0603_1608Metric; symbol Device:D -> Device:C; MPN 1N4148W-7-F -> GRM1885C1H101JA01D; Manufacturer Diodes Incorporated -> Murata
- C4153: renamed from R4158; value 13k 0.1% -> 10uF bipolar; footprint Resistor_SMD:R_0603_1608Metric -> Capacitor_THT:CP_Radial_D5.0mm_P2.00mm; symbol Device:R -> Device:C; MPN RC0603FR-0713KL -> UES1H100MDM1TD; Manufacturer Yageo -> Nichicon
- C4154: renamed from R4180; value 100R -> 3.3nF C0G; footprint Resistor_SMD:R_0603_1608Metric -> Capacitor_SMD:C_0603_1608Metric; symbol Device:R -> Device:C; MPN RC0603FR-07100RL -> GRM1885C1H332JA01D; Manufacturer Yageo -> Murata
- C4155: renamed from R4181; value 100R -> 100nF; footprint Resistor_SMD:R_0603_1608Metric -> Capacitor_SMD:C_0402_1005Metric; symbol Device:R -> Device:C; MPN RC0603FR-07100RL -> C1005X7R1H104K050BB; Manufacturer Yageo -> TDK
- C4156: renamed from R4156; value 13k 0.1% -> 100nF; footprint Resistor_SMD:R_0603_1608Metric -> Capacitor_SMD:C_0402_1005Metric; symbol Device:R -> Device:C; MPN RC0603FR-0713KL -> C1005X7R1H104K050BB; Manufacturer Yageo -> TDK
- C4157: renamed from R4157; value 1k 0.1% -> 100nF; footprint Resistor_SMD:R_0603_1608Metric -> Capacitor_SMD:C_0402_1005Metric; symbol Device:R -> Device:C; MPN TNPW06031K00BEEA -> C1005X7R1H104K050BB; Manufacturer Vishay -> TDK
- C4180: renamed from D4180; value 1N4148W -> 470pF C0G; footprint Diode_SMD:D_SOD-123 -> Capacitor_SMD:C_0603_1608Metric; symbol Device:D -> Device:C; MPN 1N4148W-7-F -> GRM1885C1H471JA01D; Manufacturer Diodes Incorporated -> Murata
- C4181: renamed from D4181; value 1N4148W -> 470pF C0G; footprint Diode_SMD:D_SOD-123 -> Capacitor_SMD:C_0603_1608Metric; symbol Device:D -> Device:C; MPN 1N4148W-7-F -> GRM1885C1H471JA01D; Manufacturer Diodes Incorporated -> Murata
- C4182: renamed from D4182; value 1N4148W -> 100pF C0G; footprint Diode_SMD:D_SOD-123 -> Capacitor_SMD:C_0603_1608Metric; symbol Device:D -> Device:C; MPN 1N4148W-7-F -> GRM1885C1H101JA01D; Manufacturer Diodes Incorporated -> Murata
- C4183: renamed from R4188; value 13k 0.1% -> 10uF bipolar; footprint Resistor_SMD:R_0603_1608Metric -> Capacitor_THT:CP_Radial_D5.0mm_P2.00mm; symbol Device:R -> Device:C; MPN RC0603FR-0713KL -> UES1H100MDM1TD; Manufacturer Yageo -> Nichicon
- C4184: renamed from R4210; value 100R -> 3.3nF C0G; footprint Resistor_SMD:R_0603_1608Metric -> Capacitor_SMD:C_0603_1608Metric; symbol Device:R -> Device:C; MPN RC0603FR-07100RL -> GRM1885C1H332JA01D; Manufacturer Yageo -> Murata
- C4185: renamed from R4211; value 100R -> 100nF; footprint Resistor_SMD:R_0603_1608Metric -> Capacitor_SMD:C_0402_1005Metric; symbol Device:R -> Device:C; MPN RC0603FR-07100RL -> C1005X7R1H104K050BB; Manufacturer Yageo -> TDK
- C4186: renamed from R4186; value 13k 0.1% -> 100nF; footprint Resistor_SMD:R_0603_1608Metric -> Capacitor_SMD:C_0402_1005Metric; symbol Device:R -> Device:C; MPN RC0603FR-0713KL -> C1005X7R1H104K050BB; Manufacturer Yageo -> TDK
- C4187: renamed from R4187; value 1k 0.1% -> 100nF; footprint Resistor_SMD:R_0603_1608Metric -> Capacitor_SMD:C_0402_1005Metric; symbol Device:R -> Device:C; MPN TNPW06031K00BEEA -> C1005X7R1H104K050BB; Manufacturer Vishay -> TDK
- C4210: renamed from D4210; value 1N4148W -> 470pF C0G; footprint Diode_SMD:D_SOD-123 -> Capacitor_SMD:C_0603_1608Metric; symbol Device:D -> Device:C; MPN 1N4148W-7-F -> GRM1885C1H471JA01D; Manufacturer Diodes Incorporated -> Murata
- C4211: renamed from D4211; value 1N4148W -> 470pF C0G; footprint Diode_SMD:D_SOD-123 -> Capacitor_SMD:C_0603_1608Metric; symbol Device:D -> Device:C; MPN 1N4148W-7-F -> GRM1885C1H471JA01D; Manufacturer Diodes Incorporated -> Murata
- C4212: renamed from D4212; value 1N4148W -> 100pF C0G; footprint Diode_SMD:D_SOD-123 -> Capacitor_SMD:C_0603_1608Metric; symbol Device:D -> Device:C; MPN 1N4148W-7-F -> GRM1885C1H101JA01D; Manufacturer Diodes Incorporated -> Murata
- C4213: renamed from R4218; value 13k 0.1% -> 10uF bipolar; footprint Resistor_SMD:R_0603_1608Metric -> Capacitor_THT:CP_Radial_D5.0mm_P2.00mm; symbol Device:R -> Device:C; MPN RC0603FR-0713KL -> UES1H100MDM1TD; Manufacturer Yageo -> Nichicon
- C4214: renamed from R4240; value 100R -> 3.3nF C0G; footprint Resistor_SMD:R_0603_1608Metric -> Capacitor_SMD:C_0603_1608Metric; symbol Device:R -> Device:C; MPN RC0603FR-07100RL -> GRM1885C1H332JA01D; Manufacturer Yageo -> Murata
- C4215: renamed from R4241; value 100R -> 100nF; footprint Resistor_SMD:R_0603_1608Metric -> Capacitor_SMD:C_0402_1005Metric; symbol Device:R -> Device:C; MPN RC0603FR-07100RL -> C1005X7R1H104K050BB; Manufacturer Yageo -> TDK
- C4216: renamed from R4216; value 13k 0.1% -> 100nF; footprint Resistor_SMD:R_0603_1608Metric -> Capacitor_SMD:C_0402_1005Metric; symbol Device:R -> Device:C; MPN RC0603FR-0713KL -> C1005X7R1H104K050BB; Manufacturer Yageo -> TDK
- C4217: renamed from R4217; value 1k 0.1% -> 100nF; footprint Resistor_SMD:R_0603_1608Metric -> Capacitor_SMD:C_0402_1005Metric; symbol Device:R -> Device:C; MPN TNPW06031K00BEEA -> C1005X7R1H104K050BB; Manufacturer Vishay -> TDK
- C4240: renamed from D4240; value 1N4148W -> 470pF C0G; footprint Diode_SMD:D_SOD-123 -> Capacitor_SMD:C_0603_1608Metric; symbol Device:D -> Device:C; MPN 1N4148W-7-F -> GRM1885C1H471JA01D; Manufacturer Diodes Incorporated -> Murata
- C4241: renamed from D4241; value 1N4148W -> 470pF C0G; footprint Diode_SMD:D_SOD-123 -> Capacitor_SMD:C_0603_1608Metric; symbol Device:D -> Device:C; MPN 1N4148W-7-F -> GRM1885C1H471JA01D; Manufacturer Diodes Incorporated -> Murata
- C4242: renamed from D4242; value 1N4148W -> 100pF C0G; footprint Diode_SMD:D_SOD-123 -> Capacitor_SMD:C_0603_1608Metric; symbol Device:D -> Device:C; MPN 1N4148W-7-F -> GRM1885C1H101JA01D; Manufacturer Diodes Incorporated -> Murata
- C4243: renamed from R4248; value 13k 0.1% -> 10uF bipolar; footprint Resistor_SMD:R_0603_1608Metric -> Capacitor_THT:CP_Radial_D5.0mm_P2.00mm; symbol Device:R -> Device:C; MPN RC0603FR-0713KL -> UES1H100MDM1TD; Manufacturer Yageo -> Nichicon
- C4246: renamed from R4246; value 13k 0.1% -> 100nF; footprint Resistor_SMD:R_0603_1608Metric -> Capacitor_SMD:C_0402_1005Metric; symbol Device:R -> Device:C; MPN RC0603FR-0713KL -> C1005X7R1H104K050BB; Manufacturer Yageo -> TDK
- C4247: renamed from R4247; value 1k 0.1% -> 100nF; footprint Resistor_SMD:R_0603_1608Metric -> Capacitor_SMD:C_0402_1005Metric; symbol Device:R -> Device:C; MPN TNPW06031K00BEEA -> C1005X7R1H104K050BB; Manufacturer Vishay -> TDK
- D4031: renamed from D4034; value 12V zener -> 1N4148W; symbol Device:D_Zener -> Device:D; MPN BZT52C12-7-F -> 1N4148W-7-F
- D4032: renamed from D4035; value 12V zener -> 1N4148W; symbol Device:D_Zener -> Device:D; MPN BZT52C12-7-F -> 1N4148W-7-F
- D4033: renamed from U401; value THAT1206S08-U -> 1N4148W; footprint Package_SO:SOIC-8_3.9x4.9mm_P1.27mm -> Diode_SMD:D_SOD-123; symbol CM5Carrier:THAT1206 -> Device:D; MPN THAT1206S08-U -> 1N4148W-7-F; Manufacturer THAT Corporation -> Diodes Incorporated
- D4061: renamed from D4064; value 12V zener -> 1N4148W; symbol Device:D_Zener -> Device:D; MPN BZT52C12-7-F -> 1N4148W-7-F
- D4062: renamed from D4065; value 12V zener -> 1N4148W; symbol Device:D_Zener -> Device:D; MPN BZT52C12-7-F -> 1N4148W-7-F
- D4063: renamed from U402; value THAT1206S08-U -> 1N4148W; footprint Package_SO:SOIC-8_3.9x4.9mm_P1.27mm -> Diode_SMD:D_SOD-123; symbol CM5Carrier:THAT1206 -> Device:D; MPN THAT1206S08-U -> 1N4148W-7-F; Manufacturer THAT Corporation -> Diodes Incorporated
- D4091: renamed from D4094; value 12V zener -> 1N4148W; symbol Device:D_Zener -> Device:D; MPN BZT52C12-7-F -> 1N4148W-7-F
- D4092: renamed from D4095; value 12V zener -> 1N4148W; symbol Device:D_Zener -> Device:D; MPN BZT52C12-7-F -> 1N4148W-7-F
- D4093: renamed from U403; value THAT1206S08-U -> 1N4148W; footprint Package_SO:SOIC-8_3.9x4.9mm_P1.27mm -> Diode_SMD:D_SOD-123; symbol CM5Carrier:THAT1206 -> Device:D; MPN THAT1206S08-U -> 1N4148W-7-F; Manufacturer THAT Corporation -> Diodes Incorporated
- D4121: renamed from D4124; value 12V zener -> 1N4148W; symbol Device:D_Zener -> Device:D; MPN BZT52C12-7-F -> 1N4148W-7-F
- D4122: renamed from D4125; value 12V zener -> 1N4148W; symbol Device:D_Zener -> Device:D; MPN BZT52C12-7-F -> 1N4148W-7-F
- D4123: renamed from U404; value THAT1206S08-U -> 1N4148W; footprint Package_SO:SOIC-8_3.9x4.9mm_P1.27mm -> Diode_SMD:D_SOD-123; symbol CM5Carrier:THAT1206 -> Device:D; MPN THAT1206S08-U -> 1N4148W-7-F; Manufacturer THAT Corporation -> Diodes Incorporated
- D4151: renamed from D4154; value 12V zener -> 1N4148W; symbol Device:D_Zener -> Device:D; MPN BZT52C12-7-F -> 1N4148W-7-F
- D4152: renamed from D4155; value 12V zener -> 1N4148W; symbol Device:D_Zener -> Device:D; MPN BZT52C12-7-F -> 1N4148W-7-F
- D4153: renamed from U405; value THAT1206S08-U -> 1N4148W; footprint Package_SO:SOIC-8_3.9x4.9mm_P1.27mm -> Diode_SMD:D_SOD-123; symbol CM5Carrier:THAT1206 -> Device:D; MPN THAT1206S08-U -> 1N4148W-7-F; Manufacturer THAT Corporation -> Diodes Incorporated
- D4181: renamed from D4184; value 12V zener -> 1N4148W; symbol Device:D_Zener -> Device:D; MPN BZT52C12-7-F -> 1N4148W-7-F
- D4182: renamed from D4185; value 12V zener -> 1N4148W; symbol Device:D_Zener -> Device:D; MPN BZT52C12-7-F -> 1N4148W-7-F
- D4183: renamed from U406; value THAT1206S08-U -> 1N4148W; footprint Package_SO:SOIC-8_3.9x4.9mm_P1.27mm -> Diode_SMD:D_SOD-123; symbol CM5Carrier:THAT1206 -> Device:D; MPN THAT1206S08-U -> 1N4148W-7-F; Manufacturer THAT Corporation -> Diodes Incorporated
- D4211: renamed from D4214; value 12V zener -> 1N4148W; symbol Device:D_Zener -> Device:D; MPN BZT52C12-7-F -> 1N4148W-7-F
- D4212: renamed from D4215; value 12V zener -> 1N4148W; symbol Device:D_Zener -> Device:D; MPN BZT52C12-7-F -> 1N4148W-7-F
- D4213: renamed from U407; value THAT1206S08-U -> 1N4148W; footprint Package_SO:SOIC-8_3.9x4.9mm_P1.27mm -> Diode_SMD:D_SOD-123; symbol CM5Carrier:THAT1206 -> Device:D; MPN THAT1206S08-U -> 1N4148W-7-F; Manufacturer THAT Corporation -> Diodes Incorporated
- D4241: renamed from D4244; value 12V zener -> 1N4148W; symbol Device:D_Zener -> Device:D; MPN BZT52C12-7-F -> 1N4148W-7-F
- D4242: renamed from D4245; value 12V zener -> 1N4148W; symbol Device:D_Zener -> Device:D; MPN BZT52C12-7-F -> 1N4148W-7-F
- D4243: renamed from U408; value THAT1206S08-U -> 1N4148W; footprint Package_SO:SOIC-8_3.9x4.9mm_P1.27mm -> Diode_SMD:D_SOD-123; symbol CM5Carrier:THAT1206 -> Device:D; MPN THAT1206S08-U -> 1N4148W-7-F; Manufacturer THAT Corporation -> Diodes Incorporated
- R4030: renamed from C4031; value 470pF C0G -> 100R; footprint Capacitor_SMD:C_0603_1608Metric -> Resistor_SMD:R_0603_1608Metric; symbol Device:C -> Device:R; MPN GRM1885C1H471JA01D -> RC0603FR-07100RL; Manufacturer Murata -> Yageo
- R4031: renamed from C4032; value 100pF C0G -> 100R; footprint Capacitor_SMD:C_0603_1608Metric -> Resistor_SMD:R_0603_1608Metric; symbol Device:C -> Device:R; MPN GRM1885C1H101JA01D -> RC0603FR-07100RL; Manufacturer Murata -> Yageo
- R4036: renamed from R4039; value 1k 0.1% -> 13k 0.1%; MPN TNPW06031K00BEEA -> RC0603FR-0713KL; Manufacturer Vishay -> Yageo
- R4037: renamed from U421; value OPA1652AIDR -> 1k 0.1%; footprint Package_SO:SOIC-8_3.9x4.9mm_P1.27mm -> Resistor_SMD:R_0603_1608Metric; symbol CM5Carrier:OPA1652 -> Device:R; MPN OPA1652AIDR -> TNPW06031K00BEEA; Manufacturer Texas Instruments -> Vishay
- R4040: renamed from C4035; value 100nF -> 220R; footprint Capacitor_SMD:C_0402_1005Metric -> Resistor_SMD:R_0603_1608Metric; symbol Device:C -> Device:R; MPN C1005X7R1H104K050BB -> RC0603FR-07220RL; Manufacturer TDK -> Yageo
- R4060: renamed from C4061; value 470pF C0G -> 100R; footprint Capacitor_SMD:C_0603_1608Metric -> Resistor_SMD:R_0603_1608Metric; symbol Device:C -> Device:R; MPN GRM1885C1H471JA01D -> RC0603FR-07100RL; Manufacturer Murata -> Yageo
- R4061: renamed from C4062; value 100pF C0G -> 100R; footprint Capacitor_SMD:C_0603_1608Metric -> Resistor_SMD:R_0603_1608Metric; symbol Device:C -> Device:R; MPN GRM1885C1H101JA01D -> RC0603FR-07100RL; Manufacturer Murata -> Yageo
- R4066: renamed from R4069; value 1k 0.1% -> 13k 0.1%; MPN TNPW06031K00BEEA -> RC0603FR-0713KL; Manufacturer Vishay -> Yageo
- R4067: renamed from U422; value OPA1652AIDR -> 1k 0.1%; footprint Package_SO:SOIC-8_3.9x4.9mm_P1.27mm -> Resistor_SMD:R_0603_1608Metric; symbol CM5Carrier:OPA1652 -> Device:R; MPN OPA1652AIDR -> TNPW06031K00BEEA; Manufacturer Texas Instruments -> Vishay
- R4070: renamed from C4065; value 100nF -> 220R; footprint Capacitor_SMD:C_0402_1005Metric -> Resistor_SMD:R_0603_1608Metric; symbol Device:C -> Device:R; MPN C1005X7R1H104K050BB -> RC0603FR-07220RL; Manufacturer TDK -> Yageo
- R4090: renamed from C4091; value 470pF C0G -> 100R; footprint Capacitor_SMD:C_0603_1608Metric -> Resistor_SMD:R_0603_1608Metric; symbol Device:C -> Device:R; MPN GRM1885C1H471JA01D -> RC0603FR-07100RL; Manufacturer Murata -> Yageo
- R4091: renamed from C4092; value 100pF C0G -> 100R; footprint Capacitor_SMD:C_0603_1608Metric -> Resistor_SMD:R_0603_1608Metric; symbol Device:C -> Device:R; MPN GRM1885C1H101JA01D -> RC0603FR-07100RL; Manufacturer Murata -> Yageo
- R4096: renamed from R4099; value 1k 0.1% -> 13k 0.1%; MPN TNPW06031K00BEEA -> RC0603FR-0713KL; Manufacturer Vishay -> Yageo
- R4097: renamed from U423; value OPA1652AIDR -> 1k 0.1%; footprint Package_SO:SOIC-8_3.9x4.9mm_P1.27mm -> Resistor_SMD:R_0603_1608Metric; symbol CM5Carrier:OPA1652 -> Device:R; MPN OPA1652AIDR -> TNPW06031K00BEEA; Manufacturer Texas Instruments -> Vishay
- R4100: renamed from C4095; value 100nF -> 220R; footprint Capacitor_SMD:C_0402_1005Metric -> Resistor_SMD:R_0603_1608Metric; symbol Device:C -> Device:R; MPN C1005X7R1H104K050BB -> RC0603FR-07220RL; Manufacturer TDK -> Yageo
- R4120: renamed from C4121; value 470pF C0G -> 100R; footprint Capacitor_SMD:C_0603_1608Metric -> Resistor_SMD:R_0603_1608Metric; symbol Device:C -> Device:R; MPN GRM1885C1H471JA01D -> RC0603FR-07100RL; Manufacturer Murata -> Yageo
- R4121: renamed from C4122; value 100pF C0G -> 100R; footprint Capacitor_SMD:C_0603_1608Metric -> Resistor_SMD:R_0603_1608Metric; symbol Device:C -> Device:R; MPN GRM1885C1H101JA01D -> RC0603FR-07100RL; Manufacturer Murata -> Yageo
- R4126: renamed from R4129; value 1k 0.1% -> 13k 0.1%; MPN TNPW06031K00BEEA -> RC0603FR-0713KL; Manufacturer Vishay -> Yageo
- R4127: renamed from U424; value OPA1652AIDR -> 1k 0.1%; footprint Package_SO:SOIC-8_3.9x4.9mm_P1.27mm -> Resistor_SMD:R_0603_1608Metric; symbol CM5Carrier:OPA1652 -> Device:R; MPN OPA1652AIDR -> TNPW06031K00BEEA; Manufacturer Texas Instruments -> Vishay
- R4130: renamed from C4125; value 100nF -> 220R; footprint Capacitor_SMD:C_0402_1005Metric -> Resistor_SMD:R_0603_1608Metric; symbol Device:C -> Device:R; MPN C1005X7R1H104K050BB -> RC0603FR-07220RL; Manufacturer TDK -> Yageo
- R4150: renamed from C4151; value 470pF C0G -> 100R; footprint Capacitor_SMD:C_0603_1608Metric -> Resistor_SMD:R_0603_1608Metric; symbol Device:C -> Device:R; MPN GRM1885C1H471JA01D -> RC0603FR-07100RL; Manufacturer Murata -> Yageo
- R4151: renamed from C4152; value 100pF C0G -> 100R; footprint Capacitor_SMD:C_0603_1608Metric -> Resistor_SMD:R_0603_1608Metric; symbol Device:C -> Device:R; MPN GRM1885C1H101JA01D -> RC0603FR-07100RL; Manufacturer Murata -> Yageo
- R4156: renamed from R4159; value 1k 0.1% -> 13k 0.1%; MPN TNPW06031K00BEEA -> RC0603FR-0713KL; Manufacturer Vishay -> Yageo
- R4157: renamed from U425; value OPA1652AIDR -> 1k 0.1%; footprint Package_SO:SOIC-8_3.9x4.9mm_P1.27mm -> Resistor_SMD:R_0603_1608Metric; symbol CM5Carrier:OPA1652 -> Device:R; MPN OPA1652AIDR -> TNPW06031K00BEEA; Manufacturer Texas Instruments -> Vishay
- R4160: renamed from C4155; value 100nF -> 220R; footprint Capacitor_SMD:C_0402_1005Metric -> Resistor_SMD:R_0603_1608Metric; symbol Device:C -> Device:R; MPN C1005X7R1H104K050BB -> RC0603FR-07220RL; Manufacturer TDK -> Yageo
- R4180: renamed from C4181; value 470pF C0G -> 100R; footprint Capacitor_SMD:C_0603_1608Metric -> Resistor_SMD:R_0603_1608Metric; symbol Device:C -> Device:R; MPN GRM1885C1H471JA01D -> RC0603FR-07100RL; Manufacturer Murata -> Yageo
- R4181: renamed from C4182; value 100pF C0G -> 100R; footprint Capacitor_SMD:C_0603_1608Metric -> Resistor_SMD:R_0603_1608Metric; symbol Device:C -> Device:R; MPN GRM1885C1H101JA01D -> RC0603FR-07100RL; Manufacturer Murata -> Yageo
- R4186: renamed from R4189; value 1k 0.1% -> 13k 0.1%; MPN TNPW06031K00BEEA -> RC0603FR-0713KL; Manufacturer Vishay -> Yageo
- R4187: renamed from U426; value OPA1652AIDR -> 1k 0.1%; footprint Package_SO:SOIC-8_3.9x4.9mm_P1.27mm -> Resistor_SMD:R_0603_1608Metric; symbol CM5Carrier:OPA1652 -> Device:R; MPN OPA1652AIDR -> TNPW06031K00BEEA; Manufacturer Texas Instruments -> Vishay
- R4190: renamed from C4185; value 100nF -> 220R; footprint Capacitor_SMD:C_0402_1005Metric -> Resistor_SMD:R_0603_1608Metric; symbol Device:C -> Device:R; MPN C1005X7R1H104K050BB -> RC0603FR-07220RL; Manufacturer TDK -> Yageo
- R4210: renamed from C4211; value 470pF C0G -> 100R; footprint Capacitor_SMD:C_0603_1608Metric -> Resistor_SMD:R_0603_1608Metric; symbol Device:C -> Device:R; MPN GRM1885C1H471JA01D -> RC0603FR-07100RL; Manufacturer Murata -> Yageo
- R4211: renamed from C4212; value 100pF C0G -> 100R; footprint Capacitor_SMD:C_0603_1608Metric -> Resistor_SMD:R_0603_1608Metric; symbol Device:C -> Device:R; MPN GRM1885C1H101JA01D -> RC0603FR-07100RL; Manufacturer Murata -> Yageo
- R4216: renamed from R4219; value 1k 0.1% -> 13k 0.1%; MPN TNPW06031K00BEEA -> RC0603FR-0713KL; Manufacturer Vishay -> Yageo
- R4217: renamed from U427; value OPA1652AIDR -> 1k 0.1%; footprint Package_SO:SOIC-8_3.9x4.9mm_P1.27mm -> Resistor_SMD:R_0603_1608Metric; symbol CM5Carrier:OPA1652 -> Device:R; MPN OPA1652AIDR -> TNPW06031K00BEEA; Manufacturer Texas Instruments -> Vishay
- R4220: renamed from C4215; value 100nF -> 220R; footprint Capacitor_SMD:C_0402_1005Metric -> Resistor_SMD:R_0603_1608Metric; symbol Device:C -> Device:R; MPN C1005X7R1H104K050BB -> RC0603FR-07220RL; Manufacturer TDK -> Yageo
- R4240: renamed from C4241; value 470pF C0G -> 100R; footprint Capacitor_SMD:C_0603_1608Metric -> Resistor_SMD:R_0603_1608Metric; symbol Device:C -> Device:R; MPN GRM1885C1H471JA01D -> RC0603FR-07100RL; Manufacturer Murata -> Yageo
- R4241: renamed from C4242; value 100pF C0G -> 100R; footprint Capacitor_SMD:C_0603_1608Metric -> Resistor_SMD:R_0603_1608Metric; symbol Device:C -> Device:R; MPN GRM1885C1H101JA01D -> RC0603FR-07100RL; Manufacturer Murata -> Yageo
- R4246: renamed from R4249; value 1k 0.1% -> 13k 0.1%; MPN TNPW06031K00BEEA -> RC0603FR-0713KL; Manufacturer Vishay -> Yageo
- R4247: renamed from U428; value OPA1652AIDR -> 1k 0.1%; footprint Package_SO:SOIC-8_3.9x4.9mm_P1.27mm -> Resistor_SMD:R_0603_1608Metric; symbol CM5Carrier:OPA1652 -> Device:R; MPN OPA1652AIDR -> TNPW06031K00BEEA; Manufacturer Texas Instruments -> Vishay
- R4250: renamed from C4245; value 100nF -> 220R; footprint Capacitor_SMD:C_0402_1005Metric -> Resistor_SMD:R_0603_1608Metric; symbol Device:C -> Device:R; MPN C1005X7R1H104K050BB -> RC0603FR-07220RL; Manufacturer TDK -> Yageo
- U401: renamed from C4036; value 100nF -> THAT1206S08-U; footprint Capacitor_SMD:C_0402_1005Metric -> Package_SO:SOIC-8_3.9x4.9mm_P1.27mm; symbol Device:C -> CM5Carrier:THAT1206; MPN C1005X7R1H104K050BB -> THAT1206S08-U; Manufacturer TDK -> THAT Corporation
- U402: renamed from C4066; value 100nF -> THAT1206S08-U; footprint Capacitor_SMD:C_0402_1005Metric -> Package_SO:SOIC-8_3.9x4.9mm_P1.27mm; symbol Device:C -> CM5Carrier:THAT1206; MPN C1005X7R1H104K050BB -> THAT1206S08-U; Manufacturer TDK -> THAT Corporation
- U403: renamed from C4096; value 100nF -> THAT1206S08-U; footprint Capacitor_SMD:C_0402_1005Metric -> Package_SO:SOIC-8_3.9x4.9mm_P1.27mm; symbol Device:C -> CM5Carrier:THAT1206; MPN C1005X7R1H104K050BB -> THAT1206S08-U; Manufacturer TDK -> THAT Corporation
- U404: renamed from C4126; value 100nF -> THAT1206S08-U; footprint Capacitor_SMD:C_0402_1005Metric -> Package_SO:SOIC-8_3.9x4.9mm_P1.27mm; symbol Device:C -> CM5Carrier:THAT1206; MPN C1005X7R1H104K050BB -> THAT1206S08-U; Manufacturer TDK -> THAT Corporation
- U405: renamed from C4156; value 100nF -> THAT1206S08-U; footprint Capacitor_SMD:C_0402_1005Metric -> Package_SO:SOIC-8_3.9x4.9mm_P1.27mm; symbol Device:C -> CM5Carrier:THAT1206; MPN C1005X7R1H104K050BB -> THAT1206S08-U; Manufacturer TDK -> THAT Corporation
- U406: renamed from C4186; value 100nF -> THAT1206S08-U; footprint Capacitor_SMD:C_0402_1005Metric -> Package_SO:SOIC-8_3.9x4.9mm_P1.27mm; symbol Device:C -> CM5Carrier:THAT1206; MPN C1005X7R1H104K050BB -> THAT1206S08-U; Manufacturer TDK -> THAT Corporation
- U407: renamed from C4216; value 100nF -> THAT1206S08-U; footprint Capacitor_SMD:C_0402_1005Metric -> Package_SO:SOIC-8_3.9x4.9mm_P1.27mm; symbol Device:C -> CM5Carrier:THAT1206; MPN C1005X7R1H104K050BB -> THAT1206S08-U; Manufacturer TDK -> THAT Corporation
- U408: renamed from C4246; value 100nF -> THAT1206S08-U; footprint Capacitor_SMD:C_0402_1005Metric -> Package_SO:SOIC-8_3.9x4.9mm_P1.27mm; symbol Device:C -> CM5Carrier:THAT1206; MPN C1005X7R1H104K050BB -> THAT1206S08-U; Manufacturer TDK -> THAT Corporation
- U421: renamed from R4040; value 220R -> OPA1652AIDR; footprint Resistor_SMD:R_0603_1608Metric -> Package_SO:SOIC-8_3.9x4.9mm_P1.27mm; symbol Device:R -> CM5Carrier:OPA1652; MPN RC0603FR-07220RL -> OPA1652AIDR; Manufacturer Yageo -> Texas Instruments
- U422: renamed from R4070; value 220R -> OPA1652AIDR; footprint Resistor_SMD:R_0603_1608Metric -> Package_SO:SOIC-8_3.9x4.9mm_P1.27mm; symbol Device:R -> CM5Carrier:OPA1652; MPN RC0603FR-07220RL -> OPA1652AIDR; Manufacturer Yageo -> Texas Instruments
- U423: renamed from R4100; value 220R -> OPA1652AIDR; footprint Resistor_SMD:R_0603_1608Metric -> Package_SO:SOIC-8_3.9x4.9mm_P1.27mm; symbol Device:R -> CM5Carrier:OPA1652; MPN RC0603FR-07220RL -> OPA1652AIDR; Manufacturer Yageo -> Texas Instruments
- U424: renamed from R4130; value 220R -> OPA1652AIDR; footprint Resistor_SMD:R_0603_1608Metric -> Package_SO:SOIC-8_3.9x4.9mm_P1.27mm; symbol Device:R -> CM5Carrier:OPA1652; MPN RC0603FR-07220RL -> OPA1652AIDR; Manufacturer Yageo -> Texas Instruments
- U425: renamed from R4160; value 220R -> OPA1652AIDR; footprint Resistor_SMD:R_0603_1608Metric -> Package_SO:SOIC-8_3.9x4.9mm_P1.27mm; symbol Device:R -> CM5Carrier:OPA1652; MPN RC0603FR-07220RL -> OPA1652AIDR; Manufacturer Yageo -> Texas Instruments
- U426: renamed from R4190; value 220R -> OPA1652AIDR; footprint Resistor_SMD:R_0603_1608Metric -> Package_SO:SOIC-8_3.9x4.9mm_P1.27mm; symbol Device:R -> CM5Carrier:OPA1652; MPN RC0603FR-07220RL -> OPA1652AIDR; Manufacturer Yageo -> Texas Instruments
- U427: renamed from R4220; value 220R -> OPA1652AIDR; footprint Resistor_SMD:R_0603_1608Metric -> Package_SO:SOIC-8_3.9x4.9mm_P1.27mm; symbol Device:R -> CM5Carrier:OPA1652; MPN RC0603FR-07220RL -> OPA1652AIDR; Manufacturer Yageo -> Texas Instruments
- U428: renamed from R4250; value 220R -> OPA1652AIDR; footprint Resistor_SMD:R_0603_1608Metric -> Package_SO:SOIC-8_3.9x4.9mm_P1.27mm; symbol Device:R -> CM5Carrier:OPA1652; MPN RC0603FR-07220RL -> OPA1652AIDR; Manufacturer Yageo -> Texas Instruments
- renumbered D4033 to D4030, D4063 to D4060, D4093 to D4090, D4123 to D4120, D4153 to D4150, D4183 to D4180, D4213 to D4210, D4243 to D4240
Connections:
- net ADC_5V_A: now also C4035.1, C4065.1, C4095.1, C4125.1, C4155.1, C4185.1, C4215.1, U421.8 (V+), U422.8 (V+), U423.8 (V+), U424.8 (V+), U425.8 (V+)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; no longer R4037.8 (V+), R4040.1, R4067.8 (V+), R4070.1, R4097.8 (V+), R4100.1, R4127.8 (V+), R4130.1, R4157.8 (V+), R4160.1, R4187.8 (V+), R4190.1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
- net ADC_CH1N: now also C4034.2
- net ADC_CH1N_RAW: now also U421.7 (OUT_B), R4039.1; no longer R4036.1, R4037.7 (OUT_B)
- net ADC_CH1P: now also C4034.1, R4040.2; no longer U421.2
- net ADC_CH1P_RAW: now also R4040.1, U421.2 (IN_A-); no longer R4037.1 (OUT_A), R4037.2 (IN_A-)
- net ADC_CH2N: now also C4064.2
- net ADC_CH2N_RAW: now also U422.7 (OUT_B), R4069.1; no longer R4066.1, R4067.7 (OUT_B)
- net ADC_CH2P: now also C4064.1, R4070.2; no longer U422.2
- net ADC_CH2P_RAW: now also R4070.1, U422.2 (IN_A-); no longer R4067.1 (OUT_A), R4067.2 (IN_A-)
- net ADC_CH3N: now also C4094.2
- net ADC_CH3N_RAW: now also U423.7 (OUT_B), R4099.1; no longer R4096.1, R4097.7 (OUT_B)
- net ADC_CH3P: now also C4094.1, R4100.2; no longer U423.2
- net ADC_CH3P_RAW: now also R4100.1, U423.2 (IN_A-); no longer R4097.1 (OUT_A), R4097.2 (IN_A-)
- net ADC_CH4N: now also C4124.2
- net ADC_CH4N_RAW: now also U424.7 (OUT_B), R4129.1; no longer R4126.1, R4127.7 (OUT_B)
- net ADC_CH4P: now also C4124.1, R4130.2; no longer U424.2
- net ADC_CH4P_RAW: now also R4130.1, U424.2 (IN_A-); no longer R4127.1 (OUT_A), R4127.2 (IN_A-)
- net ADC_CH5N: now also C4154.2
- net ADC_CH5N_RAW: now also U425.7 (OUT_B), R4159.1; no longer R4156.1, R4157.7 (OUT_B)
- net ADC_CH5P: now also C4154.1, R4160.2; no longer U425.2
- net ADC_CH5P_RAW: now also R4160.1, U425.2 (IN_A-); no longer R4157.1 (OUT_A), R4157.2 (IN_A-)
- net ADC_CH6N: now also C4184.2
- net ADC_CH6N_RAW: now also U426.7 (OUT_B), R4189.1; no longer R4186.1, R4187.7 (OUT_B)
- net ADC_CH6P: now also C4184.1, R4190.2; no longer U426.2
- net ADC_CH6P_RAW: now also R4190.1, U426.2 (IN_A-); no longer R4187.1 (OUT_A), R4187.2 (IN_A-)
- net ADC_CH7N: now also C4214.2
- net ADC_CH7N_RAW: now also U427.7 (OUT_B), R4219.1; no longer R4216.1, R4217.7 (OUT_B)
- net ADC_CH7P: now also C4214.1, R4220.2; no longer U427.2
- net ADC_CH7P_RAW: now also R4220.1, U427.2 (IN_A-); no longer R4217.1 (OUT_A), R4217.2 (IN_A-)
- net ADC_CH8N_RAW: now also U428.7 (OUT_B), R4249.1; no longer R4246.1, R4247.7 (OUT_B)
- net ADC_CH8P: now also R4250.2; no longer U428.2
- net ADC_CH8P_RAW: now also R4250.1, U428.2 (IN_A-); no longer R4247.1 (OUT_A), R4247.2 (IN_A-)
- net AGND: now also C4035.2, C4036.2, C4037.2, C4065.2, C4066.2, C4067.2, C4095.2, C4096.2, C4097.2, C4125.2, C4126.2, C4127.2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; no longer D4031.2 (A), D4032.2 (A), D4033.1 (REF), D4033.5 (CM_IN), D4061.2 (A), D4062.2 (A), D4063.1 (REF), D4063.5 (CM_IN), D4091.2 (A), D4092.2 (A), D4093.1 (REF), D4093.5 (CM_IN)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
- net AIN1_AC: now also C4033.2, R4036.1, R4038.1; no longer C4033.1, C4036.1
- net AIN1_DIVP: now also R4036.2, R4037.1, U421.3 (IN_A+); no longer C4036.2, C4037.1, R4037.3 (IN_A+)
- net AIN1_INVN: now also U421.6 (IN_B-), R4038.2, R4039.2; no longer C4033.2, R4036.2, R4037.6 (IN_B-)
- net AIN1_PROT_N: now also C4031.1, C4032.2, U401.2 (IN-), D4035.1 (K); no longer C4032.1 (K), D4030.2 (A), R4030.1
- net AIN1_PROT_P: now also C4032.1, D4030.1 (K), D4031.2 (A), R4030.2, U401.3 (IN+), D4034.1 (K); no longer C4031.2 (A), D4031.1 (K), D4033.3 (IN+), R4031.1
- net AIN1_RX_SE: now also C4033.1, U401.6 (VOUT); no longer D4033.6 (VOUT)
- net AIN2_AC: now also C4063.2, R4066.1, R4068.1; no longer C4063.1, C4066.1
- net AIN2_DIVP: now also R4066.2, R4067.1, U422.3 (IN_A+); no longer C4066.2, C4067.1, R4067.3 (IN_A+)
- net AIN2_INVN: now also U422.6 (IN_B-), R4068.2, R4069.2; no longer C4063.2, R4066.2, R4067.6 (IN_B-)
- net AIN2_PROT_N: now also C4061.1, C4062.2, U402.2 (IN-), D4065.1 (K); no longer C4035.2, C4062.1 (K), D4060.2 (A), R4060.1
- net AIN2_PROT_P: now also C4062.1, D4060.1 (K), D4061.2 (A), R4060.2, U402.3 (IN+), D4064.1 (K); no longer C4034.2, C4061.2 (A), D4061.1 (K), D4063.3 (IN+), R4061.1
- net AIN2_RX_SE: now also C4063.1, U402.6 (VOUT); no longer D4063.6 (VOUT)
- net AIN3_AC: now also C4093.2, R4096.1, R4098.1; no longer C4093.1, C4096.1
- net AIN3_DIVP: now also R4096.2, R4097.1, U423.3 (IN_A+); no longer C4096.2, C4097.1, R4097.3 (IN_A+)
- net AIN3_INVN: now also U423.6 (IN_B-), R4098.2, R4099.2; no longer C4093.2, R4096.2, R4097.6 (IN_B-)
- net AIN3_PROT_N: now also C4091.1, C4092.2, U403.2 (IN-), D4095.1 (K); no longer C4065.2, C4092.1 (K), D4090.2 (A), R4090.1
- net AIN3_PROT_P: now also C4092.1, D4090.1 (K), D4091.2 (A), R4090.2, U403.3 (IN+), D4094.1 (K); no longer C4064.2, C4091.2 (A), D4091.1 (K), D4093.3 (IN+), R4091.1
- net AIN3_RX_SE: now also C4093.1, U403.6 (VOUT); no longer D4093.6 (VOUT)
- net AIN4_AC: now also C4123.2, R4126.1, R4128.1; no longer C4123.1, C4126.1
- net AIN4_DIVP: now also R4126.2, R4127.1, U424.3 (IN_A+); no longer C4126.2, C4127.1, R4127.3 (IN_A+)
- net AIN4_INVN: now also U424.6 (IN_B-), R4128.2, R4129.2; no longer C4123.2, R4126.2, R4127.6 (IN_B-)
- net AIN4_PROT_N: now also C4121.1, C4122.2, U404.2 (IN-), D4125.1 (K); no longer C4095.2, C4122.1 (K), D4120.2 (A), R4120.1
- net AIN4_PROT_P: now also C4122.1, D4120.1 (K), D4121.2 (A), R4120.2, U404.3 (IN+), D4124.1 (K); no longer C4094.2, C4121.2 (A), D4121.1 (K), D4123.3 (IN+), R4121.1
- net AIN4_RX_SE: now also C4123.1, U404.6 (VOUT); no longer D4123.6 (VOUT)
- net AIN5_AC: now also C4153.2, R4156.1, R4158.1; no longer C4153.1, C4156.1
- net AIN5_DIVP: now also R4156.2, R4157.1, U425.3 (IN_A+); no longer C4156.2, C4157.1, R4157.3 (IN_A+)
- net AIN5_INVN: now also U425.6 (IN_B-), R4158.2, R4159.2; no longer C4153.2, R4156.2, R4157.6 (IN_B-)
- net AIN5_PROT_N: now also C4151.1, C4152.2, U405.2 (IN-), D4155.1 (K); no longer C4125.2, C4152.1 (K), D4150.2 (A), R4150.1
- net AIN5_PROT_P: now also C4152.1, D4150.1 (K), D4151.2 (A), R4150.2, U405.3 (IN+), D4154.1 (K); no longer C4124.2, C4151.2 (A), D4151.1 (K), D4153.3 (IN+), R4151.1
- net AIN5_RX_SE: now also C4153.1, U405.6 (VOUT); no longer D4153.6 (VOUT)
- net AIN6_AC: now also C4183.2, R4186.1, R4188.1; no longer C4183.1, C4186.1
- net AIN6_DIVP: now also R4186.2, R4187.1, U426.3 (IN_A+); no longer C4186.2, C4187.1, R4187.3 (IN_A+)
- net AIN6_INVN: now also U426.6 (IN_B-), R4188.2, R4189.2; no longer C4183.2, R4186.2, R4187.6 (IN_B-)
- net AIN6_PROT_N: now also C4181.1, C4182.2, U406.2 (IN-), D4185.1 (K); no longer C4155.2, C4182.1 (K), D4180.2 (A), R4180.1
- net AIN6_PROT_P: now also C4182.1, D4180.1 (K), D4181.2 (A), R4180.2, U406.3 (IN+), D4184.1 (K); no longer C4154.2, C4181.2 (A), D4181.1 (K), D4183.3 (IN+), R4181.1
- net AIN6_RX_SE: now also C4183.1, U406.6 (VOUT); no longer D4183.6 (VOUT)
- net AIN7_AC: now also C4213.2, R4216.1, R4218.1; no longer C4213.1, C4216.1
- net AIN7_DIVP: now also R4216.2, R4217.1, U427.3 (IN_A+); no longer C4216.2, C4217.1, R4217.3 (IN_A+)
- net AIN7_INVN: now also U427.6 (IN_B-), R4218.2, R4219.2; no longer C4213.2, R4216.2, R4217.6 (IN_B-)
- net AIN7_PROT_N: now also C4211.1, C4212.2, U407.2 (IN-), D4215.1 (K); no longer C4185.2, C4212.1 (K), D4210.2 (A), R4210.1
- net AIN7_PROT_P: now also C4212.1, D4210.1 (K), D4211.2 (A), R4210.2, U407.3 (IN+), D4214.1 (K); no longer C4184.2, C4211.2 (A), D4211.1 (K), D4213.3 (IN+), R4211.1
- net AIN7_RX_SE: now also C4213.1, U407.6 (VOUT); no longer D4213.6 (VOUT)
- net AIN8_AC: now also C4243.2, R4246.1, R4248.1; no longer C4243.1, C4246.1
- net AIN8_DIVP: now also R4246.2, R4247.1, U428.3 (IN_A+); no longer C4246.2, C4247.1, R4247.3 (IN_A+)
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Other:
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