File: cad/kicad/AUDIO-8X8/Audio-Outputs.kicad_sch (KiCad schematic)
At the start: 200 parts, among them K501 TQ2-12V, K502 TQ2-12V, K503 TQ2-12V, K504 TQ2-12V, K505 TQ2-12V, K506 TQ2-12V, K507 TQ2-12V, K508 TQ2-12V, Q501 2N7002K, Q502 2N7002K, Q503 2N7002K, Q504 2N7002K, Q505 2N7002K, Q506 2N7002K, Q507 2N7002K, Q508 2N7002K, U501 OPA1652AIDR, U502 OPA1652AIDR, U503 OPA1652AIDR, U504 OPA1652AIDR, U505 OPA1652AIDR, U506 OPA1652AIDR, U507 OPA1652AIDR, U508 OPA1652AIDR, U521 THAT1646S08-U, U522 THAT1646S08-U, U523 THAT1646S08-U, U524 THAT1646S08-U, U525 THAT1646S08-U, U526 THAT1646S08-U, U527 THAT1646S08-U, U528 THAT1646S08-U

Commit message: Audit schematic logic against controlled datasheets
Parts:
- added C5047, C5048, C5049, C5050, C5087, C5088, C5089, C5090, C5127, C5128, C5129, C5130, C5167, C5168, C5169, C5170, C5207, C5208, C5209, C5210, C5247, C5248, C5249, C5250, C5287, C5288, C5289, C5290, C5327, C5328, C5329, C5330: 100nF, Capacitor_SMD:C_0402_1005Metric, symbol Device:C
Connections:
- net AGND: now also C5047.2, C5048.2, C5049.2, C5050.2, C5087.2, C5088.2, C5089.2, C5090.2, C5127.2, C5128.2, C5129.2, C5130.2, C5167.2, C5168.2, C5169.2, C5170.2, C5207.2, C5208.2, C5209.2, C5210.2, C5247.2, C5248.2, C5249.2, C5250.2, C5287.2, C5288.2, C5289.2, C5290.2, C5327.2, C5328.2, C5329.2, C5330.2
- net AUDIO_N15V: now also C5048.1, C5050.1, C5088.1, C5090.1, C5128.1, C5130.1, C5168.1, C5170.1, C5208.1, C5210.1, C5248.1, C5250.1, C5288.1, C5290.1, C5328.1, C5330.1
- net AUDIO_P15V: now also C5047.1, C5049.1, C5087.1, C5089.1, C5127.1, C5129.1, C5167.1, C5169.1, C5207.1, C5209.1, C5247.1, C5249.1, C5287.1, C5289.1, C5327.1, C5329.1
- net AUDIO_OUTPUT_RELAY_EN renamed AUDIO_SAFE_UNMUTE_N
Other:
- note added: "AUDIO_SAFE_UNMUTE_N is generated locally from carrier mute command AND ADC/DAC power-good; loss of any condition drops every relay."

Commit message: Implement direct socketed dual-SIM daughterboard
Parts:
- removed C5042, C5082, C5122, C5162, C5202, C5242, C5282, C5322: 3.9nF C0G, Capacitor_SMD:C_0603_1608Metric, symbol Device:C
- removed C5048, C5049, C5088, C5089, C5128, C5129, C5168, C5169, C5208, C5209, C5248, C5249, C5288, C5289, C5328, C5329: 100nF, Capacitor_SMD:C_0402_1005Metric, symbol Device:C
- removed D5040, D5080, D5120, D5160, D5200, D5240, D5280, D5320: 1N4148W, Diode_SMD:D_SOD-123, symbol Device:D
- removed L5040, L5041, L5080, L5081, L5120, L5121, L5160, L5161, L5200, L5201, L5240, L5241, L5280, L5281, L5320, L5321: 220R ferrite, Inductor_SMD:L_0805_2012Metric, symbol Device:FerriteBead
- removed R5040, R5041, R5080, R5081, R5120, R5121, R5160, R5161, R5200, R5201, R5240, R5241, R5280, R5281, R5320, R5321: 3.9k 0.1%, Resistor_SMD:R_0603_1608Metric, symbol Device:R
- removed R5042, R5082, R5122, R5162, R5202, R5242, R5282, R5322: 4.7k 0.1%, Resistor_SMD:R_0603_1608Metric, symbol Device:R
- added C5040, C5041, C5080, C5081, C5120, C5121, C5160, C5161, C5200, C5201, C5240, C5241, C5280, C5281, C5320, C5321: 470pF C0G, Capacitor_SMD:C_0603_1608Metric, symbol Device:C
- added C5043, C5044, C5083, C5084, C5123, C5124, C5163, C5164, C5203, C5204, C5243, C5244, C5283, C5284, C5323, C5324: 10uF bipolar, Capacitor_THT:CP_Radial_D5.0mm_P2.00mm, symbol Device:C
- added D5042, D5043, D5044, D5082, D5083, D5084, D5122, D5123, D5124, D5162, D5163, D5164, D5202, D5203, D5204, D5242, D5243, D5244, D5282, D5283, D5284, D5322, D5323, D5324: S1G, Diode_SMD:D_SMA, symbol Device:D
- added Q501, Q502, Q503, Q504, Q505, Q506, Q507, Q508: 2N7002K, Package_TO_SOT_SMD:SOT-23, symbol Transistor_FET:2N7002
- added R5046, R5086, R5126, R5166, R5206, R5246, R5286, R5326: 10k 0.1%, Resistor_SMD:R_0603_1608Metric, symbol Device:R
- C5042: renamed from U521; value THAT1646S08-U -> 3.9nF C0G; footprint Package_SO:SOIC-8_3.9x4.9mm_P1.27mm -> Capacitor_SMD:C_0603_1608Metric; symbol CM5Carrier:THAT1646 -> Device:C; MPN THAT1646S08-U -> GRM1885C1H392JA01D; Manufacturer THAT Corporation -> Murata
- C5045: renamed from D5042; value S1G -> 100pF C0G; footprint Diode_SMD:D_SMA -> Capacitor_SMD:C_0603_1608Metric; symbol Device:D -> Device:C; MPN S1G-13-F -> GRM1885C1H101JA01D; Manufacturer Diodes Incorporated -> Murata
- C5046: renamed from D5043; value S1G -> 100pF C0G; footprint Diode_SMD:D_SMA -> Capacitor_SMD:C_0603_1608Metric; symbol Device:D -> Device:C; MPN S1G-13-F -> GRM1885C1H101JA01D; Manufacturer Diodes Incorporated -> Murata
- C5048: renamed from C5043; value 10uF bipolar -> 100nF; footprint Capacitor_THT:CP_Radial_D5.0mm_P2.00mm -> Capacitor_SMD:C_0402_1005Metric; MPN UES1H100MDM1TD -> C1005X7R1H104K050BB; Manufacturer Nichicon -> TDK
- C5049: renamed from C5044; value 10uF bipolar -> 100nF; footprint Capacitor_THT:CP_Radial_D5.0mm_P2.00mm -> Capacitor_SMD:C_0402_1005Metric; MPN UES1H100MDM1TD -> C1005X7R1H104K050BB; Manufacturer Nichicon -> TDK
- C5050: renamed from K501; value TQ2-12V -> 100nF; footprint CM5Carrier:Panasonic_TQ2-12V_PRELIMINARY -> Capacitor_SMD:C_0402_1005Metric; symbol CM5Carrier:Panasonic_TQ2_12V -> Device:C; MPN TQ2-12V -> C1005X7R1H104K050BB; Manufacturer Panasonic Industry -> TDK
- C5082: renamed from U522; value THAT1646S08-U -> 3.9nF C0G; footprint Package_SO:SOIC-8_3.9x4.9mm_P1.27mm -> Capacitor_SMD:C_0603_1608Metric; symbol CM5Carrier:THAT1646 -> Device:C; MPN THAT1646S08-U -> GRM1885C1H392JA01D; Manufacturer THAT Corporation -> Murata
- C5085: renamed from D5082; value S1G -> 100pF C0G; footprint Diode_SMD:D_SMA -> Capacitor_SMD:C_0603_1608Metric; symbol Device:D -> Device:C; MPN S1G-13-F -> GRM1885C1H101JA01D; Manufacturer Diodes Incorporated -> Murata
- C5086: renamed from D5083; value S1G -> 100pF C0G; footprint Diode_SMD:D_SMA -> Capacitor_SMD:C_0603_1608Metric; symbol Device:D -> Device:C; MPN S1G-13-F -> GRM1885C1H101JA01D; Manufacturer Diodes Incorporated -> Murata
- C5088: renamed from C5083; value 10uF bipolar -> 100nF; footprint Capacitor_THT:CP_Radial_D5.0mm_P2.00mm -> Capacitor_SMD:C_0402_1005Metric; MPN UES1H100MDM1TD -> C1005X7R1H104K050BB; Manufacturer Nichicon -> TDK
- C5089: renamed from C5084; value 10uF bipolar -> 100nF; footprint Capacitor_THT:CP_Radial_D5.0mm_P2.00mm -> Capacitor_SMD:C_0402_1005Metric; MPN UES1H100MDM1TD -> C1005X7R1H104K050BB; Manufacturer Nichicon -> TDK
- C5090: renamed from K502; value TQ2-12V -> 100nF; footprint CM5Carrier:Panasonic_TQ2-12V_PRELIMINARY -> Capacitor_SMD:C_0402_1005Metric; symbol CM5Carrier:Panasonic_TQ2_12V -> Device:C; MPN TQ2-12V -> C1005X7R1H104K050BB; Manufacturer Panasonic Industry -> TDK
- C5122: renamed from U523; value THAT1646S08-U -> 3.9nF C0G; footprint Package_SO:SOIC-8_3.9x4.9mm_P1.27mm -> Capacitor_SMD:C_0603_1608Metric; symbol CM5Carrier:THAT1646 -> Device:C; MPN THAT1646S08-U -> GRM1885C1H392JA01D; Manufacturer THAT Corporation -> Murata
- C5125: renamed from D5122; value S1G -> 100pF C0G; footprint Diode_SMD:D_SMA -> Capacitor_SMD:C_0603_1608Metric; symbol Device:D -> Device:C; MPN S1G-13-F -> GRM1885C1H101JA01D; Manufacturer Diodes Incorporated -> Murata
- C5126: renamed from D5123; value S1G -> 100pF C0G; footprint Diode_SMD:D_SMA -> Capacitor_SMD:C_0603_1608Metric; symbol Device:D -> Device:C; MPN S1G-13-F -> GRM1885C1H101JA01D; Manufacturer Diodes Incorporated -> Murata
- C5128: renamed from C5123; value 10uF bipolar -> 100nF; footprint Capacitor_THT:CP_Radial_D5.0mm_P2.00mm -> Capacitor_SMD:C_0402_1005Metric; MPN UES1H100MDM1TD -> C1005X7R1H104K050BB; Manufacturer Nichicon -> TDK
- C5129: renamed from C5124; value 10uF bipolar -> 100nF; footprint Capacitor_THT:CP_Radial_D5.0mm_P2.00mm -> Capacitor_SMD:C_0402_1005Metric; MPN UES1H100MDM1TD -> C1005X7R1H104K050BB; Manufacturer Nichicon -> TDK
- C5130: renamed from K503; value TQ2-12V -> 100nF; footprint CM5Carrier:Panasonic_TQ2-12V_PRELIMINARY -> Capacitor_SMD:C_0402_1005Metric; symbol CM5Carrier:Panasonic_TQ2_12V -> Device:C; MPN TQ2-12V -> C1005X7R1H104K050BB; Manufacturer Panasonic Industry -> TDK
- C5162: renamed from U524; value THAT1646S08-U -> 3.9nF C0G; footprint Package_SO:SOIC-8_3.9x4.9mm_P1.27mm -> Capacitor_SMD:C_0603_1608Metric; symbol CM5Carrier:THAT1646 -> Device:C; MPN THAT1646S08-U -> GRM1885C1H392JA01D; Manufacturer THAT Corporation -> Murata
- C5165: renamed from D5162; value S1G -> 100pF C0G; footprint Diode_SMD:D_SMA -> Capacitor_SMD:C_0603_1608Metric; symbol Device:D -> Device:C; MPN S1G-13-F -> GRM1885C1H101JA01D; Manufacturer Diodes Incorporated -> Murata
- C5166: renamed from D5163; value S1G -> 100pF C0G; footprint Diode_SMD:D_SMA -> Capacitor_SMD:C_0603_1608Metric; symbol Device:D -> Device:C; MPN S1G-13-F -> GRM1885C1H101JA01D; Manufacturer Diodes Incorporated -> Murata
- C5168: renamed from C5163; value 10uF bipolar -> 100nF; footprint Capacitor_THT:CP_Radial_D5.0mm_P2.00mm -> Capacitor_SMD:C_0402_1005Metric; MPN UES1H100MDM1TD -> C1005X7R1H104K050BB; Manufacturer Nichicon -> TDK
- C5169: renamed from C5164; value 10uF bipolar -> 100nF; footprint Capacitor_THT:CP_Radial_D5.0mm_P2.00mm -> Capacitor_SMD:C_0402_1005Metric; MPN UES1H100MDM1TD -> C1005X7R1H104K050BB; Manufacturer Nichicon -> TDK
- C5170: renamed from K504; value TQ2-12V -> 100nF; footprint CM5Carrier:Panasonic_TQ2-12V_PRELIMINARY -> Capacitor_SMD:C_0402_1005Metric; symbol CM5Carrier:Panasonic_TQ2_12V -> Device:C; MPN TQ2-12V -> C1005X7R1H104K050BB; Manufacturer Panasonic Industry -> TDK
- C5202: renamed from U525; value THAT1646S08-U -> 3.9nF C0G; footprint Package_SO:SOIC-8_3.9x4.9mm_P1.27mm -> Capacitor_SMD:C_0603_1608Metric; symbol CM5Carrier:THAT1646 -> Device:C; MPN THAT1646S08-U -> GRM1885C1H392JA01D; Manufacturer THAT Corporation -> Murata
- C5205: renamed from D5202; value S1G -> 100pF C0G; footprint Diode_SMD:D_SMA -> Capacitor_SMD:C_0603_1608Metric; symbol Device:D -> Device:C; MPN S1G-13-F -> GRM1885C1H101JA01D; Manufacturer Diodes Incorporated -> Murata
- C5206: renamed from D5203; value S1G -> 100pF C0G; footprint Diode_SMD:D_SMA -> Capacitor_SMD:C_0603_1608Metric; symbol Device:D -> Device:C; MPN S1G-13-F -> GRM1885C1H101JA01D; Manufacturer Diodes Incorporated -> Murata
- C5208: renamed from C5203; value 10uF bipolar -> 100nF; footprint Capacitor_THT:CP_Radial_D5.0mm_P2.00mm -> Capacitor_SMD:C_0402_1005Metric; MPN UES1H100MDM1TD -> C1005X7R1H104K050BB; Manufacturer Nichicon -> TDK
- C5209: renamed from C5204; value 10uF bipolar -> 100nF; footprint Capacitor_THT:CP_Radial_D5.0mm_P2.00mm -> Capacitor_SMD:C_0402_1005Metric; MPN UES1H100MDM1TD -> C1005X7R1H104K050BB; Manufacturer Nichicon -> TDK
- C5210: renamed from K505; value TQ2-12V -> 100nF; footprint CM5Carrier:Panasonic_TQ2-12V_PRELIMINARY -> Capacitor_SMD:C_0402_1005Metric; symbol CM5Carrier:Panasonic_TQ2_12V -> Device:C; MPN TQ2-12V -> C1005X7R1H104K050BB; Manufacturer Panasonic Industry -> TDK
- C5242: renamed from U526; value THAT1646S08-U -> 3.9nF C0G; footprint Package_SO:SOIC-8_3.9x4.9mm_P1.27mm -> Capacitor_SMD:C_0603_1608Metric; symbol CM5Carrier:THAT1646 -> Device:C; MPN THAT1646S08-U -> GRM1885C1H392JA01D; Manufacturer THAT Corporation -> Murata
- C5245: renamed from D5242; value S1G -> 100pF C0G; footprint Diode_SMD:D_SMA -> Capacitor_SMD:C_0603_1608Metric; symbol Device:D -> Device:C; MPN S1G-13-F -> GRM1885C1H101JA01D; Manufacturer Diodes Incorporated -> Murata
- C5246: renamed from D5243; value S1G -> 100pF C0G; footprint Diode_SMD:D_SMA -> Capacitor_SMD:C_0603_1608Metric; symbol Device:D -> Device:C; MPN S1G-13-F -> GRM1885C1H101JA01D; Manufacturer Diodes Incorporated -> Murata
- C5248: renamed from C5243; value 10uF bipolar -> 100nF; footprint Capacitor_THT:CP_Radial_D5.0mm_P2.00mm -> Capacitor_SMD:C_0402_1005Metric; MPN UES1H100MDM1TD -> C1005X7R1H104K050BB; Manufacturer Nichicon -> TDK
- C5249: renamed from C5244; value 10uF bipolar -> 100nF; footprint Capacitor_THT:CP_Radial_D5.0mm_P2.00mm -> Capacitor_SMD:C_0402_1005Metric; MPN UES1H100MDM1TD -> C1005X7R1H104K050BB; Manufacturer Nichicon -> TDK
- C5250: renamed from K506; value TQ2-12V -> 100nF; footprint CM5Carrier:Panasonic_TQ2-12V_PRELIMINARY -> Capacitor_SMD:C_0402_1005Metric; symbol CM5Carrier:Panasonic_TQ2_12V -> Device:C; MPN TQ2-12V -> C1005X7R1H104K050BB; Manufacturer Panasonic Industry -> TDK
- C5282: renamed from U527; value THAT1646S08-U -> 3.9nF C0G; footprint Package_SO:SOIC-8_3.9x4.9mm_P1.27mm -> Capacitor_SMD:C_0603_1608Metric; symbol CM5Carrier:THAT1646 -> Device:C; MPN THAT1646S08-U -> GRM1885C1H392JA01D; Manufacturer THAT Corporation -> Murata
- C5285: renamed from D5282; value S1G -> 100pF C0G; footprint Diode_SMD:D_SMA -> Capacitor_SMD:C_0603_1608Metric; symbol Device:D -> Device:C; MPN S1G-13-F -> GRM1885C1H101JA01D; Manufacturer Diodes Incorporated -> Murata
- C5286: renamed from D5283; value S1G -> 100pF C0G; footprint Diode_SMD:D_SMA -> Capacitor_SMD:C_0603_1608Metric; symbol Device:D -> Device:C; MPN S1G-13-F -> GRM1885C1H101JA01D; Manufacturer Diodes Incorporated -> Murata
- C5288: renamed from C5283; value 10uF bipolar -> 100nF; footprint Capacitor_THT:CP_Radial_D5.0mm_P2.00mm -> Capacitor_SMD:C_0402_1005Metric; MPN UES1H100MDM1TD -> C1005X7R1H104K050BB; Manufacturer Nichicon -> TDK
- C5289: renamed from C5284; value 10uF bipolar -> 100nF; footprint Capacitor_THT:CP_Radial_D5.0mm_P2.00mm -> Capacitor_SMD:C_0402_1005Metric; MPN UES1H100MDM1TD -> C1005X7R1H104K050BB; Manufacturer Nichicon -> TDK
- C5290: renamed from K507; value TQ2-12V -> 100nF; footprint CM5Carrier:Panasonic_TQ2-12V_PRELIMINARY -> Capacitor_SMD:C_0402_1005Metric; symbol CM5Carrier:Panasonic_TQ2_12V -> Device:C; MPN TQ2-12V -> C1005X7R1H104K050BB; Manufacturer Panasonic Industry -> TDK
- C5322: renamed from U528; value THAT1646S08-U -> 3.9nF C0G; footprint Package_SO:SOIC-8_3.9x4.9mm_P1.27mm -> Capacitor_SMD:C_0603_1608Metric; symbol CM5Carrier:THAT1646 -> Device:C; MPN THAT1646S08-U -> GRM1885C1H392JA01D; Manufacturer THAT Corporation -> Murata
- C5325: renamed from D5322; value S1G -> 100pF C0G; footprint Diode_SMD:D_SMA -> Capacitor_SMD:C_0603_1608Metric; symbol Device:D -> Device:C; MPN S1G-13-F -> GRM1885C1H101JA01D; Manufacturer Diodes Incorporated -> Murata
- C5326: renamed from D5323; value S1G -> 100pF C0G; footprint Diode_SMD:D_SMA -> Capacitor_SMD:C_0603_1608Metric; symbol Device:D -> Device:C; MPN S1G-13-F -> GRM1885C1H101JA01D; Manufacturer Diodes Incorporated -> Murata
- C5328: renamed from C5323; value 10uF bipolar -> 100nF; footprint Capacitor_THT:CP_Radial_D5.0mm_P2.00mm -> Capacitor_SMD:C_0402_1005Metric; MPN UES1H100MDM1TD -> C1005X7R1H104K050BB; Manufacturer Nichicon -> TDK
- C5329: renamed from C5324; value 10uF bipolar -> 100nF; footprint Capacitor_THT:CP_Radial_D5.0mm_P2.00mm -> Capacitor_SMD:C_0402_1005Metric; MPN UES1H100MDM1TD -> C1005X7R1H104K050BB; Manufacturer Nichicon -> TDK
- C5330: renamed from K508; value TQ2-12V -> 100nF; footprint CM5Carrier:Panasonic_TQ2-12V_PRELIMINARY -> Capacitor_SMD:C_0402_1005Metric; symbol CM5Carrier:Panasonic_TQ2_12V -> Device:C; MPN TQ2-12V -> C1005X7R1H104K050BB; Manufacturer Panasonic Industry -> TDK
- D5040: renamed from C5045; value 100pF C0G -> 1N4148W; footprint Capacitor_SMD:C_0603_1608Metric -> Diode_SMD:D_SOD-123; symbol Device:C -> Device:D; MPN GRM1885C1H101JA01D -> 1N4148W-7-F; Manufacturer Murata -> Diodes Incorporated
- D5080: renamed from C5085; value 100pF C0G -> 1N4148W; footprint Capacitor_SMD:C_0603_1608Metric -> Diode_SMD:D_SOD-123; symbol Device:C -> Device:D; MPN GRM1885C1H101JA01D -> 1N4148W-7-F; Manufacturer Murata -> Diodes Incorporated
- D5120: renamed from C5125; value 100pF C0G -> 1N4148W; footprint Capacitor_SMD:C_0603_1608Metric -> Diode_SMD:D_SOD-123; symbol Device:C -> Device:D; MPN GRM1885C1H101JA01D -> 1N4148W-7-F; Manufacturer Murata -> Diodes Incorporated
- D5160: renamed from C5165; value 100pF C0G -> 1N4148W; footprint Capacitor_SMD:C_0603_1608Metric -> Diode_SMD:D_SOD-123; symbol Device:C -> Device:D; MPN GRM1885C1H101JA01D -> 1N4148W-7-F; Manufacturer Murata -> Diodes Incorporated
- D5200: renamed from C5205; value 100pF C0G -> 1N4148W; footprint Capacitor_SMD:C_0603_1608Metric -> Diode_SMD:D_SOD-123; symbol Device:C -> Device:D; MPN GRM1885C1H101JA01D -> 1N4148W-7-F; Manufacturer Murata -> Diodes Incorporated
- D5240: renamed from C5245; value 100pF C0G -> 1N4148W; footprint Capacitor_SMD:C_0603_1608Metric -> Diode_SMD:D_SOD-123; symbol Device:C -> Device:D; MPN GRM1885C1H101JA01D -> 1N4148W-7-F; Manufacturer Murata -> Diodes Incorporated
- D5280: renamed from C5285; value 100pF C0G -> 1N4148W; footprint Capacitor_SMD:C_0603_1608Metric -> Diode_SMD:D_SOD-123; symbol Device:C -> Device:D; MPN GRM1885C1H101JA01D -> 1N4148W-7-F; Manufacturer Murata -> Diodes Incorporated
- D5320: renamed from C5325; value 100pF C0G -> 1N4148W; footprint Capacitor_SMD:C_0603_1608Metric -> Diode_SMD:D_SOD-123; symbol Device:C -> Device:D; MPN GRM1885C1H101JA01D -> 1N4148W-7-F; Manufacturer Murata -> Diodes Incorporated
- K501: renamed from Q501; value 2N7002K -> TQ2-12V; footprint Package_TO_SOT_SMD:SOT-23 -> CM5Carrier:Panasonic_TQ2-12V_PRELIMINARY; symbol Transistor_FET:2N7002 -> CM5Carrier:Panasonic_TQ2_12V; MPN 2N7002K-7 -> TQ2-12V; Manufacturer Diodes Incorporated -> Panasonic Industry
- K502: renamed from Q502; value 2N7002K -> TQ2-12V; footprint Package_TO_SOT_SMD:SOT-23 -> CM5Carrier:Panasonic_TQ2-12V_PRELIMINARY; symbol Transistor_FET:2N7002 -> CM5Carrier:Panasonic_TQ2_12V; MPN 2N7002K-7 -> TQ2-12V; Manufacturer Diodes Incorporated -> Panasonic Industry
- K503: renamed from Q503; value 2N7002K -> TQ2-12V; footprint Package_TO_SOT_SMD:SOT-23 -> CM5Carrier:Panasonic_TQ2-12V_PRELIMINARY; symbol Transistor_FET:2N7002 -> CM5Carrier:Panasonic_TQ2_12V; MPN 2N7002K-7 -> TQ2-12V; Manufacturer Diodes Incorporated -> Panasonic Industry
- K504: renamed from Q504; value 2N7002K -> TQ2-12V; footprint Package_TO_SOT_SMD:SOT-23 -> CM5Carrier:Panasonic_TQ2-12V_PRELIMINARY; symbol Transistor_FET:2N7002 -> CM5Carrier:Panasonic_TQ2_12V; MPN 2N7002K-7 -> TQ2-12V; Manufacturer Diodes Incorporated -> Panasonic Industry
- K505: renamed from Q505; value 2N7002K -> TQ2-12V; footprint Package_TO_SOT_SMD:SOT-23 -> CM5Carrier:Panasonic_TQ2-12V_PRELIMINARY; symbol Transistor_FET:2N7002 -> CM5Carrier:Panasonic_TQ2_12V; MPN 2N7002K-7 -> TQ2-12V; Manufacturer Diodes Incorporated -> Panasonic Industry
- K506: renamed from Q506; value 2N7002K -> TQ2-12V; footprint Package_TO_SOT_SMD:SOT-23 -> CM5Carrier:Panasonic_TQ2-12V_PRELIMINARY; symbol Transistor_FET:2N7002 -> CM5Carrier:Panasonic_TQ2_12V; MPN 2N7002K-7 -> TQ2-12V; Manufacturer Diodes Incorporated -> Panasonic Industry
- K507: renamed from Q507; value 2N7002K -> TQ2-12V; footprint Package_TO_SOT_SMD:SOT-23 -> CM5Carrier:Panasonic_TQ2-12V_PRELIMINARY; symbol Transistor_FET:2N7002 -> CM5Carrier:Panasonic_TQ2_12V; MPN 2N7002K-7 -> TQ2-12V; Manufacturer Diodes Incorporated -> Panasonic Industry
- K508: renamed from Q508; value 2N7002K -> TQ2-12V; footprint Package_TO_SOT_SMD:SOT-23 -> CM5Carrier:Panasonic_TQ2-12V_PRELIMINARY; symbol Transistor_FET:2N7002 -> CM5Carrier:Panasonic_TQ2_12V; MPN 2N7002K-7 -> TQ2-12V; Manufacturer Diodes Incorporated -> Panasonic Industry
- L5040: renamed from C5046; value 100pF C0G -> 220R ferrite; footprint Capacitor_SMD:C_0603_1608Metric -> Inductor_SMD:L_0805_2012Metric; symbol Device:C -> Device:FerriteBead; MPN GRM1885C1H101JA01D -> BLM21PG221SN1D
- L5041: renamed from D5041; value S1G -> 220R ferrite; footprint Diode_SMD:D_SMA -> Inductor_SMD:L_0805_2012Metric; symbol Device:D -> Device:FerriteBead; MPN S1G-13-F -> BLM21PG221SN1D; Manufacturer Diodes Incorporated -> Murata
- L5080: renamed from C5086; value 100pF C0G -> 220R ferrite; footprint Capacitor_SMD:C_0603_1608Metric -> Inductor_SMD:L_0805_2012Metric; symbol Device:C -> Device:FerriteBead; MPN GRM1885C1H101JA01D -> BLM21PG221SN1D
- L5081: renamed from D5081; value S1G -> 220R ferrite; footprint Diode_SMD:D_SMA -> Inductor_SMD:L_0805_2012Metric; symbol Device:D -> Device:FerriteBead; MPN S1G-13-F -> BLM21PG221SN1D; Manufacturer Diodes Incorporated -> Murata
- L5120: renamed from C5126; value 100pF C0G -> 220R ferrite; footprint Capacitor_SMD:C_0603_1608Metric -> Inductor_SMD:L_0805_2012Metric; symbol Device:C -> Device:FerriteBead; MPN GRM1885C1H101JA01D -> BLM21PG221SN1D
- L5121: renamed from D5121; value S1G -> 220R ferrite; footprint Diode_SMD:D_SMA -> Inductor_SMD:L_0805_2012Metric; symbol Device:D -> Device:FerriteBead; MPN S1G-13-F -> BLM21PG221SN1D; Manufacturer Diodes Incorporated -> Murata
- L5160: renamed from C5166; value 100pF C0G -> 220R ferrite; footprint Capacitor_SMD:C_0603_1608Metric -> Inductor_SMD:L_0805_2012Metric; symbol Device:C -> Device:FerriteBead; MPN GRM1885C1H101JA01D -> BLM21PG221SN1D
- L5161: renamed from D5161; value S1G -> 220R ferrite; footprint Diode_SMD:D_SMA -> Inductor_SMD:L_0805_2012Metric; symbol Device:D -> Device:FerriteBead; MPN S1G-13-F -> BLM21PG221SN1D; Manufacturer Diodes Incorporated -> Murata
- L5200: renamed from C5206; value 100pF C0G -> 220R ferrite; footprint Capacitor_SMD:C_0603_1608Metric -> Inductor_SMD:L_0805_2012Metric; symbol Device:C -> Device:FerriteBead; MPN GRM1885C1H101JA01D -> BLM21PG221SN1D
- L5201: renamed from D5201; value S1G -> 220R ferrite; footprint Diode_SMD:D_SMA -> Inductor_SMD:L_0805_2012Metric; symbol Device:D -> Device:FerriteBead; MPN S1G-13-F -> BLM21PG221SN1D; Manufacturer Diodes Incorporated -> Murata
- L5240: renamed from C5246; value 100pF C0G -> 220R ferrite; footprint Capacitor_SMD:C_0603_1608Metric -> Inductor_SMD:L_0805_2012Metric; symbol Device:C -> Device:FerriteBead; MPN GRM1885C1H101JA01D -> BLM21PG221SN1D
- L5241: renamed from D5241; value S1G -> 220R ferrite; footprint Diode_SMD:D_SMA -> Inductor_SMD:L_0805_2012Metric; symbol Device:D -> Device:FerriteBead; MPN S1G-13-F -> BLM21PG221SN1D; Manufacturer Diodes Incorporated -> Murata
- L5280: renamed from C5286; value 100pF C0G -> 220R ferrite; footprint Capacitor_SMD:C_0603_1608Metric -> Inductor_SMD:L_0805_2012Metric; symbol Device:C -> Device:FerriteBead; MPN GRM1885C1H101JA01D -> BLM21PG221SN1D
- L5281: renamed from D5281; value S1G -> 220R ferrite; footprint Diode_SMD:D_SMA -> Inductor_SMD:L_0805_2012Metric; symbol Device:D -> Device:FerriteBead; MPN S1G-13-F -> BLM21PG221SN1D; Manufacturer Diodes Incorporated -> Murata
- L5320: renamed from C5326; value 100pF C0G -> 220R ferrite; footprint Capacitor_SMD:C_0603_1608Metric -> Inductor_SMD:L_0805_2012Metric; symbol Device:C -> Device:FerriteBead; MPN GRM1885C1H101JA01D -> BLM21PG221SN1D
- L5321: renamed from D5321; value S1G -> 220R ferrite; footprint Diode_SMD:D_SMA -> Inductor_SMD:L_0805_2012Metric; symbol Device:D -> Device:FerriteBead; MPN S1G-13-F -> BLM21PG221SN1D; Manufacturer Diodes Incorporated -> Murata
- R5040: renamed from R5043; value 4.7k 0.1% -> 3.9k 0.1%; MPN RC0603FR-074K7L -> RC0603FR-073K9L
- R5041: renamed from C5040; value 470pF C0G -> 3.9k 0.1%; footprint Capacitor_SMD:C_0603_1608Metric -> Resistor_SMD:R_0603_1608Metric; symbol Device:C -> Device:R; MPN GRM1885C1H471JA01D -> RC0603FR-073K9L; Manufacturer Murata -> Yageo
- R5042: renamed from C5041; value 470pF C0G -> 4.7k 0.1%; footprint Capacitor_SMD:C_0603_1608Metric -> Resistor_SMD:R_0603_1608Metric; symbol Device:C -> Device:R; MPN GRM1885C1H471JA01D -> RC0603FR-074K7L; Manufacturer Murata -> Yageo
- R5043: renamed from U501; value OPA1652AIDR -> 4.7k 0.1%; footprint Package_SO:SOIC-8_3.9x4.9mm_P1.27mm -> Resistor_SMD:R_0603_1608Metric; symbol CM5Carrier:OPA1652 -> Device:R; MPN OPA1652AIDR -> RC0603FR-074K7L; Manufacturer Texas Instruments -> Yageo
- R5044: renamed from R5046; value 10k 0.1% -> 150R; MPN RC0603FR-0710KL -> RC0603FR-07150RL
- R5080: renamed from R5083; value 4.7k 0.1% -> 3.9k 0.1%; MPN RC0603FR-074K7L -> RC0603FR-073K9L
- R5081: renamed from C5080; value 470pF C0G -> 3.9k 0.1%; footprint Capacitor_SMD:C_0603_1608Metric -> Resistor_SMD:R_0603_1608Metric; symbol Device:C -> Device:R; MPN GRM1885C1H471JA01D -> RC0603FR-073K9L; Manufacturer Murata -> Yageo
- R5082: renamed from C5081; value 470pF C0G -> 4.7k 0.1%; footprint Capacitor_SMD:C_0603_1608Metric -> Resistor_SMD:R_0603_1608Metric; symbol Device:C -> Device:R; MPN GRM1885C1H471JA01D -> RC0603FR-074K7L; Manufacturer Murata -> Yageo
- R5083: renamed from U502; value OPA1652AIDR -> 4.7k 0.1%; footprint Package_SO:SOIC-8_3.9x4.9mm_P1.27mm -> Resistor_SMD:R_0603_1608Metric; symbol CM5Carrier:OPA1652 -> Device:R; MPN OPA1652AIDR -> RC0603FR-074K7L; Manufacturer Texas Instruments -> Yageo
- R5084: renamed from R5086; value 10k 0.1% -> 150R; MPN RC0603FR-0710KL -> RC0603FR-07150RL
- R5120: renamed from R5123; value 4.7k 0.1% -> 3.9k 0.1%; MPN RC0603FR-074K7L -> RC0603FR-073K9L
- R5121: renamed from C5120; value 470pF C0G -> 3.9k 0.1%; footprint Capacitor_SMD:C_0603_1608Metric -> Resistor_SMD:R_0603_1608Metric; symbol Device:C -> Device:R; MPN GRM1885C1H471JA01D -> RC0603FR-073K9L; Manufacturer Murata -> Yageo
- R5122: renamed from C5121; value 470pF C0G -> 4.7k 0.1%; footprint Capacitor_SMD:C_0603_1608Metric -> Resistor_SMD:R_0603_1608Metric; symbol Device:C -> Device:R; MPN GRM1885C1H471JA01D -> RC0603FR-074K7L; Manufacturer Murata -> Yageo
- R5123: renamed from U503; value OPA1652AIDR -> 4.7k 0.1%; footprint Package_SO:SOIC-8_3.9x4.9mm_P1.27mm -> Resistor_SMD:R_0603_1608Metric; symbol CM5Carrier:OPA1652 -> Device:R; MPN OPA1652AIDR -> RC0603FR-074K7L; Manufacturer Texas Instruments -> Yageo
- R5124: renamed from R5126; value 10k 0.1% -> 150R; MPN RC0603FR-0710KL -> RC0603FR-07150RL
- R5160: renamed from R5163; value 4.7k 0.1% -> 3.9k 0.1%; MPN RC0603FR-074K7L -> RC0603FR-073K9L
- R5161: renamed from C5160; value 470pF C0G -> 3.9k 0.1%; footprint Capacitor_SMD:C_0603_1608Metric -> Resistor_SMD:R_0603_1608Metric; symbol Device:C -> Device:R; MPN GRM1885C1H471JA01D -> RC0603FR-073K9L; Manufacturer Murata -> Yageo
- R5162: renamed from C5161; value 470pF C0G -> 4.7k 0.1%; footprint Capacitor_SMD:C_0603_1608Metric -> Resistor_SMD:R_0603_1608Metric; symbol Device:C -> Device:R; MPN GRM1885C1H471JA01D -> RC0603FR-074K7L; Manufacturer Murata -> Yageo
- R5163: renamed from U504; value OPA1652AIDR -> 4.7k 0.1%; footprint Package_SO:SOIC-8_3.9x4.9mm_P1.27mm -> Resistor_SMD:R_0603_1608Metric; symbol CM5Carrier:OPA1652 -> Device:R; MPN OPA1652AIDR -> RC0603FR-074K7L; Manufacturer Texas Instruments -> Yageo
- R5164: renamed from R5166; value 10k 0.1% -> 150R; MPN RC0603FR-0710KL -> RC0603FR-07150RL
- R5200: renamed from R5203; value 4.7k 0.1% -> 3.9k 0.1%; MPN RC0603FR-074K7L -> RC0603FR-073K9L
- R5201: renamed from C5200; value 470pF C0G -> 3.9k 0.1%; footprint Capacitor_SMD:C_0603_1608Metric -> Resistor_SMD:R_0603_1608Metric; symbol Device:C -> Device:R; MPN GRM1885C1H471JA01D -> RC0603FR-073K9L; Manufacturer Murata -> Yageo
- R5202: renamed from C5201; value 470pF C0G -> 4.7k 0.1%; footprint Capacitor_SMD:C_0603_1608Metric -> Resistor_SMD:R_0603_1608Metric; symbol Device:C -> Device:R; MPN GRM1885C1H471JA01D -> RC0603FR-074K7L; Manufacturer Murata -> Yageo
- R5203: renamed from U505; value OPA1652AIDR -> 4.7k 0.1%; footprint Package_SO:SOIC-8_3.9x4.9mm_P1.27mm -> Resistor_SMD:R_0603_1608Metric; symbol CM5Carrier:OPA1652 -> Device:R; MPN OPA1652AIDR -> RC0603FR-074K7L; Manufacturer Texas Instruments -> Yageo
- R5204: renamed from R5206; value 10k 0.1% -> 150R; MPN RC0603FR-0710KL -> RC0603FR-07150RL
- R5240: renamed from R5243; value 4.7k 0.1% -> 3.9k 0.1%; MPN RC0603FR-074K7L -> RC0603FR-073K9L
- R5241: renamed from C5240; value 470pF C0G -> 3.9k 0.1%; footprint Capacitor_SMD:C_0603_1608Metric -> Resistor_SMD:R_0603_1608Metric; symbol Device:C -> Device:R; MPN GRM1885C1H471JA01D -> RC0603FR-073K9L; Manufacturer Murata -> Yageo
- R5242: renamed from C5241; value 470pF C0G -> 4.7k 0.1%; footprint Capacitor_SMD:C_0603_1608Metric -> Resistor_SMD:R_0603_1608Metric; symbol Device:C -> Device:R; MPN GRM1885C1H471JA01D -> RC0603FR-074K7L; Manufacturer Murata -> Yageo
- R5243: renamed from U506; value OPA1652AIDR -> 4.7k 0.1%; footprint Package_SO:SOIC-8_3.9x4.9mm_P1.27mm -> Resistor_SMD:R_0603_1608Metric; symbol CM5Carrier:OPA1652 -> Device:R; MPN OPA1652AIDR -> RC0603FR-074K7L; Manufacturer Texas Instruments -> Yageo
- R5244: renamed from R5246; value 10k 0.1% -> 150R; MPN RC0603FR-0710KL -> RC0603FR-07150RL
- R5280: renamed from R5283; value 4.7k 0.1% -> 3.9k 0.1%; MPN RC0603FR-074K7L -> RC0603FR-073K9L
- R5281: renamed from C5280; value 470pF C0G -> 3.9k 0.1%; footprint Capacitor_SMD:C_0603_1608Metric -> Resistor_SMD:R_0603_1608Metric; symbol Device:C -> Device:R; MPN GRM1885C1H471JA01D -> RC0603FR-073K9L; Manufacturer Murata -> Yageo
- R5282: renamed from C5281; value 470pF C0G -> 4.7k 0.1%; footprint Capacitor_SMD:C_0603_1608Metric -> Resistor_SMD:R_0603_1608Metric; symbol Device:C -> Device:R; MPN GRM1885C1H471JA01D -> RC0603FR-074K7L; Manufacturer Murata -> Yageo
- R5283: renamed from U507; value OPA1652AIDR -> 4.7k 0.1%; footprint Package_SO:SOIC-8_3.9x4.9mm_P1.27mm -> Resistor_SMD:R_0603_1608Metric; symbol CM5Carrier:OPA1652 -> Device:R; MPN OPA1652AIDR -> RC0603FR-074K7L; Manufacturer Texas Instruments -> Yageo
- R5284: renamed from R5286; value 10k 0.1% -> 150R; MPN RC0603FR-0710KL -> RC0603FR-07150RL
- R5320: renamed from R5323; value 4.7k 0.1% -> 3.9k 0.1%; MPN RC0603FR-074K7L -> RC0603FR-073K9L
- R5321: renamed from C5320; value 470pF C0G -> 3.9k 0.1%; footprint Capacitor_SMD:C_0603_1608Metric -> Resistor_SMD:R_0603_1608Metric; symbol Device:C -> Device:R; MPN GRM1885C1H471JA01D -> RC0603FR-073K9L; Manufacturer Murata -> Yageo
- R5322: renamed from C5321; value 470pF C0G -> 4.7k 0.1%; footprint Capacitor_SMD:C_0603_1608Metric -> Resistor_SMD:R_0603_1608Metric; symbol Device:C -> Device:R; MPN GRM1885C1H471JA01D -> RC0603FR-074K7L; Manufacturer Murata -> Yageo
- R5323: renamed from U508; value OPA1652AIDR -> 4.7k 0.1%; footprint Package_SO:SOIC-8_3.9x4.9mm_P1.27mm -> Resistor_SMD:R_0603_1608Metric; symbol CM5Carrier:OPA1652 -> Device:R; MPN OPA1652AIDR -> RC0603FR-074K7L; Manufacturer Texas Instruments -> Yageo
- R5324: renamed from R5326; value 10k 0.1% -> 150R; MPN RC0603FR-0710KL -> RC0603FR-07150RL
- U501: renamed from R5044; value 150R -> OPA1652AIDR; footprint Resistor_SMD:R_0603_1608Metric -> Package_SO:SOIC-8_3.9x4.9mm_P1.27mm; symbol Device:R -> CM5Carrier:OPA1652; MPN RC0603FR-07150RL -> OPA1652AIDR; Manufacturer Yageo -> Texas Instruments
- U502: renamed from R5084; value 150R -> OPA1652AIDR; footprint Resistor_SMD:R_0603_1608Metric -> Package_SO:SOIC-8_3.9x4.9mm_P1.27mm; symbol Device:R -> CM5Carrier:OPA1652; MPN RC0603FR-07150RL -> OPA1652AIDR; Manufacturer Yageo -> Texas Instruments
- U503: renamed from R5124; value 150R -> OPA1652AIDR; footprint Resistor_SMD:R_0603_1608Metric -> Package_SO:SOIC-8_3.9x4.9mm_P1.27mm; symbol Device:R -> CM5Carrier:OPA1652; MPN RC0603FR-07150RL -> OPA1652AIDR; Manufacturer Yageo -> Texas Instruments
- U504: renamed from R5164; value 150R -> OPA1652AIDR; footprint Resistor_SMD:R_0603_1608Metric -> Package_SO:SOIC-8_3.9x4.9mm_P1.27mm; symbol Device:R -> CM5Carrier:OPA1652; MPN RC0603FR-07150RL -> OPA1652AIDR; Manufacturer Yageo -> Texas Instruments
- U505: renamed from R5204; value 150R -> OPA1652AIDR; footprint Resistor_SMD:R_0603_1608Metric -> Package_SO:SOIC-8_3.9x4.9mm_P1.27mm; symbol Device:R -> CM5Carrier:OPA1652; MPN RC0603FR-07150RL -> OPA1652AIDR; Manufacturer Yageo -> Texas Instruments
- U506: renamed from R5244; value 150R -> OPA1652AIDR; footprint Resistor_SMD:R_0603_1608Metric -> Package_SO:SOIC-8_3.9x4.9mm_P1.27mm; symbol Device:R -> CM5Carrier:OPA1652; MPN RC0603FR-07150RL -> OPA1652AIDR; Manufacturer Yageo -> Texas Instruments
- U507: renamed from R5284; value 150R -> OPA1652AIDR; footprint Resistor_SMD:R_0603_1608Metric -> Package_SO:SOIC-8_3.9x4.9mm_P1.27mm; symbol Device:R -> CM5Carrier:OPA1652; MPN RC0603FR-07150RL -> OPA1652AIDR; Manufacturer Yageo -> Texas Instruments
- U508: renamed from R5324; value 150R -> OPA1652AIDR; footprint Resistor_SMD:R_0603_1608Metric -> Package_SO:SOIC-8_3.9x4.9mm_P1.27mm; symbol Device:R -> CM5Carrier:OPA1652; MPN RC0603FR-07150RL -> OPA1652AIDR; Manufacturer Yageo -> Texas Instruments
- U521: renamed from C5047; value 100nF -> THAT1646S08-U; footprint Capacitor_SMD:C_0402_1005Metric -> Package_SO:SOIC-8_3.9x4.9mm_P1.27mm; symbol Device:C -> CM5Carrier:THAT1646; MPN C1005X7R1H104K050BB -> THAT1646S08-U; Manufacturer TDK -> THAT Corporation
- U522: renamed from C5087; value 100nF -> THAT1646S08-U; footprint Capacitor_SMD:C_0402_1005Metric -> Package_SO:SOIC-8_3.9x4.9mm_P1.27mm; symbol Device:C -> CM5Carrier:THAT1646; MPN C1005X7R1H104K050BB -> THAT1646S08-U; Manufacturer TDK -> THAT Corporation
- U523: renamed from C5127; value 100nF -> THAT1646S08-U; footprint Capacitor_SMD:C_0402_1005Metric -> Package_SO:SOIC-8_3.9x4.9mm_P1.27mm; symbol Device:C -> CM5Carrier:THAT1646; MPN C1005X7R1H104K050BB -> THAT1646S08-U; Manufacturer TDK -> THAT Corporation
- U524: renamed from C5167; value 100nF -> THAT1646S08-U; footprint Capacitor_SMD:C_0402_1005Metric -> Package_SO:SOIC-8_3.9x4.9mm_P1.27mm; symbol Device:C -> CM5Carrier:THAT1646; MPN C1005X7R1H104K050BB -> THAT1646S08-U; Manufacturer TDK -> THAT Corporation
- U525: renamed from C5207; value 100nF -> THAT1646S08-U; footprint Capacitor_SMD:C_0402_1005Metric -> Package_SO:SOIC-8_3.9x4.9mm_P1.27mm; symbol Device:C -> CM5Carrier:THAT1646; MPN C1005X7R1H104K050BB -> THAT1646S08-U; Manufacturer TDK -> THAT Corporation
- U526: renamed from C5247; value 100nF -> THAT1646S08-U; footprint Capacitor_SMD:C_0402_1005Metric -> Package_SO:SOIC-8_3.9x4.9mm_P1.27mm; symbol Device:C -> CM5Carrier:THAT1646; MPN C1005X7R1H104K050BB -> THAT1646S08-U; Manufacturer TDK -> THAT Corporation
- U527: renamed from C5287; value 100nF -> THAT1646S08-U; footprint Capacitor_SMD:C_0402_1005Metric -> Package_SO:SOIC-8_3.9x4.9mm_P1.27mm; symbol Device:C -> CM5Carrier:THAT1646; MPN C1005X7R1H104K050BB -> THAT1646S08-U; Manufacturer TDK -> THAT Corporation
- U528: renamed from C5327; value 100nF -> THAT1646S08-U; footprint Capacitor_SMD:C_0402_1005Metric -> Package_SO:SOIC-8_3.9x4.9mm_P1.27mm; symbol Device:C -> CM5Carrier:THAT1646; MPN C1005X7R1H104K050BB -> THAT1646S08-U; Manufacturer TDK -> THAT Corporation
- renumbered C5050 to C5047, C5090 to C5087, C5130 to C5127, C5170 to C5167, C5210 to C5207, C5250 to C5247, C5290 to C5287, C5330 to C5327, D5044 to D5041, D5084 to D5081, D5124 to D5121, D5164 to D5161, D5204 to D5201, D5244 to D5241, D5284 to D5281, D5324 to D5321
Connections:
- net AGND: now also C5042.2, C5048.2, C5049.2, C5082.2, C5088.2, C5089.2, C5122.2, C5128.2, C5129.2, C5162.2, C5168.2, C5169.2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; no longer C5042.3 (GND), C5050.9 (NC2), C5082.3 (GND), C5090.9 (NC2), C5122.3 (GND), C5130.9 (NC2), C5162.3 (GND), C5170.9 (NC2), C5202.3 (GND), C5210.9 (NC2), C5242.3 (GND), C5250.9 (NC2)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
- net AOUT1_COIL_LOW: now also D5040.1 (K), K501.10 (COIL-), Q501.3 (D); no longer C5050.10 (COIL-), K501.3 (D)
- net AOUT1_DRIVE: now also U501.7 (OUT_B), U521.4 (IN); no longer C5042.4 (IN), R5043.7 (OUT_B)
- net AOUT1_DRV_N: now also K501.3 (COM1), U521.1 (OUT-), C5043.1; no longer C5042.1 (OUT-), C5048.1, C5050.3 (COM1)
- net AOUT1_DRV_P: now also K501.8 (COM2), U521.8 (OUT+), C5044.1; no longer C5042.8 (OUT+), C5049.1, C5050.8 (COM2)
- net AOUT1_GAIN_FB: now also U501.6 (IN_B-), R5046.1; no longer R5043.6 (IN_B-), R5044.1
- net AOUT1_LPF_N: now also R5042.2, U501.2 (IN_A-), C5040.2; no longer R5043.2 (IN_A-)
- net AOUT1_LPF_P: now also R5040.2, R5043.1, U501.3 (IN_A+), C5041.1; no longer R5040.1, R5042.1, R5043.3 (IN_A+)
- net AOUT1_LPF_POST: now also C5042.1, R5044.2, U501.5 (IN_B+); no longer R5043.5 (IN_B+), U501.2
- net AOUT1_LPF_SE: now also R5042.1, R5044.1, C5040.1; no longer R5041.1, R5043.1 (OUT_A)
- net AOUT1_RELAY_N: now also K501.4 (NO1), L5040.1; no longer C5050.4 (NO1)
- net AOUT1_RELAY_P: now also K501.7 (NO2), L5041.1; no longer C5050.7 (NO2)
- net AOUT1_SNS_N: now also U521.2 (SNS-), C5043.2; no longer C5042.2 (SNS-), C5048.2
- net AOUT1_SNS_P: now also U521.7 (SNS+), C5044.2; no longer C5042.7 (SNS+), C5049.2
- net AOUT2_COIL_LOW: now also D5080.1 (K), K502.10 (COIL-), Q502.3 (D); no longer C5090.10 (COIL-), K502.3 (D)
- net AOUT2_DRIVE: now also U502.7 (OUT_B), U522.4 (IN); no longer C5082.4 (IN), R5083.7 (OUT_B)
- net AOUT2_DRV_N: now also K502.3 (COM1), U522.1 (OUT-), C5083.1; no longer C5082.1 (OUT-), C5088.1, C5090.3 (COM1)
- net AOUT2_DRV_P: now also K502.8 (COM2), U522.8 (OUT+), C5084.1; no longer C5082.8 (OUT+), C5089.1, C5090.8 (COM2)
- net AOUT2_GAIN_FB: now also U502.6 (IN_B-), R5086.1; no longer R5083.6 (IN_B-), R5084.1
- net AOUT2_LPF_N: now also R5082.2, U502.2 (IN_A-), C5080.2; no longer R5083.2 (IN_A-)
- net AOUT2_LPF_P: now also R5080.2, R5083.1, U502.3 (IN_A+), C5081.1; no longer R5080.1, R5082.1, R5083.3 (IN_A+)
- net AOUT2_LPF_POST: now also C5082.1, R5084.2, U502.5 (IN_B+); no longer R5083.5 (IN_B+), U502.2
- net AOUT2_LPF_SE: now also R5082.1, R5084.1, C5080.1; no longer R5081.1, R5083.1 (OUT_A)
- net AOUT2_RELAY_N: now also K502.4 (NO1), L5080.1; no longer C5090.4 (NO1)
- net AOUT2_RELAY_P: now also K502.7 (NO2), L5081.1; no longer C5090.7 (NO2)
- net AOUT2_SNS_N: now also U522.2 (SNS-), C5083.2; no longer C5082.2 (SNS-), C5088.2
- net AOUT2_SNS_P: now also U522.7 (SNS+), C5084.2; no longer C5082.7 (SNS+), C5089.2
- net AOUT3_COIL_LOW: now also D5120.1 (K), K503.10 (COIL-), Q503.3 (D); no longer C5130.10 (COIL-), K503.3 (D)
- net AOUT3_DRIVE: now also U503.7 (OUT_B), U523.4 (IN); no longer C5122.4 (IN), R5123.7 (OUT_B)
- net AOUT3_DRV_N: now also K503.3 (COM1), U523.1 (OUT-), C5123.1; no longer C5122.1 (OUT-), C5128.1, C5130.3 (COM1)
- net AOUT3_DRV_P: now also K503.8 (COM2), U523.8 (OUT+), C5124.1; no longer C5122.8 (OUT+), C5129.1, C5130.8 (COM2)
- net AOUT3_GAIN_FB: now also U503.6 (IN_B-), R5126.1; no longer R5123.6 (IN_B-), R5124.1
- net AOUT3_LPF_N: now also R5122.2, U503.2 (IN_A-), C5120.2; no longer R5123.2 (IN_A-)
- net AOUT3_LPF_P: now also R5120.2, R5123.1, U503.3 (IN_A+), C5121.1; no longer R5120.1, R5122.1, R5123.3 (IN_A+)
- net AOUT3_LPF_POST: now also C5122.1, R5124.2, U503.5 (IN_B+); no longer R5123.5 (IN_B+), U503.2
- net AOUT3_LPF_SE: now also R5122.1, R5124.1, C5120.1; no longer R5121.1, R5123.1 (OUT_A)
- net AOUT3_RELAY_N: now also K503.4 (NO1), L5120.1; no longer C5130.4 (NO1)
- net AOUT3_RELAY_P: now also K503.7 (NO2), L5121.1; no longer C5130.7 (NO2)
- net AOUT3_SNS_N: now also U523.2 (SNS-), C5123.2; no longer C5122.2 (SNS-), C5128.2
- net AOUT3_SNS_P: now also U523.7 (SNS+), C5124.2; no longer C5122.7 (SNS+), C5129.2
- net AOUT4_COIL_LOW: now also D5160.1 (K), K504.10 (COIL-), Q504.3 (D); no longer C5170.10 (COIL-), K504.3 (D)
- net AOUT4_DRIVE: now also U504.7 (OUT_B), U524.4 (IN); no longer C5162.4 (IN), R5163.7 (OUT_B)
- net AOUT4_DRV_N: now also K504.3 (COM1), U524.1 (OUT-), C5163.1; no longer C5162.1 (OUT-), C5168.1, C5170.3 (COM1)
- net AOUT4_DRV_P: now also K504.8 (COM2), U524.8 (OUT+), C5164.1; no longer C5162.8 (OUT+), C5169.1, C5170.8 (COM2)
- net AOUT4_GAIN_FB: now also U504.6 (IN_B-), R5166.1; no longer R5163.6 (IN_B-), R5164.1
- net AOUT4_LPF_N: now also R5162.2, U504.2 (IN_A-), C5160.2; no longer R5163.2 (IN_A-)
- net AOUT4_LPF_P: now also R5160.2, R5163.1, U504.3 (IN_A+), C5161.1; no longer R5160.1, R5162.1, R5163.3 (IN_A+)
- net AOUT4_LPF_POST: now also C5162.1, R5164.2, U504.5 (IN_B+); no longer R5163.5 (IN_B+), U504.2
- net AOUT4_LPF_SE: now also R5162.1, R5164.1, C5160.1; no longer R5161.1, R5163.1 (OUT_A)
- net AOUT4_RELAY_N: now also K504.4 (NO1), L5160.1; no longer C5170.4 (NO1)
- net AOUT4_RELAY_P: now also K504.7 (NO2), L5161.1; no longer C5170.7 (NO2)
- net AOUT4_SNS_N: now also U524.2 (SNS-), C5163.2; no longer C5162.2 (SNS-), C5168.2
- net AOUT4_SNS_P: now also U524.7 (SNS+), C5164.2; no longer C5162.7 (SNS+), C5169.2
- net AOUT5_COIL_LOW: now also D5200.1 (K), K505.10 (COIL-), Q505.3 (D); no longer C5210.10 (COIL-), K505.3 (D)
- net AOUT5_DRIVE: now also U505.7 (OUT_B), U525.4 (IN); no longer C5202.4 (IN), R5203.7 (OUT_B)
- net AOUT5_DRV_N: now also K505.3 (COM1), U525.1 (OUT-), C5203.1; no longer C5202.1 (OUT-), C5208.1, C5210.3 (COM1)
- net AOUT5_DRV_P: now also K505.8 (COM2), U525.8 (OUT+), C5204.1; no longer C5202.8 (OUT+), C5209.1, C5210.8 (COM2)
- net AOUT5_GAIN_FB: now also U505.6 (IN_B-), R5206.1; no longer R5203.6 (IN_B-), R5204.1
- net AOUT5_LPF_N: now also R5202.2, U505.2 (IN_A-), C5200.2; no longer R5203.2 (IN_A-)
- net AOUT5_LPF_P: now also R5200.2, R5203.1, U505.3 (IN_A+), C5201.1; no longer R5200.1, R5202.1, R5203.3 (IN_A+)
- net AOUT5_LPF_POST: now also C5202.1, R5204.2, U505.5 (IN_B+); no longer R5203.5 (IN_B+), U505.2
- net AOUT5_LPF_SE: now also R5202.1, R5204.1, C5200.1; no longer R5201.1, R5203.1 (OUT_A)
- net AOUT5_RELAY_N: now also K505.4 (NO1), L5200.1; no longer C5210.4 (NO1)
- net AOUT5_RELAY_P: now also K505.7 (NO2), L5201.1; no longer C5210.7 (NO2)
- net AOUT5_SNS_N: now also U525.2 (SNS-), C5203.2; no longer C5202.2 (SNS-), C5208.2
- net AOUT5_SNS_P: now also U525.7 (SNS+), C5204.2; no longer C5202.7 (SNS+), C5209.2
- net AOUT6_COIL_LOW: now also D5240.1 (K), K506.10 (COIL-), Q506.3 (D); no longer C5250.10 (COIL-), K506.3 (D)
- net AOUT6_DRIVE: now also U506.7 (OUT_B), U526.4 (IN); no longer C5242.4 (IN), R5243.7 (OUT_B)
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Other:
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