File: cad/kicad/AUDIO-8X8/Audio-Power.kicad_sch (KiCad schematic)
At the start: 47 parts, among them J102 AUDIO_12V_POWER, U601 TRI 20-1223, U602 TPS62913RPU, U603 LT3045IMSE, U604 LT3045IMSE, U605 TPS7A2033PDBVR

Commit message: Audit schematic logic against controlled datasheets
Connections:
- net AGND: now also U602.7 (PSNS)
- net AUDIO_5V5_PRE: no longer U602.7 (PSNS)
Other:
- note added: "Release order: AUDIO_ENABLE -> 5V5_PG -> LT3045 PGs + AKM 3V3 valid -> clocks -> resets -> carrier unmute command."
- note added: "U106 on Audio-TDM-Clock hardware-gates DAC unmute and every output relay with ADC_5V_PG and DAC_5V_PG."
- note removed: "Any PG loss immediately de-energizes all output relays and reasserts DAC mute before software intervention."
- note removed: "Release order: AUDIO_ENABLE -> 5V5_PG -> LT3045 PGs + AKM 3V3 valid -> clocks -> resets -> DAC unmute -> output relays."

Commit message: Implement direct socketed dual-SIM daughterboard
Parts:
- removed C610: 4.7uF 50V, Capacitor_SMD:C_1206_3216Metric, symbol Device:C
- removed C630, C650: 470nF, Capacitor_SMD:C_0603_1608Metric, symbol Device:C
- removed C670: 1uF, Capacitor_SMD:C_0603_1608Metric, symbol Device:C
- removed C672: 4.7uF, Capacitor_SMD:C_0805_2012Metric, symbol Device:C
- removed F601: 3A fuse, Fuse:Fuse_Littelfuse-NANO2-451_453, symbol Device:Fuse
- removed L601: 2.2uH, Inductor_SMD:L_Coilcraft_XxL4040, symbol Device:L
- removed R601: 0R power star, Resistor_SMD:R_2512_6332Metric, symbol Device:R
- removed R610: 29.4k 0.1%, Resistor_SMD:R_0603_1608Metric, symbol Device:R
- removed R611: 4.99k 0.1%, Resistor_SMD:R_0603_1608Metric, symbol Device:R
- removed R630, R650: 499R 1% / 300mA ILIM, Resistor_SMD:R_0603_1608Metric, symbol Device:R
- removed R631, R651: 49.9k 0.1%, Resistor_SMD:R_0603_1608Metric, symbol Device:R
- removed U605: TPS7A2033PDBVR, Package_TO_SOT_SMD:SOT-23-5, symbol CM5Carrier:TPS7A20DBV_A1
- added C603: 22uF 25V, Capacitor_SMD:C_1210_3225Metric, symbol Device:C
- added C611, C622: 4.7uF 50V, Capacitor_SMD:C_1206_3216Metric, symbol Device:C
- added C613: 100nF, Capacitor_SMD:C_0402_1005Metric, symbol Device:C
- added C623, C624: 22uF 10V, Capacitor_SMD:C_0805_2012Metric, symbol Device:C
- added C631, C632, C651, C652: 10uF, Capacitor_SMD:C_0603_1608Metric, symbol Device:C
- added C673: 100uF 6.3V polymer, Capacitor_SMD:CP_Elec_6.3x5.8, symbol Device:C_Polarized
- added R634, R654: 100k 1%, Resistor_SMD:R_0603_1608Metric, symbol Device:R
- added R670, R671: 10k 0.1%, Resistor_SMD:R_0603_1608Metric, symbol Device:R
- C602: renamed from U601; value TRI 20-1223 -> 22uF 25V; footprint CM5Carrier:TRACO_TRI20_DUAL -> Capacitor_SMD:C_1210_3225Metric; symbol CM5Carrier:TRI20_1223 -> Device:C; MPN TRI 20-1223 -> GRM32ER71E226KE15L; Manufacturer TRACO Power -> Murata
- C610: renamed from C613; value 100nF -> 4.7uF 50V; footprint Capacitor_SMD:C_0402_1005Metric -> Capacitor_SMD:C_1206_3216Metric; MPN C1005X7R1H104K050BB -> GRM31CR71H475KA12L; Manufacturer TDK -> Murata
- C620: renamed from C621; value 4.7uF 50V -> 470nF; footprint Capacitor_SMD:C_1206_3216Metric -> Capacitor_SMD:C_0603_1608Metric; MPN GRM31CR71H475KA12L -> GRM188R71E474KA12D
- C621: renamed from C624; value 22uF 10V -> 4.7uF 50V; footprint Capacitor_SMD:C_0805_2012Metric -> Capacitor_SMD:C_1206_3216Metric; MPN GRM21BR71A226ME44L -> GRM31CR71H475KA12L
- C630: renamed from R634; value 100k 1% -> 470nF; footprint Resistor_SMD:R_0603_1608Metric -> Capacitor_SMD:C_0603_1608Metric; symbol Device:R -> Device:C; MPN RC0603FR-07100KL -> GRM188R71E474KA12D; Manufacturer Yageo -> Murata
- C650: renamed from R654; value 100k 1% -> 470nF; footprint Resistor_SMD:R_0603_1608Metric -> Capacitor_SMD:C_0603_1608Metric; symbol Device:R -> Device:C; MPN RC0603FR-07100KL -> GRM188R71E474KA12D; Manufacturer Yageo -> Murata
- C670: renamed from R670; value 10k 0.1% -> 1uF; footprint Resistor_SMD:R_0603_1608Metric -> Capacitor_SMD:C_0603_1608Metric; symbol Device:R -> Device:C; MPN RC0603FR-0710KL -> GRM188R71A105KA61D; Manufacturer Yageo -> Murata
- C671: renamed from R671; value 10k 0.1% -> 1uF; footprint Resistor_SMD:R_0603_1608Metric -> Capacitor_SMD:C_0603_1608Metric; symbol Device:R -> Device:C; MPN RC0603FR-0710KL -> GRM188R71A105KA61D; Manufacturer Yageo -> Murata
- C672: renamed from C673; value 100uF 6.3V polymer -> 4.7uF; footprint Capacitor_SMD:CP_Elec_6.3x5.8 -> Capacitor_SMD:C_0805_2012Metric; symbol Device:C_Polarized -> Device:C; MPN 6SVP100M -> GRM21BR71A475KA73L; Manufacturer Panasonic -> Murata
- F601: renamed from C602; value 22uF 25V -> 3A fuse; footprint Capacitor_SMD:C_1210_3225Metric -> Fuse:Fuse_Littelfuse-NANO2-451_453; symbol Device:C -> Device:Fuse; MPN GRM32ER71E226KE15L -> 0453003.MR; Manufacturer Murata -> Littelfuse
- L601: renamed from C620; value 470nF -> 2.2uH; footprint Capacitor_SMD:C_0603_1608Metric -> Inductor_SMD:L_Coilcraft_XxL4040; symbol Device:C -> Device:L; MPN GRM188R71E474KA12D -> XGL4030-222MEC; Manufacturer Murata -> Coilcraft
- R601: renamed from C603; value 22uF 25V -> 0R power star; footprint Capacitor_SMD:C_1210_3225Metric -> Resistor_SMD:R_2512_6332Metric; symbol Device:C -> Device:R; MPN GRM32ER71E226KE15L -> RC2512JK-070RL; Manufacturer Murata -> Yageo
- R610: renamed from R612; value 7.5k 0.1% -> 29.4k 0.1%; MPN RC0603FR-077K5L -> TNPW060329K4BEEA; Manufacturer Yageo -> Vishay
- R611: renamed from R613; value 10k 0.1% -> 4.99k 0.1%; MPN RC0603FR-0710KL -> RC0603FR-074K99L
- R612: renamed from C622; value 4.7uF 50V -> 7.5k 0.1%; footprint Capacitor_SMD:C_1206_3216Metric -> Resistor_SMD:R_0603_1608Metric; symbol Device:C -> Device:R; MPN GRM31CR71H475KA12L -> RC0603FR-077K5L; Manufacturer Murata -> Yageo
- R613: renamed from C623; value 22uF 10V -> 10k 0.1%; footprint Capacitor_SMD:C_0805_2012Metric -> Resistor_SMD:R_0603_1608Metric; symbol Device:C -> Device:R; MPN GRM21BR71A226ME44L -> RC0603FR-0710KL; Manufacturer Murata -> Yageo
- R630: renamed from R632; value 140k 1% -> 499R 1% / 300mA ILIM; MPN RC0603FR-07140KL -> RC0603FR-07499RL
- R631: renamed from R633; value 10k 0.1% -> 49.9k 0.1%; MPN RC0603FR-0710KL -> TNPW060349K9BEEA; Manufacturer Yageo -> Vishay
- R632: renamed from C631; value 10uF -> 140k 1%; footprint Capacitor_SMD:C_0603_1608Metric -> Resistor_SMD:R_0603_1608Metric; symbol Device:C -> Device:R; MPN GRM188R71A106KA73D -> RC0603FR-07140KL; Manufacturer Murata -> Yageo
- R633: renamed from C632; value 10uF -> 10k 0.1%; footprint Capacitor_SMD:C_0603_1608Metric -> Resistor_SMD:R_0603_1608Metric; symbol Device:C -> Device:R; MPN GRM188R71A106KA73D -> RC0603FR-0710KL; Manufacturer Murata -> Yageo
- R650: renamed from R652; value 140k 1% -> 499R 1% / 300mA ILIM; MPN RC0603FR-07140KL -> RC0603FR-07499RL
- R651: renamed from R653; value 10k 0.1% -> 49.9k 0.1%; MPN RC0603FR-0710KL -> TNPW060349K9BEEA; Manufacturer Yageo -> Vishay
- R652: renamed from C651; value 10uF -> 140k 1%; footprint Capacitor_SMD:C_0603_1608Metric -> Resistor_SMD:R_0603_1608Metric; symbol Device:C -> Device:R; MPN GRM188R71A106KA73D -> RC0603FR-07140KL; Manufacturer Murata -> Yageo
- R653: renamed from C652; value 10uF -> 10k 0.1%; footprint Capacitor_SMD:C_0603_1608Metric -> Resistor_SMD:R_0603_1608Metric; symbol Device:C -> Device:R; MPN GRM188R71A106KA73D -> RC0603FR-0710KL; Manufacturer Murata -> Yageo
- U601: renamed from C611; value 4.7uF 50V -> TRI 20-1223; footprint Capacitor_SMD:C_1206_3216Metric -> CM5Carrier:TRACO_TRI20_DUAL; symbol Device:C -> CM5Carrier:TRI20_1223; MPN GRM31CR71H475KA12L -> TRI 20-1223; Manufacturer Murata -> TRACO Power
- U605: renamed from C671; value 1uF -> TPS7A2033PDBVR; footprint Capacitor_SMD:C_0603_1608Metric -> Package_TO_SOT_SMD:SOT-23-5; symbol Device:C -> CM5Carrier:TPS7A20DBV_A1; MPN GRM188R71A105KA61D -> TPS7A2033PDBVR; Manufacturer Murata -> Texas Instruments
Connections:
- net ADC_5V_A: now also R632.1, C632.1, R634.1, R670.1; no longer C630.1, C670.1, R630.1, R633.1
- net ADC_5V_ILIM: now also R630.1
- net ADC_5V_PG: now also R634.2; no longer C630.2
- net ADC_5V_PGFB: now also R632.2, R633.1; no longer R630.2, R631.1
- net ADC_5V_SET: now also C630.1, R631.1
- net AGND: now also C630.2, C650.2, C670.2, R611.2, R630.2, R650.2, U601.4 (COMMON), C603.2, C611.2, C613.2, C622.2, C623.2, C624.2, C631.2, C632.2, C651.2, C652.2, C673.2, R671.2; no longer C602.4 (COMMON), F601.2, L601.2, R610.2, R613.2, R632.2, R652.2
- net AKM_3V3_D: now also C671.1, C672.1, U605.5 (OUT); no longer U605.1
- net AUDIO_12V: now also C621.1, F601.2, U601.1 (+VIN), C603.1, C622.1; no longer C620.1, F601.1, R601.1, R612.1
- net AUDIO_12V_IN: now also F601.1
- net AUDIO_5V5_FB: now also R610.2, R611.1
- net AUDIO_5V5_NRSS: now also C620.1; no longer L601.1
- net AUDIO_5V5_PG: now also R613.2, U605.3 (EN); no longer R611.2
- net AUDIO_5V5_PRE: now also C670.1, L601.2, R610.1, U605.1 (IN), C623.1, C624.1, C631.1, C651.1; no longer C621.1, R611.1, R632.1, R652.1
- net AUDIO_5V5_SCONF: now also R612.1; no longer R610.1
- net AUDIO_5V5_SW: now also L601.1
- net AUDIO_N15V: now also U601.5 (-VOUT), C611.1, C613.1; no longer C602.5 (-VOUT), C610.1, U601.1
- net AUDIO_P15V: now also C610.1, U601.3 (+VOUT); no longer C602.3 (+VOUT)
- net DAC_5V_A: now also R652.1, C652.1, R654.1; no longer C650.1, R650.1, R653.1
- net DAC_5V_ILIM: now also R650.1
- net DAC_5V_PG: now also R654.2; no longer C650.2
- net DAC_5V_PGFB: now also R652.2, R653.1; no longer R650.2, R651.1
- net DAC_5V_SET: now also C650.1, R651.1
- net GND: now also R601.1
- net VCM_2V5: now also C673.1, R670.2, R671.1; no longer C670.2, C671.1, C672.1
Other:
- moved on the sheet: C610, C620, C621, F601, R610, R611, R630, R631, R650, R651
