File: cad/kicad/AUDIO-8X8/Audio-TDM-Clock.kicad_sch (KiCad schematic)
At the start: 18 parts, among them J101 AUDIO_TDM_CONTROL, U101 SN65LVDT2D, U102 SN65LVDT2D, U103 SN65LVDT2D, U104 SN65LVDT2D, U105 SN65LVDS1D

Commit message: Audit schematic logic against controlled datasheets
Parts:
- added C107: 100nF, Capacitor_SMD:C_0402_1005Metric, symbol Device:C
- added R117: 100k 1%, Resistor_SMD:R_0603_1608Metric, symbol Device:R
- added U106: SN74LVC1G11DBVR, Package_TO_SOT_SMD:SOT-23-6, symbol 74xGxx:74LVC1G11
Connections:
- net AGND: now also C107.2, R117.2, U106.2 (GND)
- net AKM_3V3_D: now also C107.1, U106.5 (VCC)
- net AUD_DAC_MUTE_N renamed AUD_DAC_MUTE_CMD_N
- net AUD_DAC_MUTE_CMD_N: now also U106.1
- new net ADC_5V_PG: U106.3
- new net AUDIO_SAFE_UNMUTE_N: R117.1, U106.4
- new net DAC_5V_PG: U106.6
Other:
- note added: "5. HARDWARE FAIL-SILENT GATE"
- note added: "Any power-good loss forces AUDIO_SAFE_UNMUTE_N low in hardware; R117 keeps mute/relays asserted if AKM_3V3_D is absent."
- note added: "SN74LVC1G11 inputs tolerate the 5 V PG pull-ups and Ioff prevents back-powering while its 3.3 V supply is off."
- note added: "U106 permits DAC unmute and relay closure only when the carrier command, ADC_5V_PG, and DAC_5V_PG are all high."
- note removed: "AUDIO_ENABLE is consumed by the local audio-power sequence; firmware releases resets only after all PG signals and clocks are valid."
- note removed: "Reset and mute default asserted while the harness is absent or the carrier is unpowered."

Commit message: Implement direct socketed dual-SIM daughterboard
Parts:
- removed R111, R112, R113: 10k 0.1%, Resistor_SMD:R_0603_1608Metric, symbol Device:R
- removed U101, U102, U103, U104: SN65LVDT2D, Package_SO:SOIC-8_3.9x4.9mm_P1.27mm, symbol Interface:SN65LVDT2D
- removed U105: SN65LVDS1D, Package_SO:SOIC-8_3.9x4.9mm_P1.27mm, symbol Interface:SN65LVDS1D
- added C101, C102, C103, C104, C105: 100nF, Capacitor_SMD:C_0402_1005Metric, symbol Device:C
- added R114: 10k 0.1%, Resistor_SMD:R_0603_1608Metric, symbol Device:R
- added R115, R116: 4.7k 0.1%, Resistor_SMD:R_0603_1608Metric, symbol Device:R
- R112: renamed from R115; value 4.7k 0.1% -> 10k 0.1%; MPN RC0603FR-074K7L -> RC0603FR-0710KL
- R113: renamed from R116; value 4.7k 0.1% -> 10k 0.1%; MPN RC0603FR-074K7L -> RC0603FR-0710KL
- U101: renamed from C101; value 100nF -> SN65LVDT2D; footprint Capacitor_SMD:C_0402_1005Metric -> Package_SO:SOIC-8_3.9x4.9mm_P1.27mm; symbol Device:C -> Interface:SN65LVDT2D; MPN C1005X7R1H104K050BB -> SN65LVDT2DR; Manufacturer TDK -> Texas Instruments
- U102: renamed from C102; value 100nF -> SN65LVDT2D; footprint Capacitor_SMD:C_0402_1005Metric -> Package_SO:SOIC-8_3.9x4.9mm_P1.27mm; symbol Device:C -> Interface:SN65LVDT2D; MPN C1005X7R1H104K050BB -> SN65LVDT2DR; Manufacturer TDK -> Texas Instruments
- U103: renamed from C103; value 100nF -> SN65LVDT2D; footprint Capacitor_SMD:C_0402_1005Metric -> Package_SO:SOIC-8_3.9x4.9mm_P1.27mm; symbol Device:C -> Interface:SN65LVDT2D; MPN C1005X7R1H104K050BB -> SN65LVDT2DR; Manufacturer TDK -> Texas Instruments
- U104: renamed from C104; value 100nF -> SN65LVDT2D; footprint Capacitor_SMD:C_0402_1005Metric -> Package_SO:SOIC-8_3.9x4.9mm_P1.27mm; symbol Device:C -> Interface:SN65LVDT2D; MPN C1005X7R1H104K050BB -> SN65LVDT2DR; Manufacturer TDK -> Texas Instruments
- U105: renamed from C105; value 100nF -> SN65LVDS1D; footprint Capacitor_SMD:C_0402_1005Metric -> Package_SO:SOIC-8_3.9x4.9mm_P1.27mm; symbol Device:C -> Interface:SN65LVDS1D; MPN C1005X7R1H104K050BB -> SN65LVDS1DR; Manufacturer TDK -> Texas Instruments
- renumbered R114 to R111
Connections:
- net ADC_TDM_OUT: now also U105.2 (D)
- net AGND: now also R112.2, R113.2, U101.5 (GND), U102.5 (GND), U103.5 (GND), U104.5 (GND), U105.4 (GND), C101.2, C102.2, C103.2, C104.2, C105.2, R114.2; no longer U101.2, U102.2, U103.2, U104.2, U105.2
- net AKM_3V3_D: now also U101.8 (V_{CC}), U102.8 (V_{CC}), U103.8 (V_{CC}), U104.8 (V_{CC}), C101.1, C102.1, C103.1, C104.1, C105.1, R115.1, R116.1; no longer R112.1, R113.1, U101.1, U102.1, U103.1, U104.1
- net AKM_BCLK: now also U102.7 (R)
- net AKM_FSYNC: now also U103.7 (R)
- net AKM_MCLK: now also U101.7 (R)
- net AUDIO_PRESENT_N: now also R114.1; no longer R111.1
- net AUD_ADC_RST_N: now also R111.1
- net AUD_ADC_SDOUT_N: now also U105.8 (Z)
- net AUD_ADC_SDOUT_P: now also U105.7 (Y)
- net AUD_BCLK_N: now also U102.1 (B)
- net AUD_BCLK_P: now also U102.2 (A)
- net AUD_DAC_MUTE_CMD_N: now also R113.1
- net AUD_DAC_RST_N: now also R112.1
- net AUD_DAC_SDIN_N: now also U104.1 (B)
- net AUD_DAC_SDIN_P: now also U104.2 (A)
- net AUD_FSYNC_N: now also U103.1 (B)
- net AUD_FSYNC_P: now also U103.2 (A)
- net AUD_I2C_SCL: now also R115.2; no longer R112.2
- net AUD_I2C_SDA: now also R116.2; no longer R113.2
- net AUD_MCLK_N: now also U101.1 (B)
- net AUD_MCLK_P: now also U101.2 (A)
- net DAC_TDM_IN: now also U104.7 (R)
Other:
- moved on the sheet: R111, R112, R113
Changed lines of the file:
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@@
 		(instances
 			(project "Audio-TDM-Clock"
-				(path "/266cf186-0dff-5dda-b52b-b921157a0ebd"
+				(path "/eeb072c8-d9a3-536f-abab-dce987f4da60"
 					(reference "J101")
 					(unit 1)
@@
 		(instances
 			(project "Audio-TDM-Clock"
-				(path "/266cf186-0dff-5dda-b52b-b921157a0ebd"
+				(path "/eeb072c8-d9a3-536f-abab-dce987f4da60"
 					(reference "U101")
 					(unit 1)
@@
 		(instances
 			(project "Audio-TDM-Clock"
-				(path "/266cf186-0dff-5dda-b52b-b921157a0ebd"
+				(path "/eeb072c8-d9a3-536f-abab-dce987f4da60"
 					(reference "C101")
 					(unit 1)
@@
 		(instances
 			(project "Audio-TDM-Clock"
-				(path "/266cf186-0dff-5dda-b52b-b921157a0ebd"
+				(path "/eeb072c8-d9a3-536f-abab-dce987f4da60"
 					(reference "U102")
 					(unit 1)
@@
 		(instances
 			(project "Audio-TDM-Clock"
-				(path "/266cf186-0dff-5dda-b52b-b921157a0ebd"
+				(path "/eeb072c8-d9a3-536f-abab-dce987f4da60"
 					(reference "C102")
 					(unit 1)
@@
 		(instances
 			(project "Audio-TDM-Clock"
-				(path "/266cf186-0dff-5dda-b52b-b921157a0ebd"
+				(path "/eeb072c8-d9a3-536f-abab-dce987f4da60"
 					(reference "U103")
 					(unit 1)
@@
 		(instances
 			(project "Audio-TDM-Clock"
-				(path "/266cf186-0dff-5dda-b52b-b921157a0ebd"
+				(path "/eeb072c8-d9a3-536f-abab-dce987f4da60"
 					(reference "C103")
 					(unit 1)
@@
 		(instances
 			(project "Audio-TDM-Clock"
-				(path "/266cf186-0dff-5dda-b52b-b921157a0ebd"
+				(path "/eeb072c8-d9a3-536f-abab-dce987f4da60"
 					(reference "U104")
 					(unit 1)
@@
 		(instances
 			(project "Audio-TDM-Clock"
-				(path "/266cf186-0dff-5dda-b52b-b921157a0ebd"
+				(path "/eeb072c8-d9a3-536f-abab-dce987f4da60"
 					(reference "C104")
 					(unit 1)
@@
 		(instances
 			(project "Audio-TDM-Clock"
-				(path "/266cf186-0dff-5dda-b52b-b921157a0ebd"
+				(path "/eeb072c8-d9a3-536f-abab-dce987f4da60"
 					(reference "U105")
 					(unit 1)
@@
 		(instances
 			(project "Audio-TDM-Clock"
-				(path "/266cf186-0dff-5dda-b52b-b921157a0ebd"
+				(path "/eeb072c8-d9a3-536f-abab-dce987f4da60"
 					(reference "C105")
 					(unit 1)
@@
 		(instances
 			(project "Audio-TDM-Clock"
-				(path "/266cf186-0dff-5dda-b52b-b921157a0ebd"
+				(path "/eeb072c8-d9a3-536f-abab-dce987f4da60"
 					(reference "C106")
 					(unit 1)
@@
 		(instances
 			(project "Audio-TDM-Clock"
-				(path "/266cf186-0dff-5dda-b52b-b921157a0ebd"
+				(path "/eeb072c8-d9a3-536f-abab-dce987f4da60"
 					(reference "R111")
 					(unit 1)
@@
 		(instances
 			(project "Audio-TDM-Clock"
-				(path "/266cf186-0dff-5dda-b52b-b921157a0ebd"
+				(path "/eeb072c8-d9a3-536f-abab-dce987f4da60"
 					(reference "R112")
 					(unit 1)
@@
 		(instances
 			(project "Audio-TDM-Clock"
-				(path "/266cf186-0dff-5dda-b52b-b921157a0ebd"
+				(path "/eeb072c8-d9a3-536f-abab-dce987f4da60"
 					(reference "R113")
 					(unit 1)
@@
 		(instances
 			(project "Audio-TDM-Clock"
-				(path "/266cf186-0dff-5dda-b52b-b921157a0ebd"
+				(path "/eeb072c8-d9a3-536f-abab-dce987f4da60"
 					(reference "R114")
 					(unit 1)
@@
 		(instances
 			(project "Audio-TDM-Clock"
-				(path "/266cf186-0dff-5dda-b52b-b921157a0ebd"
+				(path "/eeb072c8-d9a3-536f-abab-dce987f4da60"
 					(reference "R115")
 					(unit 1)
@@
 		(instances
 			(project "Audio-TDM-Clock"
-				(path "/266cf186-0dff-5dda-b52b-b921157a0ebd"
+				(path "/eeb072c8-d9a3-536f-abab-dce987f4da60"
 					(reference "R116")
 					(unit 1)
@@
 		(instances
 			(project "Audio-TDM-Clock"
-				(path "/266cf186-0dff-5dda-b52b-b921157a0ebd"
+				(path "/eeb072c8-d9a3-536f-abab-dce987f4da60"
 					(reference "U106")
 					(unit 1)
@@
 		(instances
 			(project "Audio-TDM-Clock"
-				(path "/266cf186-0dff-5dda-b52b-b921157a0ebd"
+				(path "/eeb072c8-d9a3-536f-abab-dce987f4da60"
 					(reference "R117")
 					(unit 1)
@@
 		(instances
 			(project "Audio-TDM-Clock"
-				(path "/266cf186-0dff-5dda-b52b-b921157a0ebd"
+				(path "/eeb072c8-d9a3-536f-abab-dce987f4da60"
 					(reference "C107")
 					(unit 1)
@@
 		(instances
 			(project "Audio-TDM-Clock"
-				(path "/266cf186-0dff-5dda-b52b-b921157a0ebd"
+				(path "/eeb072c8-d9a3-536f-abab-dce987f4da60"
 					(reference "#FLG0101")
 					(unit 1)
