File: cad/kicad/CM5-CARRIER/CM5-Carrier.kicad_pcb (KiCad board)
At the start: 10 copper layers, 166 x 268 mm, 513 parts, among them J102 PWR_STATUS_FROM_SELECTOR, J1021 FFB0412EN-00Y2E CPU FAN, J1022 AFB0412SHB-SP04 MODEM FAN, J1023 THA0412AD-TZW3 INTAKE, J1024 THA0412AD-TZW3 EXHAUST, J103 PWR_TELEMETRY_FROM_SELECTOR, J1060 STATUS_LAMP_PANEL_HARNESS, J1070 NIGHT_LIGHT_PANEL_HARNESS, J1100 RAW_POWER_FROM_PWR_SELECT, J202 AUDIO_12V_POWER, J501 RADXA CM5 U13-A MATE, J502 RADXA CM5 U13-B MATE, J503 RADXA CM5 J1 MATE, J510 CM5_POWER_SERVICE, J511 DEBUG_UART_3V3, J512 INTERNAL_USB_RECOVERY, J513 CM5_POWER_ENTRY, J610 74991114412, J611 74991114412, J612 74991114412, J613 74991114412, J620 AW7915-NP1_WIFI6_4T4R, J701 WWAN_M2_B_KEY_USB3_USB2, J702 693043020611, J703 693043020611, J801 HDMI_TO_LID_DISPLAY, J802 TOUCH_USB_HOST, J803 LID_DISPLAY_12V, J901 AUDIO_8X8_TDM_CONTROL, J910 STX-353K7A-6N-KTTR, Q1060 2N7002K-7, Q1061 2N7002K-7, Q1062 2N7002K-7, Q1063 2N7002K-7, Q1064 2N7002K-7, Q1065 2N7002K-7, Q1110 NVMFS6B25NL, Q1111 FDWS86068-F085, Q1120 CSD18532Q5B, Q1121 CSD18532Q5B, Q1122 CSD17573Q5B, Q1123 CSD17573Q5B, U1000 PCA9306DP, U1001 TCA9535PWR_0x20, U1002 TCA9535PWR_0x21, U1003 TCA9535PWR_0x22, U1020 EMC2305-1-AP-TR, U1050 TMP117_CM5, U1051 TMP117_MODEM, U1052 TMP117_BOARD_POWER, U1110 LM5146RGYR, U1120 LM5176PWP, U1130 LM61460RJR, U1131 TPS259827LNRGER, U1140 LM61440RJR, U1141 TPS22990DMLR, U1150 LM61440RJR, U1160 LM61440RJR, U1170 TPS62913RPU, U1171 TPS62913RPU, U601 PI7C9X2G608GP, U606 SN74LVC1G11DBVR, U611 LAN7430, U612 LAN7430, U613 LAN7430, U630 TPD4E05U06DQA, U631 TPD4E05U06DQA, U632 TPD4E05U06DQA, U633 TPD4E05U06DQA, U634 TPD4E05U06DQA, U635 TPD4E05U06DQA, U636 TPD4E05U06DQA, U637 TPD4E05U06DQA, U702 TPD4E05U06DQA, U703 TPD4E05U06DQA, U704 FSA2567MPX, U705 TPD3F303DPV, U706 TPD3F303DPV, U801 TPD4E05U06DQA, U802 TPD4E05U06DQA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

Commit message: Fix PCB-A1 in-board 3D placement
Parts:
- moved F1182 483.6 mm to (5.73, 185.4)
- moved R6132 471.6 mm to (8.03, 13.3)
- moved R6131 469.2 mm to (3.52, 13.3)
- moved C11715 464.6 mm to (3.75, 197.5)
- moved C1133 463.5 mm to (28.3, 190.1)
- moved R1137 452.5 mm to (8.03, 200.8)
- moved J512 451.7 mm to (39.4, 229.8)
- moved C1135 450.9 mm to (57.3, 190.1)
- moved R1134 450.0 mm to (3.52, 200.8)
- moved C1134 449.4 mm to (51.3, 190.1)
- moved C1136 443.5 mm to (76.3, 198.0), turned to 90 degrees
- moved R1141 443.1 mm to (45.5, 201.3)
- moved R1140 440.7 mm to (41.0, 201.3)
- moved J510 438.3 mm to (26.5, 229.8)
- moved C810 433.0 mm to (39.7, 125.5)
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Other:
- board text added: "CM5-CARRIER PCB-A1"
- board text added: "F.Cu CM5 SUPPORT; CM5 MATE LOCKED ON B.Cu"
- board text added: "F.Cu NETWORK"
- board text added: "F.Cu POWER CONVERSION"
- board text added: "F.Cu SERVICE / WWAN / DISPLAY / AUDIO / THERMAL"
- board text removed: "CM5-CARRIER PCB-A0"
- board text removed: "HEADSET / FAN / SENSOR CANDIDATE ZONE"
- board text removed: "POWER ZONES - PLACEMENT NOT LOCKED"
- board text removed: "UNPLACED / UNVERIFIED PCB FOOTPRINT STAGING - NOT BOARD GEOMETRY"

Commit message: Implement direct socketed dual-SIM daughterboard
Parts:
- removed J703: 693043020611, CM5Carrier:J_Wurth_WR-CRD_693043020611
- removed U705, U706: TPD3F303DPV, Package_SON:Texas_R-PUSON-N8_USON-8-1EP_1.6x2.1mm_P0.5mm_EP0.4x1.7mm
- added SD1: M3_CAPTIVE_SUPPORT_3.4, ProCommMechanical:ProComm_M3_Support_NPTH_3.4mm, F.Cu at (57.0, 93.5)
- added SD2: M3_CAPTIVE_SUPPORT_3.4, ProCommMechanical:ProComm_M3_Support_NPTH_3.4mm, F.Cu at (122.0, 93.5)
- added SD3: M3_CAPTIVE_SUPPORT_3.4, ProCommMechanical:ProComm_M3_Support_NPTH_3.4mm, F.Cu at (78.5, 122.5)
- added SD4: M3_CAPTIVE_SUPPORT_3.4, ProCommMechanical:ProComm_M3_Support_NPTH_3.4mm, F.Cu at (100.5, 122.5)
- J610, J611, J612, J613: value 74991114412 -> V8BR-1AX1-GH; footprint CM5Carrier:T_Wurth_WE-RJ45LAN_74991114412 -> CM5Carrier:Bel_V8BR_1AX1_GH
- J702: value 693043020611 -> DUAL_SIM_B2B_PLUG; footprint CM5Carrier:J_Wurth_WR-CRD_693043020611 -> CM5Carrier:Hirose_DF40C-20DP-0.4V_2x10-1MP_P0.4mm
- moved C919 138.7 mm to (17.0, 123.7), turned to 90 degrees
- moved R1003 138.0 mm to (154.3, 131.5)
- moved R1001 132.8 mm to (146.0, 130.8), turned to 0 degrees
- moved C1012 128.8 mm to (17.8, 128.0), turned to 90 degrees
- moved Q1063 121.5 mm to (3.98, 124.2)
- moved C905 119.5 mm to (142.0, 136.5)
- moved C906 119.5 mm to (145.0, 136.5)
- moved C907 119.5 mm to (148.0, 136.5)
- moved R1005 116.0 mm to (26.0, 131.3)
- moved R1006 116.0 mm to (30.5, 131.3)
- moved R1063 115.0 mm to (21.5, 134.3)
- moved R1064 115.0 mm to (26.0, 134.3)
- moved R1065 115.0 mm to (30.5, 134.3)
- moved U1002 114.1 mm to (119.9, 115.2)
- moved C1013 112.3 mm to (38.8, 128.0), turned to 90 degrees
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Connections:
- J610 pad 10: (no net) -> WAN1_MDI0_N
- J610 pad 11: WAN1_LED_A1 -> WAN1_MDI0_P
- J610 pad 12: WAN1_LED0 -> GND
- J610 pad 13: WAN1_LED_A2 -> unconnected-(J610-VC12-Pad13)
- J610 pad 14: WAN1_LED1 -> unconnected-(J610-VC36-Pad14)
- J610 pad 2: WAN1_MDI0_P -> WAN1_MDI2_N
- J610 pad 3: WAN1_MDI0_N -> WAN1_MDI2_P
- J610 pad 6: WAN1_MDI2_P -> GND
- J610 pad 7: WAN1_MDI2_N -> GND
- J611 pad 10: (no net) -> WAN2_MDI_A_N
- J611 pad 11: WAN2_LED_A1 -> WAN2_MDI_A_P
- J611 pad 12: WAN2_LED0 -> GND
- J611 pad 13: WAN2_LED_A2 -> unconnected-(J611-VC12-Pad13)
- J611 pad 14: WAN2_LED1 -> unconnected-(J611-VC36-Pad14)
- J611 pad 2: WAN2_MDI_A_P -> WAN2_MDI_C_N
- J611 pad 3: WAN2_MDI_A_N -> WAN2_MDI_C_P
- J611 pad 6: WAN2_MDI_C_P -> GND
- J611 pad 7: WAN2_MDI_C_N -> GND
- J612 pad 10: (no net) -> LAN1_MDI_A_N
- J612 pad 11: LAN1_LED_A1 -> LAN1_MDI_A_P
- J612 pad 12: LAN1_LED0 -> GND
- J612 pad 13: LAN1_LED_A2 -> unconnected-(J612-VC12-Pad13)
- J612 pad 14: LAN1_LED1 -> unconnected-(J612-VC36-Pad14)
- J612 pad 2: LAN1_MDI_A_P -> LAN1_MDI_C_N
- J612 pad 3: LAN1_MDI_A_N -> LAN1_MDI_C_P
- J612 pad 6: LAN1_MDI_C_P -> GND
- J612 pad 7: LAN1_MDI_C_N -> GND
- J613 pad 10: (no net) -> LAN2_MDI_A_N
- J613 pad 11: LAN2_LED_A1 -> LAN2_MDI_A_P
- J613 pad 12: LAN2_LED0 -> GND
- J613 pad 13: LAN2_LED_A2 -> unconnected-(J613-VC12-Pad13)
- J613 pad 14: LAN2_LED1 -> unconnected-(J613-VC36-Pad14)
- J613 pad 2: LAN2_MDI_A_P -> LAN2_MDI_C_N
- J613 pad 3: LAN2_MDI_A_N -> LAN2_MDI_C_P
- J613 pad 6: LAN2_MDI_C_P -> GND
- J613 pad 7: LAN2_MDI_C_N -> GND
Other:
- board text added: "LOCKED VERTICAL BEL RJ45 BODY CENTERS"
- board text removed: "LOCKED RJ45 BODY CENTERS"
