File: cad/kicad/CM5-CARRIER/Power-Regulators-A1.kicad_sch (KiCad schematic)
At the start: 198 parts, among them J1100 RAW_POWER_FROM_PWR_SELECT, Q1110 NVMFS6B25NL, Q1111 FDWS86068-F085, Q1120 CSD18532Q5B, Q1121 CSD18532Q5B, Q1122 CSD17573Q5B, Q1123 CSD17573Q5B, U1110 LM5146RGYR, U1120 LM5176PWP, U1130 LM61460RJR, U1131 TPS259827LNRGER, U1140 LM61440RJR, U1141 TPS22990DMLR, U1150 LM61440RJR, U1160 LM61440RJR, U1170 TPS62913RPU, U1171 TPS62913RPU, U1172 TPS62913RPU, U1173 TPS62913RPU, U1180 TRI 20-1223 ON AUDIO-8X8, U1181 TPS7A2050PDBVR, U1182 TPS7A2050PDBVR, U1183 TPS7A2033PDBVR, U1184 TPS7A2018PDBVR

Commit message: Complete A1 detailed carrier and audio capture
Parts:
- removed C1100, C1101, C1102, C1103: 5600uF 50V, symbol Device:C_Polarized
- removed C1104, C1105, C1106, C1107: 5600uF 50V DNP, symbol Device:C_Polarized
- removed C1108: 2200uF 50V DNP, symbol Device:C_Polarized
- removed C1113, C1114, C1115, C1116, C1117: 47uF 6.3V X7R, symbol Device:C
- removed C1118: 100nF 25V X7R, symbol Device:C
- removed C1119: 4.7uF 10V X7R, symbol Device:C
- removed C1130, C1140: 100nF, symbol Device:C
- removed C1135: 47uF X7R, symbol Device:C
- removed C1136: 1uF 10V X7R, symbol Device:C
- removed C11700, C11710, C11720: 470nF, symbol Device:C
- removed C11701, C11702, C11703, C11712, C11713, C11721, C11722, C11723: 22uF 10V X7R, symbol Device:C
- removed C11704, C11705, C11715, C11724, C11725: 10uF 25V X7R, symbol Device:C
- removed C11802, C11803, C11804, C11805, C11806, C11807: 1uF X7R, symbol Device:C
- removed C1194, C1195, C1196, C1197: 4.7uF 50V X7R, symbol Device:C
- removed L1110: 3.3uH / 28.6A, symbol Device:L
- removed L1130, L1140: 4.7uH / 15.2A Isat, symbol Device:L
- removed L11700: 2.2uH / 2.0A rail, symbol Device:L
- removed L11710: 2.2uH / 1.5A rail, symbol Device:L
- removed L11720: 2.2uH / 1.0A rail, symbol Device:L
- removed Q1120: CSD18532Q5B, symbol Transistor_FET:Q_NMOS_GSD
- removed Q1123: CSD17573Q5B, symbol Transistor_FET:Q_NMOS_GSD
- removed R1130, R1140: 33.2k / 400kHz, symbol Device:R
- removed R1132: 35.7k 0.1%, symbol Device:R
- removed R1133, R1143: 0R RBOOT, symbol Device:R
- removed R1138: 255R 1% / 6A ILIM, symbol Device:R
- removed R1141: 100k 0.1%, symbol Device:R
- removed R1142: 43.2k 0.1%, symbol Device:R
- removed R11700: 1.24k 0.1%, symbol Device:R
- removed R11701, R11721: 4.99k 0.1%, symbol Device:R
- removed R11702, R11712, R11722: 7.5k S-CONF, symbol Device:R
- removed R11710: 6.19k 0.1%, symbol Device:R
- removed R11720: 15.6k 0.1%, symbol Device:R
- removed U1130: LM61460RJR, symbol CM5Carrier:LM61460RJR
- removed U1140: LM61440RJR, symbol CM5Carrier:LM61440RJR
- removed U1183: TPS7A2033PDBVR, Package_TO_SOT_SMD:SOT-23-5, symbol CM5Carrier:TPS7A20DBV_A1
- removed U1184: TPS7A2018PDBVR, Package_TO_SOT_SMD:SOT-23-5, symbol CM5Carrier:TPS7A20DBV_A1
- added C1124, C1125, C1126, C1127: 330uF 16V polymer, Capacitor_SMD:CP_Elec_10x12.6, symbol Device:C_Polarized
- added C1128, C1129: 100nF 25V, Capacitor_SMD:C_0603_1608Metric, symbol Device:C
- added C1131, C1152, C1162: 4.7uF 50V, Capacitor_SMD:C_1206_3216Metric, symbol Device:C
- added C1153, C1154, C1163, C1164, C1165: 47uF X7R, Capacitor_SMD:C_1210_3225Metric, symbol Device:C
- added C1156, C1166: 1uF 10V X7R, Capacitor_SMD:C_0603_1608Metric, symbol Device:C
- added C1200: 4.7uF 10V, Capacitor_SMD:C_0805_2012Metric, symbol Device:C
- added C1201: 2.2nF, Capacitor_SMD:C_0603_1608Metric, symbol Device:C
- added C1202: 4.7uF 50V X7R, Capacitor_SMD:C_1206_3216Metric, symbol Device:C
- added D1120, D1121: BAT54WS, Diode_SMD:D_SOD-323, symbol Device:D_Schottky
- added F1183: 0.25A fast, Fuse:Fuse_Littelfuse-NANO2-451_453, symbol Device:Fuse
- added F1184: 3A time-lag, Fuse:Fuse_Littelfuse-NANO2-451_453, symbol Device:Fuse
- added L1160: 4.7uH / 15.2A Isat, Inductor_SMD:L_Coilcraft_XAL7070-XXX, symbol Device:L
- added R1128: 10k 1%, Resistor_SMD:R_0603_1608Metric, symbol Device:R
- added R1151, R1161: 100k 0.1%, Resistor_SMD:R_0603_1608Metric, symbol Device:R
- added R1160: 33.2k / 400kHz, Resistor_SMD:R_0603_1608Metric, symbol Device:R
- added U1131: TPS259827LNRGER, Package_DFN_QFN:Texas_RGE0024H_VQFN-24-1EP_4x4mm_P0.5mm_EP2.7x2.7mm_ThermalVias, symbol CM5Carrier:TPS259827LNRGE
- added U1160: LM61440RJR, CM5Carrier:TI_RJR0014A, symbol CM5Carrier:LM61440RJR
- added U1180: TRI 20-1223 ON AUDIO-8X8, CM5Carrier:TRACO_TRI20_DUAL, symbol CM5Carrier:TRI20_1223
- C1109: footprint (none) -> Capacitor_SMD:C_1206_3216Metric; MPN (none) -> GRM31CR71H105KA61L; Manufacturer (none) -> Murata
- C1110, C1111, C1112, C1146: footprint (none) -> Capacitor_SMD:C_0603_1608Metric
- C1113: renamed from C1128; value 100nF 25V -> 47uF 6.3V X7R; footprint (none) -> Capacitor_SMD:C_1210_3225Metric; MPN (none) -> GCM32ER70J476KE19L; Manufacturer (none) -> Murata
- C1114: renamed from C1129; value 100nF 25V -> 47uF 6.3V X7R; footprint (none) -> Capacitor_SMD:C_1210_3225Metric; MPN (none) -> GCM32ER70J476KE19L; Manufacturer (none) -> Murata
- C1115: renamed from C1200; value 4.7uF 10V -> 47uF 6.3V X7R; footprint (none) -> Capacitor_SMD:C_1210_3225Metric; MPN (none) -> GCM32ER70J476KE19L; Manufacturer (none) -> Murata
- C1116: renamed from C1201; value 2.2nF -> 47uF 6.3V X7R; footprint (none) -> Capacitor_SMD:C_1210_3225Metric; MPN (none) -> GCM32ER70J476KE19L; Manufacturer (none) -> Murata
- C1117: renamed from C1124; value 330uF 16V polymer -> 47uF 6.3V X7R; footprint (none) -> Capacitor_SMD:C_1210_3225Metric; symbol Device:C_Polarized -> Device:C; MPN 16SVP330M -> GCM32ER70J476KE19L; Manufacturer Panasonic -> Murata
- C1118: renamed from C1125; value 330uF 16V polymer -> 100nF 25V X7R; footprint (none) -> Capacitor_SMD:C_0603_1608Metric; symbol Device:C_Polarized -> Device:C; MPN 16SVP330M -> GRM188R71E104KA01D; Manufacturer Panasonic -> Murata
- C1119: renamed from C1126; value 330uF 16V polymer -> 4.7uF 10V X7R; footprint (none) -> Capacitor_SMD:C_0805_2012Metric; symbol Device:C_Polarized -> Device:C; MPN 16SVP330M -> GRM21BR71A475KA73L; Manufacturer Panasonic -> Murata
- C1120: footprint (none) -> Capacitor_SMD:C_0603_1608Metric; MPN (none) -> GRM1885C1H221JA01D; Manufacturer (none) -> Murata
- C1121, C1150, C1160: footprint (none) -> Capacitor_SMD:C_0603_1608Metric; MPN (none) -> GRM188R71E104KA01D; Manufacturer (none) -> Murata
- C1122: footprint (none) -> Capacitor_SMD:C_0603_1608Metric; MPN (none) -> GRM188R71H333KA01D; Manufacturer (none) -> Murata
- C1123: footprint (none) -> Capacitor_SMD:C_0603_1608Metric; MPN (none) -> GRM1885C1H561JA01D; Manufacturer (none) -> Murata
- C1130: renamed from C1156; value 1uF 10V X7R -> 100nF; footprint (none) -> Capacitor_SMD:C_0603_1608Metric; MPN GRM188R71A105KA61D -> GRM188R71E104KA01D
- C1132, C1141, C1142, C1151, C1161: footprint (none) -> Capacitor_SMD:C_1206_3216Metric; MPN (none) -> GRM31CR71H475KA12L; Manufacturer (none) -> Murata
- C1133, C1134, C1143, C1144, C1145: footprint (none) -> Capacitor_SMD:C_1210_3225Metric
- C1135: renamed from L1160; value 4.7uH / 15.2A Isat -> 47uF X7R; footprint (none) -> Capacitor_SMD:C_1210_3225Metric; symbol Device:L -> Device:C; MPN XAL7070-472MEC -> GRM32ER71A476KE15L; Manufacturer Coilcraft -> Murata
- C1136: renamed from R1160; value 33.2k / 400kHz -> 1uF 10V X7R; footprint (none) -> Capacitor_SMD:C_0603_1608Metric; symbol Device:R -> Device:C; MPN (none) -> GRM188R71A105KA61D; Manufacturer (none) -> Murata
- C1138: footprint (none) -> Capacitor_SMD:C_0603_1608Metric; MPN (none) -> GRM188R71H472KA01D; Manufacturer (none) -> Murata
- C1140: renamed from C1166; value 1uF 10V X7R -> 100nF; footprint (none) -> Capacitor_SMD:C_0603_1608Metric; MPN GRM188R71A105KA61D -> GRM188R71E104KA01D
- C1149, C1210: footprint (none) -> Capacitor_SMD:C_0603_1608Metric; MPN (none) -> GRM188R71H103KA01D; Manufacturer (none) -> Murata
- C1155: renamed from U1170; value TPS62913RPU -> 47uF X7R; footprint Package_DFN_QFN:Texas_RPU0010A_VQFN-HR-10_2x2mm_P0.5mm -> Capacitor_SMD:C_1210_3225Metric; symbol CM5Carrier:TPS62913RPU -> Device:C; MPN TPS62913RPUT -> GRM32ER71A476KE15L; Manufacturer Texas Instruments -> Murata
- C11700: renamed from C11730; footprint (none) -> Capacitor_SMD:C_0603_1608Metric; MPN (none) -> GRM188R71E474KA12D; Manufacturer (none) -> Murata
- C11701: renamed from C11731; footprint (none) -> Capacitor_SMD:C_0805_2012Metric
- C11702: renamed from C11732; footprint (none) -> Capacitor_SMD:C_0805_2012Metric
- C11703: renamed from C11733; footprint (none) -> Capacitor_SMD:C_0805_2012Metric
- C11704: renamed from C11734; footprint (none) -> Capacitor_SMD:C_0805_2012Metric
- C11705: renamed from C11735; footprint (none) -> Capacitor_SMD:C_0805_2012Metric
- C11710: renamed from U1180; value TRI 20-1223 ON AUDIO-8X8 -> 470nF; footprint (none) -> Capacitor_SMD:C_0603_1608Metric; symbol CM5Carrier:TRI20_1223 -> Device:C; MPN TRI 20-1223 -> GRM188R71E474KA12D; Manufacturer TRACO Power -> Murata
- C11711, C11714: footprint (none) -> Capacitor_SMD:C_0805_2012Metric
- C11712: renamed from C11800; value 1uF X7R -> 22uF 10V X7R; footprint (none) -> Capacitor_SMD:C_0805_2012Metric; MPN (none) -> GRM21BR71A226ME44L; Manufacturer (none) -> Murata
- C11713: renamed from C11801; value 1uF X7R -> 22uF 10V X7R; footprint (none) -> Capacitor_SMD:C_0805_2012Metric; MPN (none) -> GRM21BR71A226ME44L; Manufacturer (none) -> Murata
- C11715: renamed from U1181; value TPS7A2050PDBVR -> 10uF 25V X7R; footprint Package_TO_SOT_SMD:SOT-23-5 -> Capacitor_SMD:C_0805_2012Metric; symbol CM5Carrier:TPS7A20DBV_A1 -> Device:C; MPN TPS7A2050PDBVR -> GRM21BR71E106KA73L; Manufacturer Texas Instruments -> Murata
- C1189, C1190, C1191, C1192: footprint (none) -> Capacitor_SMD:CP_Elec_10x7.9; MPN 6SVPE330M -> 6SVP330M
- C1193: footprint (none) -> Capacitor_SMD:CP_Elec_8x11.9; MPN 6SVPE470M -> 6SVP470M
- C1194: renamed from C1127; value 330uF 16V polymer -> 4.7uF 50V X7R; footprint (none) -> Capacitor_SMD:C_1206_3216Metric; symbol Device:C_Polarized -> Device:C; MPN 16SVP330M -> GRM31CR71H475KA12L; Manufacturer Panasonic -> Murata
- C1195: renamed from D1120; value BAT54WS -> 4.7uF 50V X7R; footprint (none) -> Capacitor_SMD:C_1206_3216Metric; symbol Device:D_Schottky -> Device:C; MPN BAT54WS-7-F -> GRM31CR71H475KA12L; Manufacturer Diodes Incorporated -> Murata
- C1196: renamed from D1121; value BAT54WS -> 4.7uF 50V X7R; footprint (none) -> Capacitor_SMD:C_1206_3216Metric; symbol Device:D_Schottky -> Device:C; MPN BAT54WS-7-F -> GRM31CR71H475KA12L; Manufacturer Diodes Incorporated -> Murata
- C1197: renamed from C1202; footprint (none) -> Capacitor_SMD:C_1206_3216Metric
- C1203, C1204, C1205: footprint (none) -> Capacitor_SMD:C_1206_3216Metric
- F1180, F1181, F1182: footprint (none) -> Fuse:Fuse_Littelfuse-NANO2-451_453
- L1110: renamed from R1128; value 10k 1% -> 3.3uH / 29.2A Isat; footprint (none) -> CM5Carrier:TDK_SPM10065VC; symbol Device:R -> Device:L; MPN (none) -> SPM10065VC-3R3M-D; Manufacturer (none) -> TDK
- L1120: footprint (none) -> CM5Carrier:Wurth_74439370047
- L1130: renamed from C1152; value 4.7uF 50V -> 4.7uH / 15.2A Isat; footprint (none) -> Inductor_SMD:L_Coilcraft_XAL7070-XXX; symbol Device:C -> Device:L; MPN (none) -> XAL7070-472MEC; Manufacturer (none) -> Coilcraft
- L1140: renamed from C1162; value 4.7uF 50V -> 4.7uH / 15.2A Isat; footprint (none) -> Inductor_SMD:L_Coilcraft_XAL7070-XXX; symbol Device:C -> Device:L; MPN (none) -> XAL7070-472MEC; Manufacturer (none) -> Coilcraft
- L1150: footprint (none) -> Inductor_SMD:L_Coilcraft_XAL7070-XXX
- L11700: renamed from L11730; value 2.2uH / 1.0A rail -> 2.2uH / 2.0A rail; footprint (none) -> Inductor_SMD:L_Coilcraft_XxL4040
- L11710: renamed from F1183; value 0.25A fast -> 2.2uH / 1.5A rail; footprint (none) -> Inductor_SMD:L_Coilcraft_XxL4040; symbol Device:Fuse -> Device:L; MPN 0453.250MR -> XGL4030-222MEC; Manufacturer Littelfuse -> Coilcraft
- Q1110: footprint (none) -> CM5Carrier:onsemi_DFN5_5x6_488AA_GSD
- Q1111: footprint (none) -> CM5Carrier:onsemi_DFNW8_5p2x6p3_507AU_GSD
- Q1120: renamed from R1131; value 100k 0.1% -> CSD18532Q5B; footprint (none) -> CM5Carrier:TI_DNK0008A_GSD; symbol Device:R -> Transistor_FET:Q_NMOS_GSD; MPN (none) -> CSD18532Q5B; Manufacturer (none) -> Texas Instruments
- Q1121, Q1122: footprint (none) -> CM5Carrier:TI_DNK0008A_GSD
- Q1123: renamed from C1131; value 4.7uF 50V -> CSD17573Q5B; footprint (none) -> CM5Carrier:TI_DNK0008A_GSD; symbol Device:C -> Transistor_FET:Q_NMOS_GSD; MPN (none) -> CSD17573Q5B; Manufacturer (none) -> Texas Instruments
- R1110, R1111, R1112, R1113, R1114, R1115, R1116, R1153, R1163: footprint (none) -> Resistor_SMD:R_0603_1608Metric
- R1120: footprint (none) -> CM5Carrier:Susumu_KRL6432E_6mR
- R1121: footprint (none) -> Resistor_SMD:R_0603_1608Metric; MPN (none) -> RC0603FR-0727K4L; Manufacturer (none) -> Yageo
- R1122: footprint (none) -> Resistor_SMD:R_0603_1608Metric; MPN (none) -> RC0603FR-0793K1L; Manufacturer (none) -> Yageo
- R1123: footprint (none) -> Resistor_SMD:R_0603_1608Metric; MPN (none) -> TNPW0603280KBEEA; Manufacturer (none) -> Vishay
- R1124: footprint (none) -> Resistor_SMD:R_0603_1608Metric; MPN (none) -> TNPW060320K0BEEA; Manufacturer (none) -> Vishay
- R1125: footprint (none) -> Resistor_SMD:R_0603_1608Metric; MPN (none) -> RC0603FR-0710KL; Manufacturer (none) -> Yageo
- R1126: footprint (none) -> CM5Carrier:Susumu_KRL11050_4mR
- R1127: footprint (none) -> Resistor_SMD:R_0603_1608Metric; MPN (none) -> RC0603FR-0773K2L; Manufacturer (none) -> Yageo
- R1130: renamed from C1153; value 47uF X7R -> 33.2k / 400kHz; footprint (none) -> Resistor_SMD:R_0603_1608Metric; symbol Device:C -> Device:R; MPN GRM32ER71A476KE15L -> RC0603FR-0733K2L; Manufacturer Murata -> Yageo
- R1131: renamed from C1154; value 47uF X7R -> 100k 0.1%; footprint (none) -> Resistor_SMD:R_0603_1608Metric; symbol Device:C -> Device:R; MPN GRM32ER71A476KE15L -> TNPW0603100KBEEA; Manufacturer Murata -> Vishay
- R1132: renamed from C1155; value 47uF X7R -> 35.7k 0.1%; footprint (none) -> Resistor_SMD:R_0603_1608Metric; symbol Device:C -> Device:R; MPN GRM32ER71A476KE15L -> TNPW060335K7BEEA; Manufacturer Murata -> Vishay
- R1133: renamed from U1160; value LM61440RJR -> 0R RBOOT; footprint (none) -> Resistor_SMD:R_0603_1608Metric; symbol CM5Carrier:LM61440RJR -> Device:R; MPN LM61440RJR -> RC0603JR-070RL; Manufacturer Texas Instruments -> Yageo
- R1138: renamed from U1172; value TPS62913RPU -> 255R 1% / 6A ILIM; footprint Package_DFN_QFN:Texas_RPU0010A_VQFN-HR-10_2x2mm_P0.5mm -> Resistor_SMD:R_0603_1608Metric; symbol CM5Carrier:TPS62913RPU -> Device:R; MPN TPS62913RPUT -> RC0603FR-07255RL; Manufacturer Texas Instruments -> Yageo
- R1140: renamed from C1163; value 47uF X7R -> 33.2k / 400kHz; footprint (none) -> Resistor_SMD:R_0603_1608Metric; symbol Device:C -> Device:R; MPN GRM32ER71A476KE15L -> RC0603FR-0733K2L; Manufacturer Murata -> Yageo
- R1141: renamed from C1164; value 47uF X7R -> 100k 0.1%; footprint (none) -> Resistor_SMD:R_0603_1608Metric; symbol Device:C -> Device:R; MPN GRM32ER71A476KE15L -> TNPW0603100KBEEA; Manufacturer Murata -> Vishay
- R1142: renamed from C1165; value 47uF X7R -> 43.2k 0.1%; footprint (none) -> Resistor_SMD:R_0603_1608Metric; symbol Device:C -> Device:R; MPN GRM32ER71A476KE15L -> TNPW060343K2BEEA; Manufacturer Murata -> Vishay
- R1143: renamed from U1131; value TPS259827LNRGER -> 0R RBOOT; footprint Package_DFN_QFN:Texas_RGE0024H_VQFN-24-1EP_4x4mm_P0.5mm_EP2.7x2.7mm_ThermalVias -> Resistor_SMD:R_0603_1608Metric; symbol CM5Carrier:TPS259827LNRGE -> Device:R; MPN TPS259827LNRGER -> RC0603JR-070RL; Manufacturer Texas Instruments -> Yageo
- R1150: footprint (none) -> Resistor_SMD:R_0603_1608Metric; MPN (none) -> RC0603FR-0733K2L; Manufacturer (none) -> Yageo
- R1152, R1162: footprint (none) -> Resistor_SMD:R_0603_1608Metric; MPN (none) -> TNPW060343K2BEEA; Manufacturer (none) -> Vishay
- R11700: renamed from R11730; value 29.4k 0.1% -> 1.24k 0.1%; footprint (none) -> Resistor_SMD:R_0603_1608Metric; MPN (none) -> TNPW06031K24BEEA; Manufacturer (none) -> Vishay
- R11701: renamed from R11731; footprint (none) -> Resistor_SMD:R_0603_1608Metric; MPN (none) -> TNPW06034K99BEEA; Manufacturer (none) -> Vishay
- R11702: renamed from R11732; footprint (none) -> Resistor_SMD:R_0603_1608Metric
- R11710: renamed from F1184; value 3A time-lag -> 6.19k 0.1%; footprint (none) -> Resistor_SMD:R_0603_1608Metric; symbol Device:Fuse -> Device:R; MPN 0453003.MR -> TNPW06036K19BEEA; Manufacturer Littelfuse -> Vishay
- R11711: footprint (none) -> Resistor_SMD:R_0603_1608Metric; MPN (none) -> TNPW06034K99BEEA; Manufacturer (none) -> Vishay
- R11712: renamed from U1182; value TPS7A2050PDBVR -> 7.5k S-CONF; footprint Package_TO_SOT_SMD:SOT-23-5 -> Resistor_SMD:R_0603_1608Metric; symbol CM5Carrier:TPS7A20DBV_A1 -> Device:R; MPN TPS7A2050PDBVR -> RC0603FR-077K5L; Manufacturer Texas Instruments -> Yageo
- TP1190, TP1191, TP1192, TP1193: footprint (none) -> TestPoint:TestPoint_Pad_D2.0mm
- U1130: renamed from R1151; value 100k 0.1% -> LM61460RJR; footprint (none) -> CM5Carrier:TI_RJR0014A; symbol Device:R -> CM5Carrier:LM61460RJR; MPN (none) -> LM61460RJR; Manufacturer (none) -> Texas Instruments
- U1140: renamed from R1161; value 100k 0.1% -> LM61440RJR; footprint (none) -> CM5Carrier:TI_RJR0014A; symbol Device:R -> CM5Carrier:LM61440RJR; MPN (none) -> LM61440RJR; Manufacturer (none) -> Texas Instruments
- U1141: footprint (none) -> CM5Carrier:TI_DML0010A
- U1150: footprint (none) -> CM5Carrier:TI_RJR0014A
- renumbered U1173 to U1170
Connections:
- net AUDIOPRE5V5_EN is gone; now on net PCIE1V0_EN: U1170.1 (EN/SYNC)
- net AUDIOPRE5V5_FB is gone; now on net PCIE1V0_FB: R11700.2, R11701.1, U1170.9 (FB)
- net AUDIOPRE5V5_NRSS is gone; now on net PCIE1V0_NRSS: C11700.1, U1170.8 (NR/SS)
- net AUDIOPRE5V5_SCONF is gone; now on net PCIE1V0_SCONF: R11702.1, U1170.10 (S-CONF)
- net AUDIOPRE5V5_SW is gone; now on net PCIE1V0_SW: L11700.1, U1170.2 (SW)
- net AUDIO_PRE_5V5_PG is gone; now on net PCIE_1V0_PG: U1170.5 (PG)
- net HEADSET3V3_EN is gone; now on net MODEM_ILIM: R1138.1
- net HEADSET3V3_SW is gone; now on net GND: R1138.2
- net AGND: now also U1180.2 (-VIN), U1180.4 (COMMON); no longer C11710.2 (-VIN), C11710.4 (COMMON)
- net AUDIO_12V: now also U1180.1 (+VIN); no longer C11704.1, C11705.1, C11710.1 (+VIN), U1170.6 (VIN)
- net AUDIO_N15V: now also U1180.5 (-VOUT); no longer C11710.5 (-VOUT)
- net AUDIO_P15V: now also U1180.3 (+VOUT); no longer C11710.3 (+VOUT)
- net AUX_12V: now also C1124.1, C1125.1, C1126.1, C1127.1, F1183.1, F1184.1; no longer C1117.1, C1118.1, C1119.1, C1194.1, L11710.1, R11710.1
- net AUX_BOOT1: now also C1128.1, D1120.2 (A); no longer C1113.1, C1195.2 (A)
- net AUX_BOOT2: now also C1129.1, D1121.2 (A); no longer C1114.1, C1196.2 (A)
- net AUX_CS: now also Q1123.2 (S)
- net AUX_DITH: now also C1201.1; no longer C1116.1
- net AUX_EN_UVLO: now also R1128.1; no longer L1110.1
- net AUX_HDRV1: now also Q1120.1 (G)
- net AUX_LDRV2: now also Q1123.1 (G)
- net AUX_SW1: now also Q1120.2 (S), C1128.2; no longer C1113.2
- net AUX_SW2: now also Q1123.3 (D), C1129.2; no longer C1114.2
- net AUX_VCC: now also C1200.1, D1120.1 (K), D1121.1 (K); no longer C1115.1, C1195.1 (K), C1196.1 (K)
- net FAN_AUX_12V: now also F1184.2; no longer R11710.2
- net GND: now also C1113.2, C1114.2, C1135.2, C1155.2, C11710.2, C1195.2, C1196.2, U1130.11 (PGND2), U1130.3 (AGND), U1130.9 (PGND1), U1140.11 (PGND2), U1140.3 (AGND), U1140.9 (PGND1), C1124.2, C1125.2, C1126.2, C1127.2, C1131.2, C1152.2, C1153.2, C1154.2, C1156.2, C1162.2, C1163.2, C1164.2, C1165.2, C1166.2, C1200.2, C1201.2, C1202.2, R1128.2, R1160.2, U1131.10 (RETRY_DLY), U1131.11 (NRETRY), U1131.12 (LDSTRT), U1131.14 (GND3), U1131.4 (GND1), U1131.5 (GND2), U1160.11 (PGND2), U1160.3 (AGND), U1160.9 (PGND1); no longer C1118.2, C1130.2, C1140.2, C1155.4 (PGND), C1155.7 (PSNS), L1110.2, L1130.2, L1140.2, Q1123.2, R1131.2, R1133.11 (PGND2), R1133.3 (AGND), R1133.9 (PGND1), R1138.4 (PGND), R1138.7 (PSNS), R1141.2, R1143.10 (RETRY_DLY), R1143.11 (NRETRY), R1143.12 (LDSTRT), R1143.14 (GND3), R1143.4 (GND1), R1143.5 (GND2)
- net LOGIC1V8_FB: now also R11710.2
- net LOGIC1V8_NRSS: now also C11710.1
- net LOGIC1V8_SCONF: now also R11712.1
- net LOGIC1V8_SW: now also L11710.1
- net LOGIC3V3_CBOOT: now also U1160.14 (CBOOT); no longer R1133.14 (CBOOT)
- net LOGIC3V3_FB: now also R1161.2, U1160.4 (FB); no longer R1133.4 (FB), U1140.2
- net LOGIC3V3_RBOOT: now also U1160.13 (RBOOT); no longer R1133.13 (RBOOT)
- net LOGIC3V3_RT: now also R1160.1, U1160.6 (RT); no longer C1136.1, R1133.6 (RT)
- net LOGIC3V3_SW: now also L1160.1, U1160.10 (SW); no longer C1135.1, R1133.10 (SW)
- net LOGIC3V3_VCC: now also C1166.1, U1160.2 (VCC); no longer C1140.1, R1133.2 (VCC)
- net LOGIC_1V8: now also C11712.1, C11713.1, L11710.2, R11710.1
- net LOGIC_3V3: now also C1163.1, C1164.1, C1165.1, L1160.2, R1161.1, U1160.1 (BIAS); no longer C1135.2, R1133.1 (BIAS), R1140.1, R1141.1, R1142.1, U1140.1
- net LOGIC_3V3_PG: now also U1160.5 (PGOOD); no longer R1133.5 (PGOOD)
- net MODEM3V8PRE_CBOOT: now also C1130.1, R1133.2, U1130.14 (CBOOT)
- net MODEM3V8PRE_FB: now also R1131.2, R1132.1, U1130.4 (FB); no longer Q1120.2
- net MODEM3V8PRE_RBOOT: now also R1133.1, U1130.13 (RBOOT)
- net MODEM3V8PRE_RT: now also R1130.1, U1130.6 (RT)
- net MODEM3V8PRE_SW: now also C1130.2, L1130.1, U1130.10 (SW)
- net MODEM3V8PRE_VCC: now also C1136.1, U1130.2 (VCC)
- net MODEM_3V8: now also U1131.17 (OUT1), U1131.18 (OUT2), U1131.19 (OUT3), U1131.20 (OUT4), U1131.21 (OUT5), U1131.22 (OUT6), U1131.23 (OUT7), U1131.24 (OUT8); no longer R1143.17 (OUT1), R1143.18 (OUT2), R1143.19 (OUT3), R1143.20 (OUT4), R1143.21 (OUT5), R1143.22 (OUT6), R1143.23 (OUT7), R1143.24 (OUT8)
- net MODEM_3V8_PG: now also U1131.13 (PG); no longer R1143.13 (PG)
- net MODEM_3V8_PRE: now also C1135.1, L1130.2, R1131.1, U1130.1 (BIAS), U1131.1 (IN1), U1131.16 (IN4), U1131.2 (IN2), U1131.3 (IN3); no longer Q1120.1, R1143.1 (IN1), R1143.16 (IN4), R1143.2 (IN2), R1143.3 (IN3)
- net MODEM_3V8_PRE_PG: now also U1130.5 (PGOOD)
- net MODEM_DVDT: now also U1131.15 (dVdt); no longer R1143.15 (dVdt)
- net MODEM_ILIM: now also U1131.8 (ILIM); no longer R1143.8 (ILIM)
- net MODEM_IMON: now also U1131.9 (IMON); no longer R1143.9 (IMON)
- net MODEM_ITIMER: now also U1131.7 (ITIMER); no longer R1143.7 (ITIMER)
- net MODEM_POWER_EN: now also U1131.6 (EN/UVLO); no longer R1143.6 (EN/UVLO)
- net NET3V3_FB: now also R1151.2; no longer U1130.2
- net NET3V3_VCC: now also C1156.1; no longer C1130.1
- net NET_3V3: now also C1155.1, C1153.1, C1154.1, R1151.1; no longer R1130.1, R1131.1, R1132.1, U1130.1
- net NIGHT_LIGHT_12V: now also F1183.2; no longer L11710.2
- net PCIE1V0_EN: no longer C1155.1 (EN/SYNC)
- net PCIE1V0_FB: no longer C1155.9 (FB)
- net PCIE1V0_NRSS: no longer C1155.8 (NR/SS)
- net PCIE1V0_SCONF: no longer C1155.10 (S-CONF)
- net PCIE1V0_SW: no longer C1155.2 (SW)
- net PCIE_1V0: now also C11701.1, C11702.1, C11703.1, L11700.2, R11700.1, U1170.3 (VO); no longer C1155.3 (VO)
- net PCIE_1V0_PG: no longer C1155.5 (PG)
- net RAW_OUT_LOAD: now also C1194.1, C1195.1, C1196.1, Q1120.3 (D), U1130.12 (VIN2), U1130.8 (VIN1), U1140.12 (VIN2), U1140.8 (VIN1), C1131.1, C1152.1, C1162.1, C1202.1, U1160.12 (VIN2), U1160.8 (VIN1); no longer L1130.1, L1140.1, Q1123.1, R1133.12 (VIN2), R1133.8 (VIN1)
- net RAW_RAIL_EN: now also U1130.7 (EN/SYNC), U1140.7 (EN/SYNC), U1160.7 (EN/SYNC); no longer R1133.7 (EN/SYNC)
- net SYS_5V15: now also C1113.1, C1114.1, C1115.1, C1116.1, C1117.1, C11704.1, C11705.1, C11715.1, L1110.2, U1170.6 (VIN); no longer C1155.6 (VIN), R1138.6 (VIN)
- net SYS_BST: now also C1118.1
- net SYS_SW: now also C1118.2, L1110.1
- net SYS_VCC: now also C1119.1
- net WIFI3V3PRE_CBOOT: now also C1140.1, R1143.2, U1140.14 (CBOOT)
- net WIFI3V3PRE_FB: now also R1141.2, R1142.1, U1140.4 (FB)
- net WIFI3V3PRE_RBOOT: now also R1143.1, U1140.13 (RBOOT)
- net WIFI3V3PRE_RT: now also R1140.1, U1140.6 (RT)
- net WIFI3V3PRE_SW: now also C1140.2, L1140.1, U1140.10 (SW)
- net WIFI3V3PRE_VCC: now also U1140.2 (VCC)
- net WIFI_3V3_PRE: now also L1140.2, R1141.1, U1140.1 (BIAS)
- net WIFI_3V3_PRE_PG: now also U1140.5 (PGOOD)
- removed net ADC_5V_A: C11713.1, C11715.5 (OUT)
- removed net AUDIO_ENABLE: C11715.3 (EN), R11712.3 (EN)
- removed net AUDIO_PRE_5V5: C11701.1, C11702.1, C11703.1, C11712.1, C11715.1 (IN), L11700.2, R11700.1, R11712.1 (IN), U1170.3 (VO)
- removed net DAC_5V_A: R11712.5 (OUT)
- removed net HEADSET3V3_FB: R1138.9 (FB)
- removed net HEADSET3V3_NRSS: R1138.8 (NR/SS)
- removed net HEADSET3V3_SCONF: R1138.10 (S-CONF)
- removed net HEADSET_3V3: R1138.3 (VO)
- removed net HEADSET_3V3_PG: R1138.5 (PG)
- no-connect marks 7 -> 3
Other:
- note added: "1. PROTECTED RAW INPUT FROM PWR-SELECT"
- note added: "C1109 is local high-frequency input decoupling; the clamped bulk bank is not carried by this suspended PCB."
- note added: "PWR-SELECT C306-C309 provide 27.2 mF plus 660 uF local storage upstream of its load shunt."
- note added: "TPS62913 uses 2.2 MHz, 470 nF NR/SS and 2.2 uH. Headset LDOs live on Audio-Control; all AKM rails live on AUDIO-8X8."
- note added: "U1180 is a typed off-board handoff only. AUDIO-8X8 locally creates +/-15 V, the quiet 5.5 V pre-rail, separate LT3045 ADC/DAC 5 V rails and AKM 3.3 V."
- note removed: "1. PROTECTED RAW INPUT AND NO-BLINK HOLD-UP"
- note removed: "4 x 5600 uF installed = 22.4 mF. PWR-SELECT local 660 uF remains additive."
- note removed: "AUDIO-8X8 local: TRI 20-1223 creates +/-15 V. Separate TPS7A20 LDOs feed ADC 5 V, DAC 5 V and AKM 3.3 V; headset gets its own 1.8 V LDO."
- note removed: "Stuff C1104-C1108 only after source MOSFET SOA and inrush tests; fully stuffed total is about 47.7 mF."
- note removed: "TPS62913 uses 2.2 MHz, 470 nF NR/SS and 2.2 uH. Audio/headset variants add the optional ferrite second stage on their owning sheet."
- moved on the sheet: C1113, C1114, C1115, C1116, C1130, C1140, C11700, C11701, C11702, C11703, C11704, C11705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

Commit message: Lock CM5 power and radio interfaces before routing
Parts:
- added F1185: 2A time-lag, Fuse:Fuse_Littelfuse-NANO2-451_453, symbol Device:Fuse
- R1111: value 24.0k 0.1% -> 20.0k 0.1%; MPN TNPW060324K0BEEA -> TNPW060320K0BEEA
- R1112: value 4.42k 0.1% -> 4.99k 0.1%; MPN TNPW06034K42BEEA -> TNPW06034K99BEEA
- TP1191: value SYS_5V15 -> SYS_4V0
Connections:
- net AUX_12V: now also F1185.1
- net SYS_5V15 renamed SYS_4V0
- net SYS_5V15_PG renamed SYS_4V0_PG
- new net DISPLAY_IO_12V: F1185.2
Other:
- note added: "2. SYS_4V0 / 12 A SYNCHRONOUS BUCK"
- note added: "4.006 V nominal follows Radxa RK806 guidance. 300 kHz; target loop crossover about 20 kHz."
- note added: "RAW valid -> SYS_4V0, AUX_12V, LOGIC_3V3 and radio pre-regulators start from local UVLO."
- note added: "SYS_4V0_PG enables LOGIC_1V8 and PCIE_1V0; hold PCIe reset until NET_3V3_PG and PCIE_1V0_PG are both valid."
- note removed: "2. SYS_5V15 / 12 A SYNCHRONOUS BUCK"
- note removed: "RAW valid -> SYS_5V15, AUX_12V, LOGIC_3V3 and radio pre-regulators start from local UVLO."
- note removed: "SYS_5V15_PG enables LOGIC_1V8 and PCIE_1V0; hold PCIe reset until NET_3V3_PG and PCIE_1V0_PG are both valid."
- note removed: "TI 5 V / 12 A reference adapted to 5.144 V. 300 kHz; target loop crossover about 20 kHz."
Changed lines of the file:
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@@
 			)
 		)
-		(property "Value" "24.0k 0.1%"
+		(property "Value" "20.0k 0.1%"
 			(at 420.37 190.5 90)
 			(effects
@@
 			)
 		)
-		(property "MPN" "TNPW060324K0BEEA"
+		(property "MPN" "TNPW060320K0BEEA"
 			(at 422.91 195.5799 0)
 			(effects
@@
 			)
 		)
-		(property "Value" "4.42k 0.1%"
+		(property "Value" "4.99k 0.1%"
 			(at 464.82 190.5 90)
 			(effects
@@
 			)
 		)
-		(property "MPN" "TNPW06034K42BEEA"
+		(property "MPN" "TNPW06034K99BEEA"
 			(at 467.36 195.5799 0)
 			(effects
@@
 	)
 	(symbol
+		(lib_id "Device:Fuse")
+		(at 1169.67 619.76 0)
+		(unit 1)
+		(exclude_from_sim no)
+		(in_bom yes)
+		(on_board yes)
+		(dnp no)
+		(fields_autoplaced no)
+		(property "Reference" "F1185"
+			(at 1171.702 619.76 90)
+			(effects
+				(font
+					(size 1.27 1.27)
+				)
+				(justify left)
+			)
+		)
+		(property "Value" "2A time-lag"
+			(at 1167.765 619.76 90)
+			(effects
+				(font
+					(size 1.27 1.27)
+				)
+				(justify left)
+			)
+		)
+		(property "Footprint" "Fuse:Fuse_Littelfuse-NANO2-451_453"
+			(at 1167.892 619.76 90)
+			(effects
+				(font
+					(size 1.27 1.27)
+				)
+				(hide yes)
+			)
+		)
+		(property "Manufacturer" "Littelfuse"
+			(at 1172.21 624.8399 0)
+			(effects
+				(font
+					(size 1.27 1.27)
+				)
+				(hide yes)
+			)
+		)
+		(property "MPN" "0453002.MR"
+			(at 1172.21 624.8399 0)
+			(effects
+				(font
+					(size 1.27 1.27)
+				)
+				(hide yes)
+			)
+		)
+		(pin "1"
+		)
+		(pin "2"
+		)
+		(instances
+			(project "Power-Regulators-A1"
+				(path "/d6d0e65e-868d-5bca-b21c-3fa1f886a196"
+					(reference "F1185")
+					(unit 1)
+				)
+			)
+		)
+	)
+	(symbol
 		(lib_id "CM5Carrier:TRI20_1223")
 		(at 929.64 735.33 0)
@@
 			)
 		)
-		(property "Value" "SYS_5V15"
+		(property "Value" "SYS_4V0"
 			(at 439.42 784.86 0.0000)
 			(effects
@@
 		)
 	)
-	(label "SYS_5V15_PG"
+	(label "SYS_4V0_PG"
 		(at 425.45 97.79 0.0000)
 		(effects
@@
 		)
 	)
-	(label "SYS_5V15"
+	(label "SYS_4V0"
 		(at 420.37 186.69 0.0000)
 		(effects
@@
 		)
 	)
-	(label "SYS_5V15"
+	(label "SYS_4V0"
 		(at 650.24 114.3 0.0000)
 		(effects
@@
 		)
 	)
-	(label "SYS_5V15"
+	(label "SYS_4V0"
 		(at 619.76 186.69 0.0000)
 		(effects
@@
 		)
 	)
-	(label "SYS_5V15"
+	(label "SYS_4V0"
 		(at 650.24 186.69 0.0000)
 		(effects
@@
 		)
 	)
-	(label "SYS_5V15"
+	(label "SYS_4V0"
 		(at 679.45 186.69 0.0000)
 		(effects
@@
 		)
 	)
-	(label "SYS_5V15"
+	(label "SYS_4V0"
 		(at 709.93 186.69 0.0000)
 		(effects
@@
 		)
 	)
-	(label "SYS_5V15"
+	(label "SYS_4V0"
 		(at 740.41 186.69 0.0000)
 		(effects
@@
 		)
 	)
-	(label "SYS_5V15"
+	(label "SYS_4V0"
 		(at 590.55 617.22 0.0000)
 		(effects
@@
 		)
 	)
-	(label "SYS_5V15"
+	(label "SYS_4V0"
 		(at 480.06 670.56 0.0000)
 		(effects
@@
 		)
 	)
-	(label "SYS_5V15"
+	(label "SYS_4V0"
 		(at 505.46 670.56 0.0000)
 		(effects
@@
 		)
 	)
-	(label "SYS_5V15"
+	(label "SYS_4V0"
 		(at 820.42 617.22 0.0000)
 		(effects
@@
 		)
 	)
-	(label "SYS_5V15"
+	(label "SYS_4V0"
 		(at 709.93 670.56 0.0000)
 		(effects
@@
 		)
 	)
-	(label "SYS_5V15"
+	(label "SYS_4V0"
 		(at 735.33 670.56 0.0000)
 		(effects
@@
 		)
 	)
+	(label "AUX_12V"
+		(at 1169.67 615.95 0.0000)
+		(effects
+			(font
+				(size 0.7 0.7)
+			)
+			(justify left bottom)
+		)
+	)
+	(label "DISPLAY_IO_12V"
+		(at 1169.67 623.57 0.0000)
+		(effects
+			(font
+				(size 0.7 0.7)
+			)
+			(justify left bottom)
+		)
+	)
 	(label "AUDIO_12V"
 		(at 909.32 727.71 0.0000)
@@
 		)
 	)
-	(label "SYS_5V15"
+	(label "SYS_4V0"
 		(at 439.42 779.78 0.0000)
 		(effects
@@
 		)
 	)
-	(label "SYS_5V15"
+	(label "SYS_4V0"
 		(at 464.82 834.39 0.0000)
 		(effects
@@
 		)
 	)
-	(text "2. SYS_5V15 / 12 A SYNCHRONOUS BUCK"
+	(text "2. SYS_4V0 / 12 A SYNCHRONOUS BUCK"
 		(exclude_from_sim no)
 		(at 320 18 0.0000)
@@
 		)
 	)
-	(text "TI 5 V / 12 A reference adapted to 5.144 V. 300 kHz; target loop crossover about 20 kHz."
+	(text "4.006 V nominal follows Radxa RK806 guidance. 300 kHz; target loop crossover about 20 kHz."
 		(exclude_from_sim no)
 		(at 320 280 0.0000)
@@
 		)
 	)
-	(text "RAW valid -> SYS_5V15, AUX_12V, LOGIC_3V3 and radio pre-regulators start from local UVLO."
+	(text "RAW valid -> SYS_4V0, AUX_12V, LOGIC_3V3 and radio pre-regulators start from local UVLO."
 		(exclude_from_sim no)
 		(at 35 760 0.0000)
@@
 		)
 	)
-	(text "SYS_5V15_PG enables LOGIC_1V8 and PCIE_1V0; hold PCIe reset until NET_3V3_PG and PCIE_1V0_PG are both valid."
+	(text "SYS_4V0_PG enables LOGIC_1V8 and PCIE_1V0; hold PCIe reset until NET_3V3_PG and PCIE_1V0_PG are both valid."
 		(exclude_from_sim no)
 		(at 35 771 0.0000)

Commit message: Audit schematic logic against controlled datasheets
Parts:
- removed C1111: 6.8nF, Capacitor_SMD:C_0603_1608Metric, symbol Device:C
- removed C1122: 33nF, Capacitor_SMD:C_0603_1608Metric, symbol Device:C
- removed Q1111: FDWS86068-F085, CM5Carrier:onsemi_DFNW8_5p2x6p3_507AU_GSD, symbol Transistor_FET:Q_NMOS_GSD
- removed Q1121: CSD18532Q5B, CM5Carrier:TI_DNK0008A_GSD, symbol Transistor_FET:Q_NMOS_GSD
- removed Q1123: CSD17573Q5B, CM5Carrier:TI_DNK0008A_GSD, symbol Transistor_FET:Q_NMOS_GSD
- removed R1124: 20k 0.1%, Resistor_SMD:R_0603_1608Metric, symbol Device:R
- removed U1180: TRI 20-1223 ON AUDIO-8X8, CM5Carrier:TRACO_TRI20_DUAL, symbol CM5Carrier:TRI20_1223
- added F1181: 3A time-lag, Fuse:Fuse_Littelfuse-NANO2-451_453, symbol Device:Fuse
- added R1117, R1129, R1134, R1137, R1144, R1149, R1154, R1164, R11703, R11713: 10k 1%, Resistor_SMD:R_0603_1608Metric, symbol Device:R
- added R1139, R1148: 100k 1%, Resistor_SMD:R_0603_1608Metric, symbol Device:R
- added R11712: 7.5k S-CONF, Resistor_SMD:R_0603_1608Metric, symbol Device:R
- added TP1190: RAW_OUT_LOAD, TestPoint:TestPoint_Pad_D2.0mm, symbol Connector:TestPoint
- added TP1193: MODEM_3V8, TestPoint:TestPoint_Pad_D2.0mm, symbol Connector:TestPoint
- added TP1194: MODEM_IMON, TestPoint:TestPoint_Pad_D2.0mm, symbol Connector:TestPoint
- added TP1195: SYS_SYNCOUT_TP, TestPoint:TestPoint_Pad_D2.0mm, symbol Connector:TestPoint
- added U1141: TPS22990DMLR, CM5Carrier:TI_DML0010A, symbol CM5Carrier:TPS22990DML
- added U1170: TPS62913RPU, Package_DFN_QFN:Texas_RPU0010A_VQFN-HR-10_2x2mm_P0.5mm, symbol CM5Carrier:TPS62913RPU
- C1111: renamed from U1141; value TPS22990DMLR -> 6.8nF; footprint CM5Carrier:TI_DML0010A -> Capacitor_SMD:C_0603_1608Metric; symbol CM5Carrier:TPS22990DML -> Device:C; MPN TPS22990DMLR -> GRM1885C1H682JA01D; Manufacturer Texas Instruments -> Murata
- C1122: renamed from TP1193; value MODEM_3V8 -> 33nF; footprint TestPoint:TestPoint_Pad_D2.0mm -> Capacitor_SMD:C_0603_1608Metric; symbol Connector:TestPoint -> Device:C; MPN (none) -> GRM188R71H333KA01D; Manufacturer (none) -> Murata
- Q1111: renamed from U1170; value TPS62913RPU -> FDWS86068-F085; footprint Package_DFN_QFN:Texas_RPU0010A_VQFN-HR-10_2x2mm_P0.5mm -> CM5Carrier:onsemi_DFNW8_5p2x6p3_507AU_GSD; symbol CM5Carrier:TPS62913RPU -> Transistor_FET:Q_NMOS_GSD; MPN TPS62913RPUT -> FDWS86068-F085; Manufacturer Texas Instruments -> onsemi
- Q1121: renamed from R11712; value 7.5k S-CONF -> CSD18532Q5B; footprint Resistor_SMD:R_0603_1608Metric -> CM5Carrier:TI_DNK0008A_GSD; symbol Device:R -> Transistor_FET:Q_NMOS_GSD; MPN RC0603FR-077K5L -> CSD18532Q5B; Manufacturer Yageo -> Texas Instruments
- Q1123: renamed from F1181; value 3A time-lag -> CSD17573Q5B; footprint Fuse:Fuse_Littelfuse-NANO2-451_453 -> CM5Carrier:TI_DNK0008A_GSD; symbol Device:Fuse -> Transistor_FET:Q_NMOS_GSD; MPN 0453003.MR -> CSD17573Q5B; Manufacturer Littelfuse -> Texas Instruments
- R1124: renamed from TP1190; value RAW_OUT_LOAD -> 20k 0.1%; footprint TestPoint:TestPoint_Pad_D2.0mm -> Resistor_SMD:R_0603_1608Metric; symbol Connector:TestPoint -> Device:R; MPN (none) -> TNPW060320K0BEEA; Manufacturer (none) -> Vishay
- TP1191, TP1192: now left out of the parts list
Connections:
- net LOGIC1V8_EN is gone; now on net SYS_4V0_PG: U1171.1 (EN/SYNC)
- net PCIE1V0_EN is gone; now on net SYS_LO: Q1111.1 (G)
- net RAW_RAIL_EN is gone; now on net RAW_OUT_LOAD: U1130.7 (EN/SYNC), U1140.7 (EN/SYNC), U1150.7 (EN/SYNC), U1160.7 (EN/SYNC)
- net AUX_12V: now also F1181.1; no longer Q1123.1
- net AUX_12V_PG: now also R1129.2
- net AUX_COMP_C: now also C1122.1
- net AUX_CS: now also Q1121.2 (S), Q1123.2 (S)
- net AUX_FB: now also R1124.1
- net AUX_LDRV1: now also Q1121.1 (G)
- net AUX_LDRV2: now also Q1123.1 (G)
- net AUX_SW1: now also Q1121.3 (D)
- net AUX_SW2: now also Q1123.3 (D)
- net FAN_CPU_12V: now also F1181.2; no longer Q1123.2
- net GND: now also C1111.2, C1122.2, Q1111.2 (S), R1124.2, R1139.2, R1148.2, R11712.2, U1141.6 (GND), U1170.4 (PGND), U1170.7 (PSNS); no longer C1111.6 (GND), Q1111.4 (PGND), Q1111.7 (PSNS), Q1121.2
- net LOGIC1V8_SCONF: now also R11712.1; no longer Q1121.1
- net LOGIC_1V8_PG: now also R11713.2
- net LOGIC_3V3: now also R1117.1, R1129.1, R1134.1, R1137.1, R1144.1, R1149.1, R1154.1, R1164.1, R11703.1, R11713.1, U1141.4 (VBIAS); no longer C1111.4 (VBIAS)
- net LOGIC_3V3_PG: now also R1164.2
- net MODEM_3V8: now also TP1193.1; no longer C1122.1
- net MODEM_3V8_PG: now also R1137.2
- net MODEM_3V8_PRE_PG: now also R1134.2
- net MODEM_IMON: now also TP1194.1
- net MODEM_POWER_EN: now also R1139.1
- net NET_3V3_PG: now also R1154.2
- net PCIE1V0_FB: now also U1170.9 (FB); no longer Q1111.9 (FB)
- net PCIE1V0_NRSS: now also U1170.8 (NR/SS); no longer Q1111.8 (NR/SS)
- net PCIE1V0_SCONF: now also U1170.10 (S-CONF); no longer Q1111.10 (S-CONF)
- net PCIE1V0_SW: now also U1170.2 (SW); no longer Q1111.2 (SW)
- net PCIE_1V0: now also U1170.3 (VO); no longer Q1111.3 (VO)
- net PCIE_1V0_PG: now also R11703.2, U1170.5 (PG); no longer Q1111.5 (PG)
- net RAW_OUT_LOAD: now also TP1190.1; no longer R1124.1
- net SYS_4V0: now also U1170.6 (VIN); no longer Q1111.6 (VIN)
- net SYS_4V0_PG: now also R1117.2, U1170.1 (EN/SYNC)
- net SYS_COMP_C: now also C1111.1
- net SYS_SW: now also Q1111.3 (D)
- net SYS_SYNCOUT_TP: now also TP1195.1
- net WIFI_3V3: now also U1141.10 (VOUT3), U1141.8 (VOUT1), U1141.9 (VOUT2); no longer C1111.10 (VOUT3), C1111.8 (VOUT1), C1111.9 (VOUT2)
- net WIFI_3V3_PG: now also R1149.2, U1141.7 (PG); no longer C1111.7 (PG)
- net WIFI_3V3_PRE: now also U1141.3 (VIN); no longer C1111.3 (VIN)
- net WIFI_3V3_PRE_PG: now also R1144.2
- net WIFI_DVDT: now also U1141.1 (CT); no longer C1111.1 (CT)
- net WIFI_POWER_EN: now also R1148.1, U1141.5 (ON); no longer C1111.5 (ON)
Other:
- note added: "AUDIO_12V leaves this board through the controlled inter-board harness. AUDIO-8X8 locally creates +/-15 V, the quiet 5.5 V pre-rail, separate LT3045 ADC/DAC 5 V rails and AKM 3.3 V."
- note added: "SYS_4V0_PG directly enables LOGIC_1V8 and PCIE_1V0; all open-drain PGOOD outputs have 10k LOGIC_3V3 pull-ups."
- note added: "Wi-Fi and modem final rails default off through 100k pulls; Thermal-IO U1003 asserts them only after checks."
- note removed: "SYS_4V0_PG enables LOGIC_1V8 and PCIE_1V0; hold PCIe reset until NET_3V3_PG and PCIE_1V0_PG are both valid."
- note removed: "U1180 is a typed off-board handoff only. AUDIO-8X8 locally creates +/-15 V, the quiet 5.5 V pre-rail, separate LT3045 ADC/DAC 5 V rails and AKM 3.3 V."
- note removed: "Wi-Fi and modem final rails remain off until Thermal-IO asserts WIFI_POWER_EN / MODEM_POWER_EN after checks."
