File: cad/kicad/CM5-CARRIER/Power-Regulators-A1.kicad_sch (KiCad schematic)
At the start: 169 parts, among them J1100 RAW_POWER_FROM_PWR_SELECT, Q1110 NVMFS6B25NL, Q1111 FDWS86068-F085, Q1120 CSD18532Q5B, Q1121 CSD18532Q5B, Q1122 CSD17573Q5B, Q1123 CSD17573Q5B, U1110 LM5146RGYR, U1120 LM5176PWP, U1130 LM61460RJR, U1131 TPS259827LNRGER, U1140 LM61440RJR, U1141 TPS22990DMLR, U1150 LM61440RJR, U1160 LM61440RJR, U1170 TPS62913RPU, U1171 TPS62913RPU

Commit message: Implement direct socketed dual-SIM daughterboard
Parts:
- removed C1110: 47nF, Capacitor_SMD:C_0603_1608Metric, symbol Device:C
- removed C1113, C1114: 47uF 6.3V X7R, Capacitor_SMD:C_1210_3225Metric, symbol Device:C
- removed C1138: 4.7nF, Capacitor_SMD:C_0603_1608Metric, symbol Device:C
- removed C1149, C1210: 10nF, Capacitor_SMD:C_0603_1608Metric, symbol Device:C
- removed F1180, F1181: 3A time-lag, Fuse:Fuse_Littelfuse-NANO2-451_453, symbol Device:Fuse
- removed L1110: 3.3uH / 29.2A Isat, CM5Carrier:TDK_SPM10065VC, symbol Device:L
- removed L1120: 4.7uH / 20.9A Isat, CM5Carrier:Wurth_74439370047, symbol Device:L
- removed L1130, L1140, L1150, L1160: 4.7uH / 15.2A Isat, Inductor_SMD:L_Coilcraft_XAL7070-XXX, symbol Device:L
- removed L11700: 2.2uH / 2.0A rail, Inductor_SMD:L_Coilcraft_XxL4040, symbol Device:L
- removed L11710: 2.2uH / 1.5A rail, Inductor_SMD:L_Coilcraft_XxL4040, symbol Device:L
- removed R1110: 40.2k, Resistor_SMD:R_0603_1608Metric, symbol Device:R
- removed R1111: 20.0k 0.1%, Resistor_SMD:R_0603_1608Metric, symbol Device:R
- removed R1120: 6mR 2W, CM5Carrier:Susumu_KRL6432E_6mR, symbol Device:R
- removed R1126: 4mR 6W, CM5Carrier:Susumu_KRL11050_4mR, symbol Device:R
- removed R1130, R1140, R1150, R1160: 33.2k / 400kHz, Resistor_SMD:R_0603_1608Metric, symbol Device:R
- removed R1131, R1141, R1151, R1161: 100k 0.1%, Resistor_SMD:R_0603_1608Metric, symbol Device:R
- removed R1138: 255R 1% / 6A ILIM, Resistor_SMD:R_0603_1608Metric, symbol Device:R
- removed R11700: 1.24k 0.1%, Resistor_SMD:R_0603_1608Metric, symbol Device:R
- removed R11701, R11711: 4.99k 0.1%, Resistor_SMD:R_0603_1608Metric, symbol Device:R
- removed R11710: 6.19k 0.1%, Resistor_SMD:R_0603_1608Metric, symbol Device:R
- added C1135, C1145, C1155: 47uF X7R, Capacitor_SMD:C_1210_3225Metric, symbol Device:C
- added C1136, C1146, C1156: 1uF 10V X7R, Capacitor_SMD:C_0603_1608Metric, symbol Device:C
- added C11713: 22uF 10V X7R, Capacitor_SMD:C_0805_2012Metric, symbol Device:C
- added C1190, C1191, C1192: 330uF 6.3V polymer, Capacitor_SMD:CP_Elec_10x7.9, symbol Device:C_Polarized
- added C1193: 470uF 6.3V polymer, Capacitor_SMD:CP_Elec_8x11.9, symbol Device:C_Polarized
- added C1196, C1197, C1204, C1205: 4.7uF 50V X7R, Capacitor_SMD:C_1206_3216Metric, symbol Device:C
- added F1183: 0.25A fast, Fuse:Fuse_Littelfuse-NANO2-451_453, symbol Device:Fuse
- added F1184: 3A time-lag, Fuse:Fuse_Littelfuse-NANO2-451_453, symbol Device:Fuse
- added Q1110: NVMFS6B25NL, CM5Carrier:onsemi_DFN5_5x6_488AA_GSD, symbol Transistor_FET:Q_NMOS_GSD
- added R1115: 69.8k 1%, Resistor_SMD:R_0603_1608Metric, symbol Device:R
- added R1116, R1117, R1129, R1154, R1164, R11703, R11713: 10k 1%, Resistor_SMD:R_0603_1608Metric, symbol Device:R
- added R11702, R11712: 7.5k S-CONF, Resistor_SMD:R_0603_1608Metric, symbol Device:R
- added U1131: TPS259827LNRGER, Package_DFN_QFN:Texas_RGE0024H_VQFN-24-1EP_4x4mm_P0.5mm_EP2.7x2.7mm_ThermalVias, symbol CM5Carrier:TPS259827LNRGE
- added U1140, U1150, U1160: LM61440RJR, CM5Carrier:TI_RJR0014A, symbol CM5Carrier:LM61440RJR
- added U1171: TPS62913RPU, Package_DFN_QFN:Texas_RPU0010A_VQFN-HR-10_2x2mm_P0.5mm, symbol CM5Carrier:TPS62913RPU
- C1110: renamed from R1113; value 7.5k -> 47nF; footprint Resistor_SMD:R_0603_1608Metric -> Capacitor_SMD:C_0603_1608Metric; symbol Device:R -> Device:C; MPN RC0603FR-077K5L -> GRM188R71H473KA61D; Manufacturer Yageo -> Murata
- C1111: renamed from R1115; value 69.8k 1% -> 6.8nF; footprint Resistor_SMD:R_0603_1608Metric -> Capacitor_SMD:C_0603_1608Metric; symbol Device:R -> Device:C; MPN RC0603FR-0769K8L -> GRM1885C1H682JA01D; Manufacturer Yageo -> Murata
- C1112: renamed from R1116; value 10k 1% -> 150pF C0G; footprint Resistor_SMD:R_0603_1608Metric -> Capacitor_SMD:C_0603_1608Metric; symbol Device:R -> Device:C; MPN RC0603FR-0710KL -> GRM1885C1H151JA01D; Manufacturer Yageo -> Murata
- C1115: renamed from C1118; value 100nF 25V X7R -> 47uF 6.3V X7R; footprint Capacitor_SMD:C_0603_1608Metric -> Capacitor_SMD:C_1210_3225Metric; MPN GRM188R71E104KA01D -> GCM32ER70J476KE19L
- C1116: renamed from C1119; value 4.7uF 10V X7R -> 47uF 6.3V X7R; footprint Capacitor_SMD:C_0805_2012Metric -> Capacitor_SMD:C_1210_3225Metric; MPN GRM21BR71A475KA73L -> GCM32ER70J476KE19L
- C1117: renamed from C1194; value 4.7uF 50V X7R -> 47uF 6.3V X7R; footprint Capacitor_SMD:C_1206_3216Metric -> Capacitor_SMD:C_1210_3225Metric; MPN GRM31CR71H475KA12L -> GCM32ER70J476KE19L
- C1118: renamed from C1195; value 4.7uF 50V X7R -> 100nF 25V X7R; footprint Capacitor_SMD:C_1206_3216Metric -> Capacitor_SMD:C_0603_1608Metric; MPN GRM31CR71H475KA12L -> GRM188R71E104KA01D
- C1119: renamed from C1196; value 4.7uF 50V X7R -> 4.7uF 10V X7R; footprint Capacitor_SMD:C_1206_3216Metric -> Capacitor_SMD:C_0805_2012Metric; MPN GRM31CR71H475KA12L -> GRM21BR71A475KA73L
- C1120: renamed from R1124; value 20k 0.1% -> 220pF; footprint Resistor_SMD:R_0603_1608Metric -> Capacitor_SMD:C_0603_1608Metric; symbol Device:R -> Device:C; MPN TNPW060320K0BEEA -> GRM1885C1H221JA01D; Manufacturer Vishay -> Murata
- C1121: renamed from R1125; value 10k -> 100nF; footprint Resistor_SMD:R_0603_1608Metric -> Capacitor_SMD:C_0603_1608Metric; symbol Device:R -> Device:C; MPN RC0603FR-0710KL -> GRM188R71E104KA01D; Manufacturer Yageo -> Murata
- C1122: renamed from R1128; value 10k 1% -> 33nF; footprint Resistor_SMD:R_0603_1608Metric -> Capacitor_SMD:C_0603_1608Metric; symbol Device:R -> Device:C; MPN RC0603FR-0710KL -> GRM188R71H333KA01D; Manufacturer Yageo -> Murata
- C1123: renamed from C1128; value 100nF 25V -> 560pF; MPN GRM188R71E104KA01D -> GRM1885C1H561JA01D
- C1125: renamed from D1120; value BAT54WS -> 330uF 16V polymer; footprint Diode_SMD:D_SOD-323 -> Capacitor_SMD:CP_Elec_10x12.6; symbol Device:D_Schottky -> Device:C_Polarized; MPN BAT54WS-7-F -> 16SVP330M; Manufacturer Diodes Incorporated -> Panasonic
- C1126: renamed from D1121; value BAT54WS -> 330uF 16V polymer; footprint Diode_SMD:D_SOD-323 -> Capacitor_SMD:CP_Elec_10x12.6; symbol Device:D_Schottky -> Device:C_Polarized; MPN BAT54WS-7-F -> 16SVP330M; Manufacturer Diodes Incorporated -> Panasonic
- C1127: renamed from C1202; value 4.7uF 50V X7R -> 330uF 16V polymer; footprint Capacitor_SMD:C_1206_3216Metric -> Capacitor_SMD:CP_Elec_10x12.6; symbol Device:C -> Device:C_Polarized; MPN GRM31CR71H475KA12L -> 16SVP330M; Manufacturer Murata -> Panasonic
- C1128: renamed from C1201; value 2.2nF -> 100nF 25V; MPN GRM188R71H222KA01D -> GRM188R71E104KA01D
- C1129: renamed from C1124; value 330uF 16V polymer -> 100nF 25V; footprint Capacitor_SMD:CP_Elec_10x12.6 -> Capacitor_SMD:C_0603_1608Metric; symbol Device:C_Polarized -> Device:C; MPN 16SVP330M -> GRM188R71E104KA01D; Manufacturer Panasonic -> Murata
- C1130: renamed from C1132; value 4.7uF 50V -> 100nF; footprint Capacitor_SMD:C_1206_3216Metric -> Capacitor_SMD:C_0603_1608Metric; MPN GRM31CR71H475KA12L -> GRM188R71E104KA01D
- C1131: renamed from C1134; value 47uF X7R -> 4.7uF 50V; footprint Capacitor_SMD:C_1210_3225Metric -> Capacitor_SMD:C_1206_3216Metric; MPN GRM32ER71A476KE15L -> GRM31CR71H475KA12L
- C1132: renamed from C1135; value 47uF X7R -> 4.7uF 50V; footprint Capacitor_SMD:C_1210_3225Metric -> Capacitor_SMD:C_1206_3216Metric; MPN GRM32ER71A476KE15L -> GRM31CR71H475KA12L
- C1133: renamed from C1136; value 1uF 10V X7R -> 47uF X7R; footprint Capacitor_SMD:C_0603_1608Metric -> Capacitor_SMD:C_1210_3225Metric; MPN GRM188R71A105KA61D -> GRM32ER71A476KE15L
- C1134: renamed from U1140; value LM61440RJR -> 47uF X7R; footprint CM5Carrier:TI_RJR0014A -> Capacitor_SMD:C_1210_3225Metric; symbol CM5Carrier:LM61440RJR -> Device:C; MPN LM61440RJR -> GRM32ER71A476KE15L; Manufacturer Texas Instruments -> Murata
- C1138: renamed from R1137; value 10k 1% -> 4.7nF; footprint Resistor_SMD:R_0603_1608Metric -> Capacitor_SMD:C_0603_1608Metric; symbol Device:R -> Device:C; MPN RC0603FR-0710KL -> GRM188R71H472KA01D; Manufacturer Yageo -> Murata
- C1140: renamed from C1142; value 4.7uF 50V -> 100nF; footprint Capacitor_SMD:C_1206_3216Metric -> Capacitor_SMD:C_0603_1608Metric; MPN GRM31CR71H475KA12L -> GRM188R71E104KA01D
- C1141: renamed from C1144; value 47uF X7R -> 4.7uF 50V; footprint Capacitor_SMD:C_1210_3225Metric -> Capacitor_SMD:C_1206_3216Metric; MPN GRM32ER71A476KE15L -> GRM31CR71H475KA12L
- C1142: renamed from C1145; value 47uF X7R -> 4.7uF 50V; footprint Capacitor_SMD:C_1210_3225Metric -> Capacitor_SMD:C_1206_3216Metric; MPN GRM32ER71A476KE15L -> GRM31CR71H475KA12L
- C1143: renamed from C1146; value 1uF 10V X7R -> 47uF X7R; footprint Capacitor_SMD:C_0603_1608Metric -> Capacitor_SMD:C_1210_3225Metric; MPN GRM188R71A105KA61D -> GRM32ER71A476KE15L
- C1144: renamed from U1150; value LM61440RJR -> 47uF X7R; footprint CM5Carrier:TI_RJR0014A -> Capacitor_SMD:C_1210_3225Metric; symbol CM5Carrier:LM61440RJR -> Device:C; MPN LM61440RJR -> GRM32ER71A476KE15L; Manufacturer Texas Instruments -> Murata
- C1149: renamed from C1193; value 470uF 6.3V polymer -> 10nF; footprint Capacitor_SMD:CP_Elec_8x11.9 -> Capacitor_SMD:C_0603_1608Metric; symbol Device:C_Polarized -> Device:C; MPN 6SVP470M -> GRM188R71H103KA01D; Manufacturer Panasonic -> Murata
- C1150: renamed from C1152; value 4.7uF 50V -> 100nF; footprint Capacitor_SMD:C_1206_3216Metric -> Capacitor_SMD:C_0603_1608Metric; MPN GRM31CR71H475KA12L -> GRM188R71E104KA01D
- C1151: renamed from C1154; value 47uF X7R -> 4.7uF 50V; footprint Capacitor_SMD:C_1210_3225Metric -> Capacitor_SMD:C_1206_3216Metric; MPN GRM32ER71A476KE15L -> GRM31CR71H475KA12L
- C1152: renamed from C1155; value 47uF X7R -> 4.7uF 50V; footprint Capacitor_SMD:C_1210_3225Metric -> Capacitor_SMD:C_1206_3216Metric; MPN GRM32ER71A476KE15L -> GRM31CR71H475KA12L
- C1153: renamed from C1156; value 1uF 10V X7R -> 47uF X7R; footprint Capacitor_SMD:C_0603_1608Metric -> Capacitor_SMD:C_1210_3225Metric; MPN GRM188R71A105KA61D -> GRM32ER71A476KE15L
- C1154: renamed from U1160; value LM61440RJR -> 47uF X7R; footprint CM5Carrier:TI_RJR0014A -> Capacitor_SMD:C_1210_3225Metric; symbol CM5Carrier:LM61440RJR -> Device:C; MPN LM61440RJR -> GRM32ER71A476KE15L; Manufacturer Texas Instruments -> Murata
- C1160: renamed from C1162; value 4.7uF 50V -> 100nF; footprint Capacitor_SMD:C_1206_3216Metric -> Capacitor_SMD:C_0603_1608Metric; MPN GRM31CR71H475KA12L -> GRM188R71E104KA01D
- C1161: renamed from C1164; value 47uF X7R -> 4.7uF 50V; footprint Capacitor_SMD:C_1210_3225Metric -> Capacitor_SMD:C_1206_3216Metric; MPN GRM32ER71A476KE15L -> GRM31CR71H475KA12L
- C1162: renamed from C1165; value 47uF X7R -> 4.7uF 50V; footprint Capacitor_SMD:C_1210_3225Metric -> Capacitor_SMD:C_1206_3216Metric; MPN GRM32ER71A476KE15L -> GRM31CR71H475KA12L
- C1163: renamed from C1166; value 1uF 10V X7R -> 47uF X7R; footprint Capacitor_SMD:C_0603_1608Metric -> Capacitor_SMD:C_1210_3225Metric; MPN GRM188R71A105KA61D -> GRM32ER71A476KE15L
- C1164: renamed from R1134; value 10k 1% -> 47uF X7R; footprint Resistor_SMD:R_0603_1608Metric -> Capacitor_SMD:C_1210_3225Metric; symbol Device:R -> Device:C; MPN RC0603FR-0710KL -> GRM32ER71A476KE15L; Manufacturer Yageo -> Murata
- C1165: renamed from R1144; value 10k 1% -> 47uF X7R; footprint Resistor_SMD:R_0603_1608Metric -> Capacitor_SMD:C_1210_3225Metric; symbol Device:R -> Device:C; MPN RC0603FR-0710KL -> GRM32ER71A476KE15L; Manufacturer Yageo -> Murata
- C1166: renamed from R1154; value 10k 1% -> 1uF 10V X7R; footprint Resistor_SMD:R_0603_1608Metric -> Capacitor_SMD:C_0603_1608Metric; symbol Device:R -> Device:C; MPN RC0603FR-0710KL -> GRM188R71A105KA61D; Manufacturer Yageo -> Murata
- C11700: renamed from C11701; value 22uF 10V X7R -> 470nF; footprint Capacitor_SMD:C_0805_2012Metric -> Capacitor_SMD:C_0603_1608Metric; MPN GRM21BR71A226ME44L -> GRM188R71E474KA12D
- C11701: renamed from R11702; value 7.5k S-CONF -> 22uF 10V X7R; footprint Resistor_SMD:R_0603_1608Metric -> Capacitor_SMD:C_0805_2012Metric; symbol Device:R -> Device:C; MPN RC0603FR-077K5L -> GRM21BR71A226ME44L; Manufacturer Yageo -> Murata
- C11702: renamed from R11703; value 10k 1% -> 22uF 10V X7R; footprint Resistor_SMD:R_0603_1608Metric -> Capacitor_SMD:C_0805_2012Metric; symbol Device:R -> Device:C; MPN RC0603FR-0710KL -> GRM21BR71A226ME44L; Manufacturer Yageo -> Murata
- C11703: renamed from U1171; value TPS62913RPU -> 22uF 10V X7R; footprint Package_DFN_QFN:Texas_RPU0010A_VQFN-HR-10_2x2mm_P0.5mm -> Capacitor_SMD:C_0805_2012Metric; symbol CM5Carrier:TPS62913RPU -> Device:C; MPN TPS62913RPUT -> GRM21BR71A226ME44L; Manufacturer Texas Instruments -> Murata
- C11704: renamed from C11702; value 22uF 10V X7R -> 10uF 25V X7R; MPN GRM21BR71A226ME44L -> GRM21BR71E106KA73L
- C11705: renamed from C11703; value 22uF 10V X7R -> 10uF 25V X7R; MPN GRM21BR71A226ME44L -> GRM21BR71E106KA73L
- C11710: renamed from C11711; value 22uF 10V X7R -> 470nF; footprint Capacitor_SMD:C_0805_2012Metric -> Capacitor_SMD:C_0603_1608Metric; MPN GRM21BR71A226ME44L -> GRM188R71E474KA12D
- C11711: renamed from R11712; value 7.5k S-CONF -> 22uF 10V X7R; footprint Resistor_SMD:R_0603_1608Metric -> Capacitor_SMD:C_0805_2012Metric; symbol Device:R -> Device:C; MPN RC0603FR-077K5L -> GRM21BR71A226ME44L; Manufacturer Yageo -> Murata
- C11712: renamed from R11713; value 10k 1% -> 22uF 10V X7R; footprint Resistor_SMD:R_0603_1608Metric -> Capacitor_SMD:C_0805_2012Metric; symbol Device:R -> Device:C; MPN RC0603FR-0710KL -> GRM21BR71A226ME44L; Manufacturer Yageo -> Murata
- C11714: renamed from C11712; value 22uF 10V X7R -> 10uF 25V X7R; MPN GRM21BR71A226ME44L -> GRM21BR71E106KA73L
- C11715: renamed from C11713; value 22uF 10V X7R -> 10uF 25V X7R; MPN GRM21BR71A226ME44L -> GRM21BR71E106KA73L
- C1195: renamed from R1117; value 10k 1% -> 4.7uF 50V X7R; footprint Resistor_SMD:R_0603_1608Metric -> Capacitor_SMD:C_1206_3216Metric; symbol Device:R -> Device:C; MPN RC0603FR-0710KL -> GRM31CR71H475KA12L; Manufacturer Yageo -> Murata
- C1200: renamed from C1125; value 330uF 16V polymer -> 4.7uF 10V; footprint Capacitor_SMD:CP_Elec_10x12.6 -> Capacitor_SMD:C_0805_2012Metric; symbol Device:C_Polarized -> Device:C; MPN 16SVP330M -> GRM21BR71A475KA73L; Manufacturer Panasonic -> Murata
- C1201: renamed from C1126; value 330uF 16V polymer -> 2.2nF; footprint Capacitor_SMD:CP_Elec_10x12.6 -> Capacitor_SMD:C_0603_1608Metric; symbol Device:C_Polarized -> Device:C; MPN 16SVP330M -> GRM188R71H222KA01D; Manufacturer Panasonic -> Murata
- C1203: renamed from R1129; value 10k 1% -> 4.7uF 50V X7R; footprint Resistor_SMD:R_0603_1608Metric -> Capacitor_SMD:C_1206_3216Metric; symbol Device:R -> Device:C; MPN RC0603FR-0710KL -> GRM31CR71H475KA12L; Manufacturer Yageo -> Murata
- C1210: renamed from C1189; value 330uF 6.3V polymer -> 10nF; footprint Capacitor_SMD:CP_Elec_10x7.9 -> Capacitor_SMD:C_0603_1608Metric; symbol Device:C_Polarized -> Device:C; MPN 6SVP330M -> GRM188R71H103KA01D; Manufacturer Panasonic -> Murata
- D1120: renamed from C1203; value 4.7uF 50V X7R -> BAT54WS; footprint Capacitor_SMD:C_1206_3216Metric -> Diode_SMD:D_SOD-323; symbol Device:C -> Device:D_Schottky; MPN GRM31CR71H475KA12L -> BAT54WS-7-F; Manufacturer Murata -> Diodes Incorporated
- D1121: renamed from C1204; value 4.7uF 50V X7R -> BAT54WS; footprint Capacitor_SMD:C_1206_3216Metric -> Diode_SMD:D_SOD-323; symbol Device:C -> Device:D_Schottky; MPN GRM31CR71H475KA12L -> BAT54WS-7-F; Manufacturer Murata -> Diodes Incorporated
- F1180: renamed from F1183; value 0.25A fast -> 3A time-lag; MPN 0453.250MR -> 0453003.MR
- L1110: renamed from C1115; value 47uF 6.3V X7R -> 3.3uH / 29.2A Isat; footprint Capacitor_SMD:C_1210_3225Metric -> CM5Carrier:TDK_SPM10065VC; symbol Device:C -> Device:L; MPN GCM32ER70J476KE19L -> SPM10065VC-3R3M-D; Manufacturer Murata -> TDK
- L1120: renamed from R1121; value 27.4k -> 4.7uH / 20.9A Isat; footprint Resistor_SMD:R_0603_1608Metric -> CM5Carrier:Wurth_74439370047; symbol Device:R -> Device:L; MPN RC0603FR-0727K4L -> 74439370047; Manufacturer Yageo -> Wurth Elektronik
- L1130: renamed from R1132; value 35.7k 0.1% -> 4.7uH / 15.2A Isat; footprint Resistor_SMD:R_0603_1608Metric -> Inductor_SMD:L_Coilcraft_XAL7070-XXX; symbol Device:R -> Device:L; MPN TNPW060335K7BEEA -> XAL7070-472MEC; Manufacturer Vishay -> Coilcraft
- L1140: renamed from R1142; value 43.2k 0.1% -> 4.7uH / 15.2A Isat; footprint Resistor_SMD:R_0603_1608Metric -> Inductor_SMD:L_Coilcraft_XAL7070-XXX; symbol Device:R -> Device:L; MPN TNPW060343K2BEEA -> XAL7070-472MEC; Manufacturer Vishay -> Coilcraft
- L1150: renamed from R1152; value 43.2k 0.1% -> 4.7uH / 15.2A Isat; footprint Resistor_SMD:R_0603_1608Metric -> Inductor_SMD:L_Coilcraft_XAL7070-XXX; symbol Device:R -> Device:L; MPN TNPW060343K2BEEA -> XAL7070-472MEC; Manufacturer Vishay -> Coilcraft
- L1160: renamed from R1162; value 43.2k 0.1% -> 4.7uH / 15.2A Isat; footprint Resistor_SMD:R_0603_1608Metric -> Inductor_SMD:L_Coilcraft_XAL7070-XXX; symbol Device:R -> Device:L; MPN TNPW060343K2BEEA -> XAL7070-472MEC; Manufacturer Vishay -> Coilcraft
- L11700: renamed from C11700; value 470nF -> 2.2uH / 2.0A rail; footprint Capacitor_SMD:C_0603_1608Metric -> Inductor_SMD:L_Coilcraft_XxL4040; symbol Device:C -> Device:L; MPN GRM188R71E474KA12D -> XGL4030-222MEC; Manufacturer Murata -> Coilcraft
- L11710: renamed from C11710; value 470nF -> 2.2uH / 1.5A rail; footprint Capacitor_SMD:C_0603_1608Metric -> Inductor_SMD:L_Coilcraft_XxL4040; symbol Device:C -> Device:L; MPN GRM188R71E474KA12D -> XGL4030-222MEC; Manufacturer Murata -> Coilcraft
- R1110: renamed from R1112; value 4.99k 0.1% -> 40.2k; MPN TNPW06034K99BEEA -> RC0603FR-0740K2L; Manufacturer Vishay -> Yageo
- R1111: renamed from C1111; value 6.8nF -> 20.0k 0.1%; footprint Capacitor_SMD:C_0603_1608Metric -> Resistor_SMD:R_0603_1608Metric; symbol Device:C -> Device:R; MPN GRM1885C1H682JA01D -> TNPW060320K0BEEA; Manufacturer Murata -> Vishay
- R1112: renamed from C1112; value 150pF C0G -> 4.99k 0.1%; footprint Capacitor_SMD:C_0603_1608Metric -> Resistor_SMD:R_0603_1608Metric; symbol Device:C -> Device:R; MPN GRM1885C1H151JA01D -> TNPW06034K99BEEA; Manufacturer Murata -> Vishay
- R1113: renamed from R1114; value 499R -> 7.5k; MPN RC0603FR-07499RL -> RC0603FR-077K5L
- R1114: renamed from Q1110; value NVMFS6B25NL -> 499R; footprint CM5Carrier:onsemi_DFN5_5x6_488AA_GSD -> Resistor_SMD:R_0603_1608Metric; symbol Transistor_FET:Q_NMOS_GSD -> Device:R; MPN NVMFS6B25NLT1G -> RC0603FR-07499RL; Manufacturer onsemi -> Yageo
- R1120: renamed from R1122; value 93.1k -> 6mR 2W; footprint Resistor_SMD:R_0603_1608Metric -> CM5Carrier:Susumu_KRL6432E_6mR; MPN RC0603FR-0793K1L -> KRL6432E-M-R006-F-T1; Manufacturer Yageo -> Susumu
- R1121: renamed from C1121; value 100nF -> 27.4k; footprint Capacitor_SMD:C_0603_1608Metric -> Resistor_SMD:R_0603_1608Metric; symbol Device:C -> Device:R; MPN GRM188R71E104KA01D -> RC0603FR-0727K4L; Manufacturer Murata -> Yageo
- R1122: renamed from R1123; value 280k 0.1% -> 93.1k; MPN TNPW0603280KBEEA -> RC0603FR-0793K1L; Manufacturer Vishay -> Yageo
- R1123: renamed from C1122; value 33nF -> 280k 0.1%; footprint Capacitor_SMD:C_0603_1608Metric -> Resistor_SMD:R_0603_1608Metric; symbol Device:C -> Device:R; MPN GRM188R71H333KA01D -> TNPW0603280KBEEA; Manufacturer Murata -> Vishay
- R1124: renamed from C1123; value 560pF -> 20k 0.1%; footprint Capacitor_SMD:C_0603_1608Metric -> Resistor_SMD:R_0603_1608Metric; symbol Device:C -> Device:R; MPN GRM1885C1H561JA01D -> TNPW060320K0BEEA; Manufacturer Murata -> Vishay
- R1125: renamed from R1127; value 73.2k 1% -> 10k; MPN RC0603FR-0773K2L -> RC0603FR-0710KL
- R1126: renamed from C1120; value 220pF -> 4mR 6W; footprint Capacitor_SMD:C_0603_1608Metric -> CM5Carrier:Susumu_KRL11050_4mR; symbol Device:C -> Device:R; MPN GRM1885C1H221JA01D -> KRL11050-C-R004-F-T1; Manufacturer Murata -> Susumu
- R1127: renamed from C1129; value 100nF 25V -> 73.2k 1%; footprint Capacitor_SMD:C_0603_1608Metric -> Resistor_SMD:R_0603_1608Metric; symbol Device:C -> Device:R; MPN GRM188R71E104KA01D -> RC0603FR-0773K2L; Manufacturer Murata -> Yageo
- R1128: renamed from C1200; value 4.7uF 10V -> 10k 1%; footprint Capacitor_SMD:C_0805_2012Metric -> Resistor_SMD:R_0603_1608Metric; symbol Device:C -> Device:R; MPN GRM21BR71A475KA73L -> RC0603FR-0710KL; Manufacturer Murata -> Yageo
- R1130: renamed from C1130; value 100nF -> 33.2k / 400kHz; footprint Capacitor_SMD:C_0603_1608Metric -> Resistor_SMD:R_0603_1608Metric; symbol Device:C -> Device:R; MPN GRM188R71E104KA01D -> RC0603FR-0733K2L; Manufacturer Murata -> Yageo
- R1131: renamed from R1133; value 0R RBOOT -> 100k 0.1%; MPN RC0603JR-070RL -> TNPW0603100KBEEA; Manufacturer Yageo -> Vishay
- R1132: renamed from C1131; value 4.7uF 50V -> 35.7k 0.1%; footprint Capacitor_SMD:C_1206_3216Metric -> Resistor_SMD:R_0603_1608Metric; symbol Device:C -> Device:R; MPN GRM31CR71H475KA12L -> TNPW060335K7BEEA; Manufacturer Murata -> Vishay
- R1133: renamed from C1133; value 47uF X7R -> 0R RBOOT; footprint Capacitor_SMD:C_1210_3225Metric -> Resistor_SMD:R_0603_1608Metric; symbol Device:C -> Device:R; MPN GRM32ER71A476KE15L -> RC0603JR-070RL; Manufacturer Murata -> Yageo
- R1137: renamed from C1191; value 330uF 6.3V polymer -> 10k 1%; footprint Capacitor_SMD:CP_Elec_10x7.9 -> Resistor_SMD:R_0603_1608Metric; symbol Device:C_Polarized -> Device:R; MPN 6SVP330M -> RC0603FR-0710KL; Manufacturer Panasonic -> Yageo
- R1138: renamed from R1139; value 100k 1% -> 255R 1% / 6A ILIM; MPN RC0603FR-07100KL -> RC0603FR-07255RL
- R1139: renamed from C1190; value 330uF 6.3V polymer -> 100k 1%; footprint Capacitor_SMD:CP_Elec_10x7.9 -> Resistor_SMD:R_0603_1608Metric; symbol Device:C_Polarized -> Device:R; MPN 6SVP330M -> RC0603FR-07100KL; Manufacturer Panasonic -> Yageo
- R1140: renamed from C1140; value 100nF -> 33.2k / 400kHz; footprint Capacitor_SMD:C_0603_1608Metric -> Resistor_SMD:R_0603_1608Metric; symbol Device:C -> Device:R; MPN GRM188R71E104KA01D -> RC0603FR-0733K2L; Manufacturer Murata -> Yageo
- R1141: renamed from R1143; value 0R RBOOT -> 100k 0.1%; MPN RC0603JR-070RL -> TNPW0603100KBEEA; Manufacturer Yageo -> Vishay
- R1142: renamed from C1141; value 4.7uF 50V -> 43.2k 0.1%; footprint Capacitor_SMD:C_1206_3216Metric -> Resistor_SMD:R_0603_1608Metric; symbol Device:C -> Device:R; MPN GRM31CR71H475KA12L -> TNPW060343K2BEEA; Manufacturer Murata -> Vishay
- R1143: renamed from C1143; value 47uF X7R -> 0R RBOOT; footprint Capacitor_SMD:C_1210_3225Metric -> Resistor_SMD:R_0603_1608Metric; symbol Device:C -> Device:R; MPN GRM32ER71A476KE15L -> RC0603JR-070RL; Manufacturer Murata -> Yageo
- R1144: renamed from U1131; value TPS259827LNRGER -> 10k 1%; footprint Package_DFN_QFN:Texas_RGE0024H_VQFN-24-1EP_4x4mm_P0.5mm_EP2.7x2.7mm_ThermalVias -> Resistor_SMD:R_0603_1608Metric; symbol CM5Carrier:TPS259827LNRGE -> Device:R; MPN TPS259827LNRGER -> RC0603FR-0710KL; Manufacturer Texas Instruments -> Yageo
- R1150: renamed from C1150; value 100nF -> 33.2k / 400kHz; footprint Capacitor_SMD:C_0603_1608Metric -> Resistor_SMD:R_0603_1608Metric; symbol Device:C -> Device:R; MPN GRM188R71E104KA01D -> RC0603FR-0733K2L; Manufacturer Murata -> Yageo
- R1151: renamed from R1153; value 0R RBOOT -> 100k 0.1%; MPN RC0603JR-070RL -> TNPW0603100KBEEA; Manufacturer Yageo -> Vishay
- R1152: renamed from C1151; value 4.7uF 50V -> 43.2k 0.1%; footprint Capacitor_SMD:C_1206_3216Metric -> Resistor_SMD:R_0603_1608Metric; symbol Device:C -> Device:R; MPN GRM31CR71H475KA12L -> TNPW060343K2BEEA; Manufacturer Murata -> Vishay
- R1153: renamed from C1153; value 47uF X7R -> 0R RBOOT; footprint Capacitor_SMD:C_1210_3225Metric -> Resistor_SMD:R_0603_1608Metric; symbol Device:C -> Device:R; MPN GRM32ER71A476KE15L -> RC0603JR-070RL; Manufacturer Murata -> Yageo
- R1160: renamed from C1160; value 100nF -> 33.2k / 400kHz; footprint Capacitor_SMD:C_0603_1608Metric -> Resistor_SMD:R_0603_1608Metric; symbol Device:C -> Device:R; MPN GRM188R71E104KA01D -> RC0603FR-0733K2L; Manufacturer Murata -> Yageo
- R1161: renamed from R1163; value 0R RBOOT -> 100k 0.1%; MPN RC0603JR-070RL -> TNPW0603100KBEEA; Manufacturer Yageo -> Vishay
- R1162: renamed from C1161; value 4.7uF 50V -> 43.2k 0.1%; footprint Capacitor_SMD:C_1206_3216Metric -> Resistor_SMD:R_0603_1608Metric; symbol Device:C -> Device:R; MPN GRM31CR71H475KA12L -> TNPW060343K2BEEA; Manufacturer Murata -> Vishay
- R1163: renamed from C1163; value 47uF X7R -> 0R RBOOT; footprint Capacitor_SMD:C_1210_3225Metric -> Resistor_SMD:R_0603_1608Metric; symbol Device:C -> Device:R; MPN GRM32ER71A476KE15L -> RC0603JR-070RL; Manufacturer Murata -> Yageo
- R11700: renamed from C11704; value 10uF 25V X7R -> 1.24k 0.1%; footprint Capacitor_SMD:C_0805_2012Metric -> Resistor_SMD:R_0603_1608Metric; symbol Device:C -> Device:R; MPN GRM21BR71E106KA73L -> TNPW06031K24BEEA; Manufacturer Murata -> Vishay
- R11701: renamed from C11705; value 10uF 25V X7R -> 4.99k 0.1%; footprint Capacitor_SMD:C_0805_2012Metric -> Resistor_SMD:R_0603_1608Metric; symbol Device:C -> Device:R; MPN GRM21BR71E106KA73L -> TNPW06034K99BEEA; Manufacturer Murata -> Vishay
- R11710: renamed from C11714; value 10uF 25V X7R -> 6.19k 0.1%; footprint Capacitor_SMD:C_0805_2012Metric -> Resistor_SMD:R_0603_1608Metric; symbol Device:C -> Device:R; MPN GRM21BR71E106KA73L -> TNPW06036K19BEEA; Manufacturer Murata -> Vishay
- R11711: renamed from C11715; value 10uF 25V X7R -> 4.99k 0.1%; footprint Capacitor_SMD:C_0805_2012Metric -> Resistor_SMD:R_0603_1608Metric; symbol Device:C -> Device:R; MPN GRM21BR71E106KA73L -> TNPW06034K99BEEA; Manufacturer Murata -> Vishay
- renumbered C1116 to C1113, C1117 to C1114, C1127 to C1124, C1192 to C1189, C1197 to C1194, C1205 to C1202, F1184 to F1181, R1164 to R1134
Connections:
- net AUX_12V: now also C1125.1, C1126.1, C1127.1, R1120.2, R1123.1, F1183.1, F1184.1; no longer C1129.1, C1200.1, C1201.1, R1122.1
- net AUX_12V_PG: now also R1129.2; no longer C1203.2
- net AUX_12V_PRE: now also R1120.1
- net AUX_BOOT1: now also C1128.1, D1120.2 (A); no longer C1123.1, C1125.2 (A)
- net AUX_BOOT2: now also C1129.1, D1121.2 (A); no longer C1126.2 (A), R1127.1
- net AUX_COMP: now also C1123.1, R1125.1; no longer C1121.1, R1124.1
- net AUX_COMP_C: now also C1122.1, R1125.2; no longer C1121.2, R1123.1
- net AUX_CS: now also R1126.1
- net AUX_DITH: now also C1201.1; no longer C1128.1
- net AUX_EN_UVLO: now also R1127.2, R1128.1; no longer C1122.1, R1125.2
- net AUX_FB: now also C1123.2, R1123.2, R1124.1; no longer C1120.1, R1122.2, R1124.2
- net AUX_MODE: now also R1122.1; no longer R1120.1
- net AUX_RT: now also R1121.1; no longer L1120.1
- net AUX_SLOPE: now also C1120.1; no longer R1126.1
- net AUX_SS: now also C1121.1; no longer R1121.1
- net AUX_SW1: now also C1128.2, L1120.1; no longer C1123.2
- net AUX_SW2: now also C1129.2, L1120.2; no longer R1127.2
- net AUX_VCC: now also C1200.1, D1120.1 (K), D1121.1 (K); no longer C1125.1 (K), C1126.1 (K), R1128.1
- net DISPLAY_12V: now also F1180.2
- net FAN_AUX_12V: now also F1184.2; no longer F1181.2
- net FAN_CPU_12V: now also F1181.2
- net GND: now also C1110.2, C1111.2, C1115.2, C1121.2, C1125.2, C1126.2, C1134.2, C1138.2, C1144.2, C1154.2, C1164.2, C1165.2, C1166.2, C11702.2, C11703.2, C11712.2, C1195.2, C1203.2, R1112.2, R1122.2, R1124.2, R1130.2, R1140.2, R1150.2, R1160.2, C1135.2, C1136.2, C1145.2, C1146.2, C1155.2, C1156.2, C11713.2, C1190.2, C1191.2, C1192.2, C1193.2, C1196.2, C1197.2, C1204.2, C1205.2, R1116.2, R11702.2, R11712.2, U1131.10 (RETRY_DLY), U1131.11 (NRETRY), U1131.12 (LDSTRT), U1131.14 (GND3), U1131.4 (GND1), U1131.5 (GND2), U1140.11 (PGND2), U1140.3 (AGND), U1140.9 (PGND1), U1150.11 (PGND2), U1150.3 (AGND), U1150.9 (PGND1), U1160.11 (PGND2), U1160.3 (AGND), U1160.9 (PGND1), U1171.4 (PGND), U1171.7 (PSNS); no longer C1112.2, C1118.2, C1128.2, C1129.2, C1130.2, C1134.11 (PGND2), C1134.3 (AGND), C1134.9 (PGND1), C1140.2, C1144.11 (PGND2), C1144.3 (AGND), C1144.9 (PGND1), C1150.2, C1154.11 (PGND2), C1154.3 (AGND), C1154.9 (PGND1), C1160.2, C11703.4 (PGND), C11703.7 (PSNS), D1120.2, D1121.2, L1110.2, L1120.2, L1130.2, L1140.2, L1150.2, L1160.2, L11700.2, L11710.2, R1111.2, R1120.2, R1123.2, R1133.2, R1137.2, R1143.2, R1144.10 (RETRY_DLY), R1144.11 (NRETRY), R1144.12 (LDSTRT), R1144.14 (GND3), R1144.4 (GND1), R1144.5 (GND2), R1153.2, R1163.2, R11700.2, R11710.2
- net LOGIC1V8_FB: now also R11710.2, R11711.1, U1171.9 (FB); no longer C11703.9 (FB)
- net LOGIC1V8_NRSS: now also C11710.1, U1171.8 (NR/SS); no longer C11703.8 (NR/SS), L11710.1
- net LOGIC1V8_SCONF: now also R11712.1, U1171.10 (S-CONF); no longer C11703.10 (S-CONF), C11711.1
- net LOGIC1V8_SW: now also L11710.1, U1171.2 (SW); no longer C11703.2 (SW)
- net LOGIC3V3_CBOOT: now also C1160.1, R1163.2, U1160.14 (CBOOT); no longer C1154.14 (CBOOT), R1160.1, R1161.2
- net LOGIC3V3_FB: now also R1161.2, R1162.1, U1160.4 (FB); no longer C1154.4 (FB), L1160.1
- net LOGIC3V3_RBOOT: now also R1163.1, U1160.13 (RBOOT); no longer C1154.13 (RBOOT), R1161.1
- net LOGIC3V3_RT: now also R1160.1, U1160.6 (RT); no longer C1154.6 (RT)
- net LOGIC3V3_SW: now also C1160.2, L1160.1, U1160.10 (SW); no longer C1154.10 (SW), R1160.2
- net LOGIC3V3_VCC: now also C1166.1, U1160.2 (VCC); no longer C1154.2 (VCC), C1163.1
- net LOGIC_1V8: now also C11711.1, C11712.1, L11710.2, R11710.1, C11713.1, U1171.3 (VO); no longer C11703.3 (VO), C11710.1, C11714.1, C11715.1
- net LOGIC_1V8_PG: now also R11713.2, U1171.5 (PG); no longer C11703.5 (PG), C11712.2
- net LOGIC_3V3: now also C1163.1, L1160.2, R1137.1, R1144.1, R1161.1, R1117.1, R1129.1, R1154.1, R1164.1, R11703.1, R11713.1, U1160.1 (BIAS); no longer C1138.1, C1154.1 (BIAS), C1161.1, C1162.1, C1166.1, C11702.1, C11712.1, C1195.1, C1203.1, R1163.1
- net LOGIC_3V3_PG: now also R1164.2, U1160.5 (PGOOD); no longer C1154.5 (PGOOD), R1134.2
- net MODEM3V8PRE_CBOOT: now also C1130.1, R1133.2; no longer R1130.1, R1131.2
- net MODEM3V8PRE_FB: now also R1131.2, R1132.1; no longer L1130.1
- net MODEM3V8PRE_RBOOT: now also R1133.1; no longer R1131.1
- net MODEM3V8PRE_RT: now also R1130.1
- net MODEM3V8PRE_SW: now also C1130.2, L1130.1; no longer R1130.2
- net MODEM3V8PRE_VCC: now also C1136.1; no longer C1133.1
- net MODEM_3V8: now also C1190.1, C1191.1, C1192.1, U1131.17 (OUT1), U1131.18 (OUT2), U1131.19 (OUT3), U1131.20 (OUT4), U1131.21 (OUT5), U1131.22 (OUT6), U1131.23 (OUT7), U1131.24 (OUT8); no longer C1210.1, R1137.1, R1139.1, R1144.17 (OUT1), R1144.18 (OUT2), R1144.19 (OUT3), R1144.20 (OUT4), R1144.21 (OUT5), R1144.22 (OUT6), R1144.23 (OUT7), R1144.24 (OUT8)
- net MODEM_3V8_PG: now also R1137.2, U1131.13 (PG); no longer C1138.2, R1144.13 (PG)
- net MODEM_3V8_PRE: now also C1133.1, C1134.1, L1130.2, R1131.1, C1135.1, U1131.1 (IN1), U1131.16 (IN4), U1131.2 (IN2), U1131.3 (IN3); no longer C1131.1, C1132.1, R1133.1, R1144.1 (IN1), R1144.16 (IN4), R1144.2 (IN2), R1144.3 (IN3)
- net MODEM_3V8_PRE_PG: now also R1134.2; no longer C1164.2
- net MODEM_DVDT: now also C1210.1, U1131.15 (dVdt); no longer R1144.15 (dVdt)
- net MODEM_ILIM: now also R1138.1, U1131.8 (ILIM); no longer R1144.8 (ILIM)
- net MODEM_IMON: now also U1131.9 (IMON); no longer R1144.9 (IMON)
- net MODEM_ITIMER: now also C1138.1, U1131.7 (ITIMER); no longer R1144.7 (ITIMER)
- net MODEM_POWER_EN: now also R1139.1, U1131.6 (EN/UVLO); no longer R1138.1, R1144.6 (EN/UVLO)
- net NET3V3_CBOOT: now also C1150.1, R1153.2, U1150.14 (CBOOT); no longer C1144.14 (CBOOT), R1150.1, R1151.2
- net NET3V3_FB: now also R1151.2, R1152.1, U1150.4 (FB); no longer C1144.4 (FB), L1150.1
- net NET3V3_RBOOT: now also R1153.1, U1150.13 (RBOOT); no longer C1144.13 (RBOOT), R1151.1
- net NET3V3_RT: now also R1150.1, U1150.6 (RT); no longer C1144.6 (RT)
- net NET3V3_SW: now also C1150.2, L1150.1, U1150.10 (SW); no longer C1144.10 (SW), R1150.2
- net NET3V3_VCC: now also C1156.1, U1150.2 (VCC); no longer C1144.2 (VCC), C1153.1
- net NET_3V3: now also C1153.1, C1154.1, L1150.2, R1151.1, C1155.1, U1150.1 (BIAS); no longer C1144.1 (BIAS), C1151.1, C1152.1, R1153.1
- net NET_3V3_PG: now also R1154.2, U1150.5 (PGOOD); no longer C1144.5 (PGOOD), C1166.2
- net NIGHT_LIGHT_12V: now also F1183.2; no longer F1180.2
- net PCIE1V0_FB: now also R11700.2, R11701.1
- net PCIE1V0_NRSS: now also C11700.1; no longer L11700.1
- net PCIE1V0_SCONF: now also R11702.1; no longer C11701.1
- net PCIE1V0_SW: now also L11700.1
- net PCIE_1V0: now also C11701.1, C11702.1, C11703.1, L11700.2, R11700.1; no longer C11700.1, C11704.1, C11705.1
- net PCIE_1V0_PG: now also R11703.2; no longer C11702.2
- net RAW_OUT_LOAD: now also C1131.1, C1132.1, C1141.1, C1142.1, C1151.1, C1152.1, C1161.1, C1162.1, C1195.1, C1203.1, R1127.1, C1196.1, C1197.1, C1204.1, C1205.1, Q1110.3 (D), R1115.1, U1140.12 (VIN2), U1140.7 (EN/SYNC), U1140.8 (VIN1), U1150.12 (VIN2), U1150.7 (EN/SYNC), U1150.8 (VIN1), U1160.12 (VIN2), U1160.7 (EN/SYNC), U1160.8 (VIN1); no longer C1111.1, C1117.1, C1118.1, C1119.1, C1127.1, C1130.1, C1134.12 (VIN2), C1134.7 (EN/SYNC), C1134.8 (VIN1), C1140.1, C1144.12 (VIN2), C1144.7 (EN/SYNC), C1144.8 (VIN1), C1150.1, C1154.12 (VIN2), C1154.7 (EN/SYNC), C1154.8 (VIN1), C1160.1, D1120.1, D1121.1, R1114.3 (D), R1125.1, R1132.1, R1142.1, R1152.1, R1162.1
- net SYS_4V0: now also C1115.1, C1116.1, C1117.1, C11704.1, C11705.1, C11714.1, C11715.1, L1110.2, R1111.1, U1171.6 (VIN); no longer C11703.6 (VIN), L1110.1, R11700.1, R11701.1, R11710.1, R11711.1
- net SYS_4V0_PG: now also R1117.2, U1171.1 (EN/SYNC); no longer C11703.1 (EN/SYNC), C1195.2
- net SYS_BST: now also C1118.1; no longer C1115.1
- net SYS_COMP: now also C1112.1, R1113.1; no longer C1110.1, R1112.1
- net SYS_COMP_C: now also C1111.1, R1113.2; no longer C1110.2, R1111.1
- net SYS_EN_UVLO: now also R1115.2, R1116.1; no longer C1111.2, C1112.1
- net SYS_FB: now also C1112.2, R1111.2, R1112.1; no longer R1110.1, R1112.2
- net SYS_HO: now also Q1110.1 (G); no longer R1114.1 (G)
- net SYS_ILIM: now also R1114.1; no longer R1113.1
- net SYS_RT: now also R1110.1
- net SYS_SS: now also C1110.1
- net SYS_SW: now also C1118.2, L1110.1, Q1110.2 (S); no longer C1115.2, R1113.2
- net SYS_VCC: now also C1119.1; no longer C1116.1
- net WIFI3V3PRE_CBOOT: now also C1140.1, R1143.2, U1140.14 (CBOOT); no longer C1134.14 (CBOOT), R1140.1, R1141.2
- net WIFI3V3PRE_FB: now also R1141.2, R1142.1, U1140.4 (FB); no longer C1134.4 (FB), L1140.1
- net WIFI3V3PRE_RBOOT: now also R1143.1, U1140.13 (RBOOT); no longer C1134.13 (RBOOT), R1141.1
- net WIFI3V3PRE_RT: now also R1140.1, U1140.6 (RT); no longer C1134.6 (RT)
- net WIFI3V3PRE_SW: now also C1140.2, L1140.1, U1140.10 (SW); no longer C1134.10 (SW), R1140.2
- net WIFI3V3PRE_VCC: now also C1146.1, U1140.2 (VCC); no longer C1134.2 (VCC), C1143.1
- net WIFI_3V3: now also C1193.1; no longer C1149.1
- net WIFI_3V3_PRE: now also C1143.1, C1144.1, L1140.2, R1141.1, C1145.1, U1140.1 (BIAS); no longer C1134.1 (BIAS), C1141.1, C1142.1, R1143.1
- net WIFI_3V3_PRE_PG: now also R1144.2, U1140.5 (PGOOD); no longer C1134.5 (PGOOD), C1165.2
- net WIFI_DVDT: now also C1149.1
Other:
- moved on the sheet: C1113, C1114, C1115, C1116, C1117, C1118, C1119, C1123, C1124, C1128, C1130, C1131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
