File: cad/kicad/CM5-CARRIER/Thermal-IO.kicad_sch (KiCad schematic)
At the start: 60 parts, among them J1021 CPU_FAN, J1022 MODEM_FAN, J1023 THA0412AD-TZW3 INTAKE, J1024 THA0412AD-TZW3 EXHAUST, U1000 PCA9306D, U1001 TCA9535PWR_0x20, U1002 TCA9535PWR_0x21, U1020 EMC2305-1-AP-TR, U1050 TMP117_CM5, U1051 TMP117_MODEM, U1052 TMP117_BOARD_POWER

Commit message: Complete A1 detailed carrier and audio capture
Parts:
- removed C1051: 100nF, symbol Device:C
- removed D1060: PWR_GREEN, symbol Device:LED
- removed D1061: BACKUP_VIOLET, symbol Device:LED
- removed D1062: WIFI_BLUE, symbol Device:LED
- removed D1063: CELL_AMBER, symbol Device:LED
- removed D1064: TEMP_RED, symbol Device:LED
- removed D1065: AUDIO_CYAN, symbol Device:LED
- removed D1070, D1071: YIS LS102W 12V WARM WHITE, symbol Device:LED
- removed J1021: CPU_FAN, symbol Connector_Generic:Conn_01x04
- removed J1022: MODEM_FAN, symbol Connector_Generic:Conn_01x04
- removed J1024: THA0412AD-TZW3 EXHAUST, symbol Connector_Generic:Conn_01x04
- removed R1065: 1k, symbol Device:R
- removed S1070: CS7L2FR TOUCH LATCH, symbol Connector_Generic:Conn_01x06
- removed U1050: TMP117_CM5, symbol Sensor_Temperature:TMP117xxDRV
- added F1023: 1.1A hold / 33V, Fuse:Fuse_1812_4532Metric, symbol Device:Polyfuse
- added F1060: 0.25A fast, Fuse:Fuse_Littelfuse-NANO2-451_453, symbol Device:Fuse
- added J1021: FFB0412EN-00Y2E CPU FAN, Connector_Molex:Molex_Micro-Fit_3.0_43045-0412_2x02_P3.00mm_Vertical, symbol Connector_Generic:Conn_02x02_Odd_Even
- added J1022: AFB0412SHB-SP04 MODEM FAN, Connector_Molex:Molex_Micro-Fit_3.0_43045-0412_2x02_P3.00mm_Vertical, symbol Connector_Generic:Conn_02x02_Odd_Even
- added J1023: THA0412AD-TZW3 INTAKE, Connector_Molex:Molex_Micro-Fit_3.0_43045-0412_2x02_P3.00mm_Vertical, symbol Connector_Generic:Conn_02x02_Odd_Even
- added J1024: THA0412AD-TZW3 EXHAUST, Connector_Molex:Molex_Micro-Fit_3.0_43045-0412_2x02_P3.00mm_Vertical, symbol Connector_Generic:Conn_02x02_Odd_Even
- added J1060: STATUS_LAMP_PANEL_HARNESS, Connector_Molex:Molex_Micro-Fit_3.0_43045-0812_2x04_P3.00mm_Vertical, symbol Connector_Generic:Conn_02x04_Odd_Even
- added J1070: NIGHT_LIGHT_PANEL_HARNESS, Connector_Molex:Molex_Micro-Fit_3.0_43045-0812_2x04_P3.00mm_Vertical, symbol Connector_Generic:Conn_02x04_Odd_Even
- added Q1060, Q1061, Q1063: 2N7002K-7, Package_TO_SOT_SMD:SOT-23, symbol Transistor_FET:Q_NMOS_GSD
- added R1005: 4.7k, Resistor_SMD:R_0603_1608Metric, symbol Device:R
- added R1010, R1017, R1080, R1081, R1083, R1084: 100k, Resistor_SMD:R_0603_1608Metric, symbol Device:R
- added R1031, R1033, R1043: 10k, Resistor_SMD:R_0603_1608Metric, symbol Device:R
- C1020, C1050, C1052: footprint (none) -> Capacitor_SMD:C_0603_1608Metric; MPN (none) -> GRM188R71E104KA01D; Manufacturer (none) -> Murata
- C1051: renamed from R1017; value 100k -> 100nF; footprint (none) -> Capacitor_SMD:C_0603_1608Metric; symbol Device:R -> Device:C; MPN (none) -> GRM188R71E104KA01D; Manufacturer (none) -> Murata
- F1021: renamed from R1005; value 4.7k -> 3.0A hold / 15V; footprint (none) -> Fuse:Fuse_2920_7451Metric; symbol Device:R -> Device:Polyfuse; MPN (none) -> 2920L300/15DR; Manufacturer (none) -> Littelfuse
- F1022, F1024: value 1.0A hold -> 1.1A hold / 33V; footprint (none) -> Fuse:Fuse_1812_4532Metric; MPN (none) -> 1812L110/33DR; Manufacturer (none) -> Littelfuse
- Q1062: renamed from R1031; value 10k -> 2N7002K-7; footprint (none) -> Package_TO_SOT_SMD:SOT-23; symbol Device:R -> Transistor_FET:Q_NMOS_GSD; MPN (none) -> 2N7002K-7; Manufacturer (none) -> Diodes Incorporated
- Q1064: renamed from J1023; value THA0412AD-TZW3 INTAKE -> 2N7002K-7; footprint (none) -> Package_TO_SOT_SMD:SOT-23; symbol Connector_Generic:Conn_01x04 -> Transistor_FET:Q_NMOS_GSD; MPN (none) -> 2N7002K-7; Manufacturer (none) -> Diodes Incorporated
- Q1065: renamed from R1043; value 10k -> 2N7002K-7; footprint (none) -> Package_TO_SOT_SMD:SOT-23; symbol Device:R -> Transistor_FET:Q_NMOS_GSD; MPN (none) -> 2N7002K-7; Manufacturer (none) -> Diodes Incorporated
- R1001, R1002, R1003, R1004: footprint (none) -> Resistor_SMD:R_0603_1608Metric; MPN (none) -> RC0603FR-072K2L; Manufacturer (none) -> Yageo
- R1011, R1012, R1013, R1014, R1015, R1016, R1018: footprint (none) -> Resistor_SMD:R_0603_1608Metric; MPN (none) -> RC0603FR-07100KL; Manufacturer (none) -> Yageo
- R1020, R1021: footprint (none) -> Resistor_SMD:R_0603_1608Metric; MPN (none) -> RC0603FR-074K7L; Manufacturer (none) -> Yageo
- R1032, R1034, R1041, R1042, R1044: footprint (none) -> Resistor_SMD:R_0603_1608Metric; MPN (none) -> RC0603FR-0710KL; Manufacturer (none) -> Yageo
- R1050: footprint (none) -> Resistor_SMD:R_0603_1608Metric; MPN (none) -> RC0603FR-075K1L; Manufacturer (none) -> Yageo
- R1060, R1061, R1062, R1063, R1064: footprint (none) -> Resistor_SMD:R_0603_1608Metric; MPN (none) -> RC0603FR-071KL; Manufacturer (none) -> Yageo
- R1065: renamed from F1023; value 1.0A hold -> 1k; footprint (none) -> Resistor_SMD:R_0603_1608Metric; symbol Device:Polyfuse -> Device:R; MPN (none) -> RC0603FR-071KL; Manufacturer (none) -> Yageo
- R1070: footprint (none) -> Resistor_SMD:R_0603_1608Metric
- R1082: renamed from F1021; value 2.0A hold -> 100k; footprint (none) -> Resistor_SMD:R_0603_1608Metric; symbol Device:Polyfuse -> Device:R; MPN (none) -> RC0603FR-07100KL; Manufacturer (none) -> Yageo
- R1085: renamed from R1033; value 10k -> 100k; footprint (none) -> Resistor_SMD:R_0603_1608Metric; MPN (none) -> RC0603FR-07100KL; Manufacturer (none) -> Yageo
- U1000: value PCA9306D -> PCA9306DP; footprint (none) -> Package_SO:TSSOP-8_3x3mm_P0.65mm; MPN PCA9306D,118 -> PCA9306DP,118
- U1001, U1002: footprint (none) -> Package_SO:TSSOP-24_4.4x7.8mm_P0.65mm
- U1020: footprint (none) -> Package_DFN_QFN:QFN-16-1EP_4x4mm_P0.65mm_EP2.1x2.1mm
- U1050: renamed from R1010; value 100k -> TMP117_CM5; footprint (none) -> Package_SON:WSON-6-1EP_2x2mm_P0.65mm_EP1x1.6mm; symbol Device:R -> Sensor_Temperature:TMP117xxDRV; MPN (none) -> TMP117AIDRVR; Manufacturer (none) -> Texas Instruments
- U1051, U1052: footprint (none) -> Package_SON:WSON-6-1EP_2x2mm_P0.65mm_EP1x1.6mm; MPN TMP117MAIDRVR -> TMP117AIDRVR
Connections:
- net AUDIO_ENABLE: now also R1010.1; no longer U1050.1
- net CPU_FAN_12V: now also F1021.2, J1021.2 (Pin_2); no longer R1082.2
- net CPU_FAN_PWM: now also J1021.4 (Pin_4), R1031.2; no longer Q1062.2
- net CPU_FAN_TACH: now also J1021.3 (Pin_3)
- net CS_GREEN_RING_K: now also J1070.3 (Pin_3)
- net CTRL_I2C_SCL: now also U1050.1 (SCL)
- net CTRL_I2C_SDA: now also U1050.6 (SDA)
- net EXHAUST_FAN_12V: now also J1024.2 (Pin_2)
- net EXHAUST_FAN_PWM: now also J1024.4 (Pin_4)
- net EXHAUST_FAN_TACH: now also J1024.3 (Pin_3)
- net FAN_AUX_12V: now also F1023.1; no longer R1065.1
- net FAN_CPU_12V: now also F1021.1; no longer R1082.1
- net GND: now also C1051.2, Q1062.2 (S), Q1064.2 (S), Q1065.2 (S), R1082.2, R1085.2, U1050.4 (ADD0), J1021.1 (Pin_1), J1022.1 (Pin_1), J1023.1 (Pin_1), J1024.1 (Pin_1), J1070.1 (Pin_1), Q1060.2 (S), Q1061.2 (S), Q1063.2 (S), R1010.2, R1080.2, R1081.2, R1083.2, R1084.2; no longer Q1064.1 (Pin_1)
- net INTAKE_FAN_12V: now also F1023.2, J1023.2 (Pin_2); no longer Q1064.2 (Pin_2), R1065.2
- net INTAKE_FAN_PWM: now also J1023.4 (Pin_4), R1033.2; no longer Q1064.4 (Pin_4), R1085.2
- net INTAKE_FAN_TACH: now also J1023.3 (Pin_3), R1043.2; no longer Q1064.3 (Pin_3), Q1065.2
- net LAN1_RESET_LOCAL_N: now also R1017.1; no longer C1051.1
- net LOGIC_3V3: now also C1051.1, U1050.5 (V+), R1005.1, R1017.2, R1031.1, R1033.1, R1043.1; no longer C1051.2, F1021.1, Q1062.1, Q1065.1, R1060.1, R1061.1, R1062.1, R1063.1, R1064.1, R1085.1
- net MODEM_FAN_12V: now also J1022.2 (Pin_2)
- net MODEM_FAN_PWM: now also J1022.4 (Pin_4)
- net MODEM_FAN_TACH: now also J1022.3 (Pin_3)
- net NIGHT_LIGHT_12V: now also J1070.2 (Pin_2), J1070.5 (Pin_5), J1070.7 (Pin_7)
- net NIGHT_LIGHT_SINK: now also J1070.4 (Pin_4), J1070.6 (Pin_6), J1070.8 (Pin_8)
- net PWR_MON_ALERT_N: now also R1005.2; no longer F1021.2
- net TEMP_ALERT_N: now also U1050.3 (ALERT)
- net BACKUP_VIOLET_A renamed STATUS_BACKUP_GATE
- net STATUS_BACKUP_GATE: now also Q1061.1 (G), R1081.1
- net CELL_AMBER_A renamed STATUS_CELL_GATE
- net STATUS_CELL_GATE: now also Q1063.1 (G), R1083.1
- net LED_AUDIO_N renamed LED_AUDIO_GATE
- net LED_AUDIO_GATE: now also R1065.1
- net LED_BACKUP_N renamed LED_BACKUP_GATE
- net LED_BACKUP_GATE: now also R1061.1
- net LED_CELL_N renamed LED_CELL_GATE
- net LED_CELL_GATE: now also R1063.1
- net LED_PWR_N renamed LED_PWR_GATE
- net LED_PWR_GATE: now also R1060.1
- net LED_TEMP_N renamed LED_TEMP_GATE
- net LED_TEMP_GATE: now also R1064.1
- net LED_WIFI_N renamed LED_WIFI_GATE
- net LED_WIFI_GATE: now also R1062.1
- net PWR_GREEN_A renamed STATUS_PWR_GATE
- net STATUS_PWR_GATE: now also Q1060.1 (G), R1080.1
- net TEMP_RED_A renamed STATUS_TEMP_GATE
- net STATUS_TEMP_GATE: now also Q1064.1 (G), R1084.1
- net WIFI_BLUE_A renamed STATUS_WIFI_GATE
- net STATUS_WIFI_GATE: now also Q1062.1 (G), R1082.1
- new net AUX_12V: F1060.1
- new net STATUS_AUDIO_GATE: Q1065.1 (G), R1065.2, R1085.1
- new net STATUS_AUDIO_SINK: J1060.8 (Pin_8), Q1065.3 (D)
- new net STATUS_BACKUP_SINK: J1060.4 (Pin_4), Q1061.3 (D)
- new net STATUS_CELL_SINK: J1060.6 (Pin_6), Q1063.3 (D)
- new net STATUS_LED_12V: F1060.2, J1060.1 (Pin_1), J1060.2 (Pin_2)
- new net STATUS_PWR_SINK: J1060.3 (Pin_3), Q1060.3 (D)
- new net STATUS_TEMP_SINK: J1060.7 (Pin_7), Q1064.3 (D)
- new net STATUS_WIFI_SINK: J1060.5 (Pin_5), Q1062.3 (D)
- no-connect marks 5 -> 3
Other:
- note added: "5. SIX 12 V TOP-PANEL STATUS-LAMP DRIVERS"
- note added: "AFB0412SHB-SP04 MODEM FAN"
- note added: "AUDIO / DX06WG012B"
- note added: "BACKUP / DX06WY012B"
- note added: "CELL / DX06WW012B"
- note added: "FFB0412EN-00Y2E CPU FAN"
- note added: "J1060 feeds six external Bulgin DX06 12 V wire-lead indicators. Two supply contacts plus six protected low-side returns."
- note added: "J1070 is the keyed eight-circuit boundary to external CS7L2FR and two LS102W panel lights. Unused blue/red switch-ring leads are insulated in the harness."
- note added: "PWR / DX06WG012B"
- note added: "Pins 1-4 serve switch GND, 12 V, green ring, and latching sink. Pins 5-8 are the two lamp +/- pairs; the PCB joins both lamps to the switched sink."
- note added: "TEMP / DX06WR012B"
- note added: "WIFI / DX06WB012B"
- note removed: "5. SIX TOP-PANEL STATUS LED DRIVERS"
- note removed: "AUDIO CYAN"
- note removed: "BACKUP VIOLET"
- note removed: "CELL AMBER"
- note removed: "CPU FAN"
- note removed: "MODEM FAN"
- note removed: "NIGHT LED 1"
- note removed: "NIGHT LED 2"
- note removed: "PWR GREEN"
- note removed: "S1070 pin 5 is the rated low-side load output. Both 12 V LS102W courtesy lights switch together; pin 3 adds a dim green ON ring through R1070."
- note removed: "TCA9535 sinks LED current. Final LED MPNs and resistor values follow top-panel brightness and color review."
- note removed: "TEMP RED"
- note removed: "WIFI BLUE"
- moved on the sheet: R1085

Commit message: Audit schematic logic against controlled datasheets
Parts:
- added C1011, C1012, C1013: 100nF, Capacitor_SMD:C_0603_1608Metric, symbol Device:C
- added R1006: 200k, Resistor_SMD:R_0603_1608Metric, symbol Device:R
- added R1019, R1022: 100k, Resistor_SMD:R_0603_1608Metric, symbol Device:R
- added TP1001: U1001_INT_N, TestPoint:TestPoint_Pad_D2.0mm, symbol Connector:TestPoint
- added TP1002: U1002_INT_N, TestPoint:TestPoint_Pad_D2.0mm, symbol Connector:TestPoint
- added TP1003: U1003_INT_N, TestPoint:TestPoint_Pad_D2.0mm, symbol Connector:TestPoint
- added U1003: TCA9535PWR_0x22, Package_SO:TSSOP-24_4.4x7.8mm_P0.65mm, symbol Interface_Expansion:TCA9535PWR
Connections:
- net CTRL_I2C_SCL: now also U1003.22 (SCL)
- net CTRL_I2C_SDA: now also U1003.23 (SDA)
- net GND: now also C1011.2, C1012.2, C1013.2, R1019.2, R1022.2, U1003.12 (GND), U1003.21 (A0), U1003.3 (A2)
- net LOGIC_3V3: now also C1011.1, C1012.1, C1013.1, R1006.1, U1003.2 (A1), U1003.24 (VCC); no longer U1000.7 (VREF2), U1000.8 (EN)
- net U1001_INT_N: now also TP1001.1
- net U1002_INT_N: now also TP1002.1
- net AUD_DAC_MUTE_N renamed AUD_DAC_MUTE_CMD_N
- new net AUX_12V_PG: U1003.15 (P12)
- new net CTRL_I2C_BIAS: R1006.2, U1000.7 (VREF2), U1000.8 (EN)
- new net IO_5V0_PG: U1003.17 (P14)
- new net LOGIC_1V8_PG: U1003.14 (P11)
- new net LOGIC_3V3_PG: U1003.16 (P13)
- new net MODEM_3V8_PG: U1003.8 (P04)
- new net MODEM_3V8_PRE_PG: U1003.7 (P03)
- new net MODEM_POWER_EN: R1019.1, U1003.4 (P00)
- new net NET_3V3_PG: U1003.11 (P07)
- new net PCIE_1V0_PG: U1003.13 (P10)
- new net SYS_4V0_PG: U1003.6 (P02)
- new net U1003_INT_N: TP1003.1, U1003.1 (~{INT})
- new net VALID_DTAP_N: U1003.18 (P15)
- new net VALID_GOLD_N: U1003.19 (P16)
- new net WIFI_3V3_PG: U1003.10 (P06)
- new net WIFI_3V3_PRE_PG: U1003.9 (P05)
- new net WIFI_POWER_EN: R1022.1, U1003.5 (P01)
- no-connect marks 3 -> 4
Other:
- note added: "2. THREE 16-BIT GPIO EXPANDERS"
- note added: "Radio final rails default off; W_DISABLE/WIFI_DISABLE remain asserted until firmware verifies power and thermal state."
- note added: "TCA9535 outputs power up as inputs. External straps define safe reset, mute, radio-power, and amplifier states."
- note added: "U1003: 7-bit address 0x22; INT is test-point only and firmware polls status."
- note removed: "2. TWO 16-BIT GPIO EXPANDERS"
- note removed: "TCA9535 outputs power up as inputs. External straps below define safe reset, mute, radio, and amplifier states."
- note removed: "W_DISABLE and WIFI_DISABLE are held active during boot; software releases them only after power and thermal checks pass."

Commit message: Implement direct socketed dual-SIM daughterboard
Parts:
- removed C1052: 100nF, Capacitor_SMD:C_0603_1608Metric, symbol Device:C
- removed J1060: STATUS_LAMP_PANEL_HARNESS, Connector_Molex:Molex_Micro-Fit_3.0_43045-0812_2x04_P3.00mm_Vertical, symbol Connector_Generic:Conn_02x04_Odd_Even
- removed J1070: NIGHT_LIGHT_PANEL_HARNESS, Connector_Molex:Molex_Micro-Fit_3.0_43045-0812_2x04_P3.00mm_Vertical, symbol Connector_Generic:Conn_02x04_Odd_Even
- removed R1002, R1003: 2.2k, Resistor_SMD:R_0603_1608Metric, symbol Device:R
- removed R1010, R1011, R1012: 100k, Resistor_SMD:R_0603_1608Metric, symbol Device:R
- removed R1041, R1042, R1043: 10k, Resistor_SMD:R_0603_1608Metric, symbol Device:R
- removed U1000: PCA9306DP, Package_SO:TSSOP-8_3x3mm_P0.65mm, symbol Interface:PCA9306D
- added F1022, F1023, F1024: 1.1A hold / 33V, Fuse:Fuse_1812_4532Metric, symbol Device:Polyfuse
- added F1060: 0.25A fast, Fuse:Fuse_Littelfuse-NANO2-451_453, symbol Device:Fuse
- added R1004: 2.2k, Resistor_SMD:R_0603_1608Metric, symbol Device:R
- added R1005: 4.7k, Resistor_SMD:R_0603_1608Metric, symbol Device:R
- added R1006: 200k, Resistor_SMD:R_0603_1608Metric, symbol Device:R
- added R1018, R1019, R1022, R1080: 100k, Resistor_SMD:R_0603_1608Metric, symbol Device:R
- added R1070: 1k ring limit, Resistor_SMD:R_0603_1608Metric, symbol Device:R
- C1052: renamed from R1080; value 100k -> 100nF; footprint Resistor_SMD:R_0603_1608Metric -> Capacitor_SMD:C_0603_1608Metric; symbol Device:R -> Device:C; MPN RC0603FR-07100KL -> GRM188R71E104KA01D; Manufacturer Yageo -> Murata
- J1060: renamed from F1060; value 0.25A fast -> STATUS_LAMP_PANEL_HARNESS; footprint Fuse:Fuse_Littelfuse-NANO2-451_453 -> Connector_Molex:Molex_Micro-Fit_3.0_43045-0812_2x04_P3.00mm_Vertical; symbol Device:Fuse -> Connector_Generic:Conn_02x04_Odd_Even; MPN 0453.250MR -> 43045-0812; Manufacturer Littelfuse -> Molex
- J1070: renamed from R1070; value 1k ring limit -> NIGHT_LIGHT_PANEL_HARNESS; footprint Resistor_SMD:R_0603_1608Metric -> Connector_Molex:Molex_Micro-Fit_3.0_43045-0812_2x04_P3.00mm_Vertical; symbol Device:R -> Connector_Generic:Conn_02x04_Odd_Even; MPN RC0603FR-071KL -> 43045-0812; Manufacturer Yageo -> Molex
- R1002: renamed from R1005; value 4.7k -> 2.2k; MPN RC0603FR-074K7L -> RC0603FR-072K2L
- R1003: renamed from R1006; value 200k -> 2.2k; MPN RC0603FR-07200KL -> RC0603FR-072K2L
- R1041: renamed from F1022; value 1.1A hold / 33V -> 10k; footprint Fuse:Fuse_1812_4532Metric -> Resistor_SMD:R_0603_1608Metric; symbol Device:Polyfuse -> Device:R; MPN 1812L110/33DR -> RC0603FR-0710KL; Manufacturer Littelfuse -> Yageo
- R1042: renamed from F1023; value 1.1A hold / 33V -> 10k; footprint Fuse:Fuse_1812_4532Metric -> Resistor_SMD:R_0603_1608Metric; symbol Device:Polyfuse -> Device:R; MPN 1812L110/33DR -> RC0603FR-0710KL; Manufacturer Littelfuse -> Yageo
- R1043: renamed from F1024; value 1.1A hold / 33V -> 10k; footprint Fuse:Fuse_1812_4532Metric -> Resistor_SMD:R_0603_1608Metric; symbol Device:Polyfuse -> Device:R; MPN 1812L110/33DR -> RC0603FR-0710KL; Manufacturer Littelfuse -> Yageo
- U1000: renamed from R1001; value 2.2k -> PCA9306DP; footprint Resistor_SMD:R_0603_1608Metric -> Package_SO:TSSOP-8_3x3mm_P0.65mm; symbol Device:R -> Interface:PCA9306D; MPN RC0603FR-072K2L -> PCA9306DP,118; Manufacturer Yageo -> NXP
- renumbered R1004 to R1001, R1013 to R1010, R1014 to R1011, R1015 to R1012, R1016 to R1013, R1017 to R1014, R1018 to R1015, R1019 to R1016, R1022 to R1017
Connections:
- net AUDIO_ENABLE: now also R1010.1
- net AUD_DAC_MUTE_CMD_N: now also R1011.1
- net AUX_12V: now also F1060.1; no longer J1060.1
- net CPU_FAN_TACH: now also R1041.2
- net CS_GREEN_RING_K: now also J1070.3 (Pin_3), R1070.1; no longer J1070.1
- net CTRL_I2C_BIAS: now also U1000.7 (VREF2), U1000.8 (EN), R1006.2; no longer R1003.2
- net CTRL_I2C_SCL: now also R1003.2, U1000.6 (SCL2)
- net CTRL_I2C_SDA: now also U1000.5 (SDA2), R1004.2; no longer R1001.2
- net EXHAUST_FAN_12V: now also F1024.2; no longer R1043.2
- net FAN_AUX_12V: now also F1022.1, F1023.1, F1024.1; no longer R1041.1, R1042.1, R1043.1
- net GND: now also J1070.1 (Pin_1), R1011.2, R1013.2, R1015.2, U1000.1 (GND), R1019.2, R1022.2, R1080.2; no longer R1012.2, R1016.2, R1017.2
- net INTAKE_FAN_12V: now also F1023.2; no longer R1042.2
- net INTAKE_FAN_TACH: now also R1043.2
- net LAN1_RESET_LOCAL_N: now also R1017.1; no longer R1014.1
- net LAN2_RESET_LOCAL_N: now also R1018.1; no longer R1015.1
- net LOGIC_1V8: now also R1001.1, R1002.1, U1000.2 (VREF1); no longer U1000.1
- net LOGIC_3V3: now also C1052.1, R1012.2, R1016.2, R1017.2, R1041.1, R1042.1, R1043.1, R1004.1, R1005.1, R1006.1, R1018.2; no longer R1001.1, R1002.1, R1011.2, R1013.2, R1015.2
- net MODEM_FAN_12V: now also F1022.2; no longer R1041.2
- net MODEM_FAN_TACH: now also R1042.2
- net MODEM_FULL_CARD_POWER_OFF_N: now also R1012.1
- net MODEM_POWER_EN: now also R1019.1; no longer R1016.1
- net MODEM_RESET_N: now also R1014.1; no longer R1011.1
- net MODEM_W_DISABLE1_N: now also R1013.1; no longer R1010.1
- net NIGHT_LIGHT_12V: now also J1070.2 (Pin_2), J1070.5 (Pin_5), J1070.7 (Pin_7)
- net NIGHT_LIGHT_SINK: now also J1070.4 (Pin_4), J1070.6 (Pin_6), J1070.8 (Pin_8), R1070.2; no longer J1070.2
- net PWR_MON_ALERT_N: now also R1005.2; no longer R1002.2
- net STATUS_AUDIO_SINK: now also J1060.8 (Pin_8)
- net STATUS_BACKUP_SINK: now also J1060.4 (Pin_4)
- net STATUS_CELL_SINK: now also J1060.6 (Pin_6)
- net STATUS_LED_12V: now also J1060.1 (Pin_1), F1060.2
- net STATUS_PWR_GATE: now also R1080.1; no longer C1052.1
- net STATUS_PWR_SINK: now also J1060.3 (Pin_3)
- net STATUS_TEMP_SINK: now also J1060.7 (Pin_7)
- net STATUS_WIFI_SINK: now also J1060.5 (Pin_5)
- net SYS_I2C7_SCL: now also R1001.2, U1000.3 (SCL1); no longer U1000.2
- net SYS_I2C7_SDA: now also R1002.2, U1000.4 (SDA1)
- net WAN2_RESET_LOCAL_N: now also R1016.1; no longer R1013.1
- net WIFI_DISABLE1_N: now also R1015.1; no longer R1012.1
- net WIFI_POWER_EN: now also R1022.1; no longer R1017.1
Other:
- moved on the sheet: R1001, R1002, R1003, R1010, R1011, R1012, R1013, R1014, R1015, R1016, R1017
