File: cad/kicad/SYSTEM/Radxa-CM5-ProComm-System.kicad_sch (KiCad schematic)
At the start: 0 parts

Commit message: Replace system index with complete electrical schematic
Parts:
- added F9001: C14 INLET FUSE, symbol Device:Fuse
- added J9001: FUSED C14 AC INLET, symbol Connector_Generic:Conn_01x03
- added J9002: RPS-400-24-C AC CN1, symbol Connector_Generic:Conn_01x03
- added J9003: RPS-400-24-C DC CN2/CN3, symbol Connector_Generic:Conn_01x02
- added J9004: PWR-SELECT J101 PSU INPUT, symbol Connector_Generic:Conn_01x02
- added J9005: ANTON/BAUER QRC-GOLD, symbol Connector_Generic:Conn_01x02
- added J9006: D-TAP BACKUP INPUT, symbol Connector_Generic:Conn_01x02
- added J9101: CM5-CARRIER J101, symbol Connector_Generic:Conn_02x02_Odd_Even
- added J9102: CM5-CARRIER J102, symbol Connector_Generic:Conn_01x08
- added J9103: CM5-CARRIER J103, symbol Connector_Generic:Conn_01x06
- added J9201: CM5-CARRIER J201, symbol Connector_Generic:Conn_02x15_Odd_Even
- added J9202: CM5-CARRIER J202, symbol Connector_Generic:Conn_02x02_Odd_Even
- added J9301: PWR-SELECT J301, symbol Connector_Generic:Conn_02x02_Odd_Even
- added J9401: PWR-SELECT J401, symbol Connector_Generic:Conn_01x08
- added J9402: PWR-SELECT J402, symbol Connector_Generic:Conn_01x06
- added J9411: CPU HEATSINK FAN, symbol Connector_Generic:Conn_01x04
- added J9412: MODEM HEATSINK FAN, symbol Connector_Generic:Conn_01x04
- added J9413: THA0412AD INTAKE, symbol Connector_Generic:Conn_01x04
- added J9414: THA0412AD EXHAUST, symbol Connector_Generic:Conn_01x04
- added J9421: WAN1 RJ45, symbol Connector_Generic:Conn_01x08
- added J9422: WAN2 RJ45, symbol Connector_Generic:Conn_01x08
- added J9423: LAN1 RJ45, symbol Connector_Generic:Conn_01x08
- added J9424: LAN2 RJ45, symbol Connector_Generic:Conn_01x08
- added J9430: CTIA HEADSET JACK, symbol Connector_Generic:Conn_01x04
- added J9431: NANO-SIM 1, symbol Connector_Generic:Conn_01x06
- added J9432: NANO-SIM 2, symbol Connector_Generic:Conn_01x06
- added J9440: WIFI_1, symbol Connector_Generic:Conn_01x01
- added J9441: WIFI_2, symbol Connector_Generic:Conn_01x01
- added J9442: WIFI_3, symbol Connector_Generic:Conn_01x01
- added J9443: WIFI_4, symbol Connector_Generic:Conn_01x01
- added J9444: CELL_1, symbol Connector_Generic:Conn_01x01
- added J9445: CELL_2, symbol Connector_Generic:Conn_01x01
- added J9446: CELL_3, symbol Connector_Generic:Conn_01x01
- added J9447: CELL_4_GNSS, symbol Connector_Generic:Conn_01x01
- added J9501: AUDIO-8X8 J101, symbol Connector_Generic:Conn_02x15_Odd_Even
- added J9502: AUDIO-8X8 J102, symbol Connector_Generic:Conn_02x02_Odd_Even
- added J9601: NC3MAV CH1 OUT, symbol Connector_Generic:Conn_01x03
- added J9602: NC3MAV CH2 OUT, symbol Connector_Generic:Conn_01x03
- added J9603: NC3MAV CH3 OUT, symbol Connector_Generic:Conn_01x03
- added J9604: NC3MAV CH4 OUT, symbol Connector_Generic:Conn_01x03
- added J9605: NC3MAV CH5 OUT, symbol Connector_Generic:Conn_01x03
- added J9606: NC3MAV CH6 OUT, symbol Connector_Generic:Conn_01x03
- added J9607: NC3MAV CH7 OUT, symbol Connector_Generic:Conn_01x03
- added J9608: NC3MAV CH8 OUT, symbol Connector_Generic:Conn_01x03
- added J9701: NC3FAV CH1 IN, symbol Connector_Generic:Conn_01x03
- added J9702: NC3FAV CH2 IN, symbol Connector_Generic:Conn_01x03
- added J9703: NC3FAV CH3 IN, symbol Connector_Generic:Conn_01x03
- added J9704: NC3FAV CH4 IN, symbol Connector_Generic:Conn_01x03
- added J9705: NC3FAV CH5 IN, symbol Connector_Generic:Conn_01x03
- added J9706: NC3FAV CH6 IN, symbol Connector_Generic:Conn_01x03
- added J9707: NC3FAV CH7 IN, symbol Connector_Generic:Conn_01x03
- added J9708: NC3FAV CH8 IN, symbol Connector_Generic:Conn_01x03
- added J9801: CM5-CARRIER J801 HDMI-A, symbol Connector_Generic:Conn_01x19
- added J9802: CM5-CARRIER J802 USB-A, symbol Connector_Generic:Conn_01x04
- added J9803: CM5-CARRIER J803, symbol Connector_Generic:Conn_02x02_Odd_Even
- added J9851: 15.6-IN MONITOR HDMI IN, symbol Connector_Generic:Conn_01x19
- added J9852: MONITOR USB-B TOUCH, symbol Connector_Generic:Conn_01x04
- added J9853: MONITOR DC 12 V, symbol Connector_Generic:Conn_02x02_Odd_Even
Connections:
- new net AC_L_FUSED: F9001.2, J9002.1 (Pin_1)
- new net AC_L_IN: F9001.1, J9001.1 (Pin_1)
- new net AC_N: J9001.2 (Pin_2), J9002.2 (Pin_2)
- new net AIN_CH1_COLD: J9701.3 (Pin_3)
- new net AIN_CH1_HOT: J9701.2 (Pin_2)
- new net AIN_CH2_COLD: J9702.3 (Pin_3)
- new net AIN_CH2_HOT: J9702.2 (Pin_2)
- new net AIN_CH3_COLD: J9703.3 (Pin_3)
- new net AIN_CH3_HOT: J9703.2 (Pin_2)
- new net AIN_CH4_COLD: J9704.3 (Pin_3)
- new net AIN_CH4_HOT: J9704.2 (Pin_2)
- new net AIN_CH5_COLD: J9705.3 (Pin_3)
- new net AIN_CH5_HOT: J9705.2 (Pin_2)
- new net AIN_CH6_COLD: J9706.3 (Pin_3)
- new net AIN_CH6_HOT: J9706.2 (Pin_2)
- new net AIN_CH7_COLD: J9707.3 (Pin_3)
- new net AIN_CH7_HOT: J9707.2 (Pin_2)
- new net AIN_CH8_COLD: J9708.3 (Pin_3)
- new net AIN_CH8_HOT: J9708.2 (Pin_2)
- new net AOUT_CH1_COLD: J9601.3 (Pin_3)
- new net AOUT_CH1_HOT: J9601.2 (Pin_2)
- new net AOUT_CH2_COLD: J9602.3 (Pin_3)
- new net AOUT_CH2_HOT: J9602.2 (Pin_2)
- new net AOUT_CH3_COLD: J9603.3 (Pin_3)
- new net AOUT_CH3_HOT: J9603.2 (Pin_2)
- new net AOUT_CH4_COLD: J9604.3 (Pin_3)
- new net AOUT_CH4_HOT: J9604.2 (Pin_2)
- new net AOUT_CH5_COLD: J9605.3 (Pin_3)
- new net AOUT_CH5_HOT: J9605.2 (Pin_2)
- new net AOUT_CH6_COLD: J9606.3 (Pin_3)
- new net AOUT_CH6_HOT: J9606.2 (Pin_2)
- new net AOUT_CH7_COLD: J9607.3 (Pin_3)
- new net AOUT_CH7_HOT: J9607.2 (Pin_2)
- new net AOUT_CH8_COLD: J9608.3 (Pin_3)
- new net AOUT_CH8_HOT: J9608.2 (Pin_2)
- new net AUDIO_12V: J9202.1 (Pin_1), J9202.2 (Pin_2), J9502.1 (Pin_1), J9502.2 (Pin_2)
- new net AUDIO_ENABLE: J9201.24 (Pin_24), J9501.24 (Pin_24)
- new net AUDIO_PRESENT_N: J9201.23 (Pin_23), J9501.23 (Pin_23)
- new net AUD_ADC_RST_N: J9201.19 (Pin_19), J9501.19 (Pin_19)
- new net AUD_ADC_SDOUT_N: J9201.14 (Pin_14), J9501.14 (Pin_14)
- new net AUD_ADC_SDOUT_P: J9201.13 (Pin_13), J9501.13 (Pin_13)
- new net AUD_BCLK_N: J9201.6 (Pin_6), J9501.6 (Pin_6)
- new net AUD_BCLK_P: J9201.5 (Pin_5), J9501.5 (Pin_5)
- new net AUD_DAC_MUTE_N: J9201.21 (Pin_21), J9501.21 (Pin_21)
- new net AUD_DAC_RST_N: J9201.20 (Pin_20), J9501.20 (Pin_20)
- new net AUD_DAC_SDIN_N: J9201.12 (Pin_12), J9501.12 (Pin_12)
- new net AUD_DAC_SDIN_P: J9201.11 (Pin_11), J9501.11 (Pin_11)
- new net AUD_FSYNC_N: J9201.8 (Pin_8), J9501.8 (Pin_8)
- new net AUD_FSYNC_P: J9201.7 (Pin_7), J9501.7 (Pin_7)
- new net AUD_I2C_SCL: J9201.17 (Pin_17), J9501.17 (Pin_17)
- new net AUD_I2C_SDA: J9201.18 (Pin_18), J9501.18 (Pin_18)
- new net AUD_IRQ_N: J9201.22 (Pin_22), J9501.22 (Pin_22)
- new net AUD_MCLK_N: J9201.2 (Pin_2), J9501.2 (Pin_2)
- new net AUD_MCLK_P: J9201.1 (Pin_1), J9501.1 (Pin_1)
- new net BAT_LOW_N: J9102.6 (Pin_6), J9401.6 (Pin_6)
- new net CELL_1_RF: J9444.1 (Pin_1)
- new net CELL_2_RF: J9445.1 (Pin_1)
- new net CELL_3_RF: J9446.1 (Pin_1)
- new net CELL_4_GNSS_RF: J9447.1 (Pin_1)
- new net CHASSIS_PE: J9001.3 (Pin_3), J9002.3 (Pin_3)
- new net CH_24V_N: J9102.2 (Pin_2), J9401.2 (Pin_2)
- new net CH_BAT_N: J9102.3 (Pin_3), J9401.3 (Pin_3)
- new net CPU_FAN_12V: J9411.2 (Pin_2)
- new net CPU_FAN_PWM: J9411.4 (Pin_4)
- new net CPU_FAN_TACH: J9411.3 (Pin_3)
- new net CTRL_I2C_SCL: J9103.4 (Pin_4), J9402.4 (Pin_4)
- new net CTRL_I2C_SDA: J9103.3 (Pin_3), J9402.3 (Pin_3)
- new net DISPLAY_12V: J9803.1 (Pin_1), J9803.2 (Pin_2), J9853.1 (Pin_1), J9853.2 (Pin_2)
- new net DTAP_IN: J9006.1 (Pin_1)
- new net EXHAUST_FAN_12V: J9414.2 (Pin_2)
- new net EXHAUST_FAN_PWM: J9414.4 (Pin_4)
- new net EXHAUST_FAN_TACH: J9414.3 (Pin_3)
- new net GND: J9003.2 (Pin_2), J9004.2 (Pin_2), J9005.2 (Pin_2), J9006.2 (Pin_2), J9101.3 (Pin_3), J9101.4 (Pin_4), J9102.1 (Pin_1), J9103.2 (Pin_2), J9103.6 (Pin_6), J9201.10 (Pin_10), J9201.15 (Pin_15), J9201.16 (Pin_16), J9201.26 (Pin_26), J9201.29 (Pin_29), J9201.3 (Pin_3), J9201.30 (Pin_30), J9201.4 (Pin_4), J9201.9 (Pin_9), J9202.3 (Pin_3), J9202.4 (Pin_4), J9301.3 (Pin_3), J9301.4 (Pin_4), J9401.1 (Pin_1), J9402.2 (Pin_2), J9402.6 (Pin_6), J9411.1 (Pin_1), J9412.1 (Pin_1), J9413.1 (Pin_1), J9414.1 (Pin_1), J9431.5 (Pin_5), J9432.5 (Pin_5), J9501.10 (Pin_10), J9501.15 (Pin_15), J9501.16 (Pin_16), J9501.26 (Pin_26), J9501.29 (Pin_29), J9501.3 (Pin_3), J9501.30 (Pin_30), J9501.4 (Pin_4), J9501.9 (Pin_9), J9502.3 (Pin_3), J9502.4 (Pin_4), J9801.11 (Pin_11), J9801.17 (Pin_17), J9801.2 (Pin_2), J9801.5 (Pin_5), J9801.8 (Pin_8), J9802.4 (Pin_4), J9803.3 (Pin_3), J9803.4 (Pin_4), J9851.11 (Pin_11), J9851.17 (Pin_17), J9851.2 (Pin_2), J9851.5 (Pin_5), J9851.8 (Pin_8), J9852.4 (Pin_4), J9853.3 (Pin_3), J9853.4 (Pin_4)
- new net GOLD_IN: J9005.1 (Pin_1)
- new net HDMI_5V_OUT: J9801.18 (Pin_18), J9851.18 (Pin_18)
- new net HDMI_CEC: J9801.13 (Pin_13), J9851.13 (Pin_13)
- new net HDMI_CLK_N: J9801.12 (Pin_12), J9851.12 (Pin_12)
- new net HDMI_CLK_P: J9801.10 (Pin_10), J9851.10 (Pin_10)
- new net HDMI_D0_N: J9801.9 (Pin_9), J9851.9 (Pin_9)
- new net HDMI_D0_P: J9801.7 (Pin_7), J9851.7 (Pin_7)
- new net HDMI_D1_N: J9801.6 (Pin_6), J9851.6 (Pin_6)
- new net HDMI_D1_P: J9801.4 (Pin_4), J9851.4 (Pin_4)
- new net HDMI_D2_N: J9801.3 (Pin_3), J9851.3 (Pin_3)
- new net HDMI_D2_P: J9801.1 (Pin_1), J9851.1 (Pin_1)
- new net HDMI_DDC_SCL: J9801.15 (Pin_15), J9851.15 (Pin_15)
- new net HDMI_DDC_SDA: J9801.16 (Pin_16), J9851.16 (Pin_16)
- new net HDMI_HEAC_P: J9801.14 (Pin_14), J9851.14 (Pin_14)
- new net HDMI_HPD: J9801.19 (Pin_19), J9851.19 (Pin_19)
- new net HEADSET_GND: J9430.3 (Pin_3)
- new net HEADSET_L: J9430.1 (Pin_1)
- new net HEADSET_MIC: J9430.4 (Pin_4)
- new net HEADSET_R: J9430.2 (Pin_2)
- new net INTAKE_FAN_12V: J9413.2 (Pin_2)
- new net INTAKE_FAN_PWM: J9413.4 (Pin_4)
- new net INTAKE_FAN_TACH: J9413.3 (Pin_3)
- new net LAN1_RJ45_1: J9423.1 (Pin_1)
- new net LAN1_RJ45_2: J9423.2 (Pin_2)
- new net LAN1_RJ45_3: J9423.3 (Pin_3)
- new net LAN1_RJ45_4: J9423.4 (Pin_4)
- new net LAN1_RJ45_5: J9423.5 (Pin_5)
- new net LAN1_RJ45_6: J9423.6 (Pin_6)
- new net LAN1_RJ45_7: J9423.7 (Pin_7)
- new net LAN1_RJ45_8: J9423.8 (Pin_8)
- new net LAN2_RJ45_1: J9424.1 (Pin_1)
- new net LAN2_RJ45_2: J9424.2 (Pin_2)
- new net LAN2_RJ45_3: J9424.3 (Pin_3)
- new net LAN2_RJ45_4: J9424.4 (Pin_4)
- new net LAN2_RJ45_5: J9424.5 (Pin_5)
- new net LAN2_RJ45_6: J9424.6 (Pin_6)
- new net LAN2_RJ45_7: J9424.7 (Pin_7)
- new net LAN2_RJ45_8: J9424.8 (Pin_8)
- new net LOGIC_3V3: J9201.25 (Pin_25), J9501.25 (Pin_25)
- new net MODEM_FAN_12V: J9412.2 (Pin_2)
- new net MODEM_FAN_PWM: J9412.4 (Pin_4)
- new net MODEM_FAN_TACH: J9412.3 (Pin_3)
- new net PWR_MON_ALERT_N: J9103.5 (Pin_5), J9402.5 (Pin_5)
- new net PWR_TELEM_3V3: J9103.1 (Pin_1), J9402.1 (Pin_1)
- new net RAW_OUT_LOAD: J9101.1 (Pin_1), J9101.2 (Pin_2), J9301.1 (Pin_1), J9301.2 (Pin_2)
- new net SIM1_CLK: J9431.3 (Pin_3)
- new net SIM1_DET: J9431.6 (Pin_6)
- new net SIM1_IO: J9431.4 (Pin_4)
- new net SIM1_RST: J9431.2 (Pin_2)
- new net SIM1_VCC: J9431.1 (Pin_1)
- new net SIM2_CLK: J9432.3 (Pin_3)
- new net SIM2_DET: J9432.6 (Pin_6)
- new net SIM2_IO: J9432.4 (Pin_4)
- new net SIM2_RST: J9432.2 (Pin_2)
- new net SIM2_VCC: J9432.1 (Pin_1)
- new net TDM_SPARE_1: J9201.27 (Pin_27), J9501.27 (Pin_27)
- new net TDM_SPARE_2: J9201.28 (Pin_28), J9501.28 (Pin_28)
- new net TOUCH_USB_5V: J9802.1 (Pin_1), J9852.1 (Pin_1)
- new net TOUCH_USB_DM: J9802.2 (Pin_2), J9852.2 (Pin_2)
- new net TOUCH_USB_DP: J9802.3 (Pin_3), J9852.3 (Pin_3)
- new net V24_IN: J9003.1 (Pin_1), J9004.1 (Pin_1)
- new net VALID_24V_N: J9102.4 (Pin_4), J9401.4 (Pin_4)
- new net VALID_BAT_N: J9102.5 (Pin_5), J9401.5 (Pin_5)
- new net VALID_DTAP_N: J9102.7 (Pin_7), J9401.7 (Pin_7)
- new net VALID_GOLD_N: J9102.8 (Pin_8), J9401.8 (Pin_8)
- new net WAN1_RJ45_1: J9421.1 (Pin_1)
- new net WAN1_RJ45_2: J9421.2 (Pin_2)
- new net WAN1_RJ45_3: J9421.3 (Pin_3)
- new net WAN1_RJ45_4: J9421.4 (Pin_4)
- new net WAN1_RJ45_5: J9421.5 (Pin_5)
- new net WAN1_RJ45_6: J9421.6 (Pin_6)
- new net WAN1_RJ45_7: J9421.7 (Pin_7)
- new net WAN1_RJ45_8: J9421.8 (Pin_8)
- new net WAN2_RJ45_1: J9422.1 (Pin_1)
- new net WAN2_RJ45_2: J9422.2 (Pin_2)
- new net WAN2_RJ45_3: J9422.3 (Pin_3)
- new net WAN2_RJ45_4: J9422.4 (Pin_4)
- new net WAN2_RJ45_5: J9422.5 (Pin_5)
- new net WAN2_RJ45_6: J9422.6 (Pin_6)
- new net WAN2_RJ45_7: J9422.7 (Pin_7)
- new net WAN2_RJ45_8: J9422.8 (Pin_8)
- new net WIFI_1_RF: J9440.1 (Pin_1)
- new net WIFI_2_RF: J9441.1 (Pin_1)
- new net WIFI_3_RF: J9442.1 (Pin_1)
- new net WIFI_4_RF: J9443.1 (Pin_1)
- new net XLR_CHASSIS: J9601.1 (Pin_1), J9602.1 (Pin_1), J9603.1 (Pin_1), J9604.1 (Pin_1), J9605.1 (Pin_1), J9606.1 (Pin_1), J9607.1 (Pin_1), J9608.1 (Pin_1), J9701.1 (Pin_1), J9702.1 (Pin_1), J9703.1 (Pin_1), J9704.1 (Pin_1), J9705.1 (Pin_1), J9706.1 (Pin_1), J9707.1 (Pin_1), J9708.1 (Pin_1)
Other:
- note added: "1. AC, PSU, AND BACKUP SOURCES"
- note added: "2. PWR-SELECT TO CM5-CARRIER"
- note added: "3. CM5-CARRIER TO AUDIO-8X8"
- note added: "4. LID DISPLAY ELECTRICAL HARNESS"
- note added: "5. COOLING, NETWORK, SERVICE, AND RF"
- note added: "6. BALANCED AUDIO PANEL - 8 OUTPUTS / 8 INPUTS"
- note added: "DETAILED ELECTRICAL CIRCUIT PAGES - DOUBLE-CLICK A SHEET TO OPEN"
- note added: "H01 - FOUR-CONDUCTOR RAW POWER HARNESS"
- note added: "H02A - SOURCE STATUS HARNESS"
- note added: "H02B - VOLTAGE / CURRENT TELEMETRY I2C"
- note added: "H03A - HDMI VIDEO"
- note added: "H03B - USB 2 TOUCH DATA"
- note added: "H03C - 12 V / 2.5 A MONITOR POWER"
- note added: "H04 - 30-PIN BUFFERED DIFFERENTIAL TDM / CONTROL"
- note added: "H05 - DEDICATED AUDIO 12 V POWER"
- note added: "PWR_TELEM_3V3 is MON_3V3 on PWR-SELECT and LOGIC_3V3 on CM5-CARRIER."
- note added: "Page 1 shows real electrical pin/net interconnects. Pages 2-17 contain the complete component-level circuits for PWR-SELECT, CM5-CARRIER, and AUDIO-8X8."
- note added: "RADXA CM5 PROCOMM - COMPLETE ELECTRICAL SCHEMATIC"
- note added: "RPS-400-24-C is primary. PWR-SELECT performs break-before-make source priority and no-blink hold-up."
- note removed: "BALANCED AUDIO 8X8"
- note removed: "CM5 CARRIER"
- note removed: "COMPLETE SYSTEM SCHEMATIC - 16 REVIEWED DESIGN SHEETS"
- note removed: "Open this project to navigate the entire design from one KiCad file. The source selector, carrier, and audio board remain separate physical PCBs with separate ERC, BOM, netlist, and layout release gates."
- note removed: "POWER SOURCE AND NO-BLINK SELECTOR"
- title: Radxa CM5 ProComm - Complete System Schematic -> Radxa CM5 ProComm - Complete Electrical Schematic

Commit message: Audit schematic logic against controlled datasheets
Connections:
- net AUD_DAC_MUTE_N renamed AUD_DAC_MUTE_CMD_N
Other:
- removed sheet AK4458VN DAC
- removed sheet AK5558VN ADC
- removed sheet AUDIO-8X8 Interface
- removed sheet Audio Power
- removed sheet Balanced Inputs 1-8
- removed sheet Balanced Outputs 1-8
- removed sheet CM5 Interface Contract
- removed sheet CM5 Pin Allocation
- removed sheet Display Harness
- removed sheet Headset / Audio Control
- removed sheet Network / PCIe / Wi-Fi
- removed sheet Power Regulators
- removed sheet TDM / Clock / Control
- removed sheet Thermal / Fans / IO
- removed sheet WWAN / Dual SIM
- added sheet AUDIO-8X8 Connected Root (../AUDIO-8X8/Audio-8x8.kicad_sch)
- added sheet CM5-CARRIER Connected Root (../CM5-CARRIER/CM5-Carrier.kicad_sch)
- note added: "PHYSICAL BOARD ROOTS - EACH ROOT CONTAINS ITS CONNECTED DETAILED PAGES"
- note added: "Page 1 shows system harness interconnects. The three physical board roots contain the complete connected component-level circuits."
- note removed: "DETAILED ELECTRICAL CIRCUIT PAGES - DOUBLE-CLICK A SHEET TO OPEN"
- note removed: "Page 1 shows real electrical pin/net interconnects. Pages 2-17 contain the complete component-level circuits for PWR-SELECT, CM5-CARRIER, and AUDIO-8X8."

Commit message: Implement direct socketed dual-SIM daughterboard
Connections:
- net SIM2_DET is gone; now on net CHASSIS_GND: J9432.6 (Pin_6)
- net SIM1_DET renamed CHASSIS_GND
- net SIM1_IO renamed SIM1_DATA
- net SIM1_RST renamed SIM1_RESET
- net SIM2_IO renamed SIM2_DATA
- net SIM2_RST renamed SIM2_RESET
Other:
- added sheet SIM-SERVICE Connected Root (../SIM-SERVICE/Sim-Service.kicad_sch)
- note added: "Page 1 shows system harness interconnects. The four physical board roots contain the complete connected component-level circuits."
- note removed: "Page 1 shows system harness interconnects. The three physical board roots contain the complete connected component-level circuits."
Changed lines of the file:
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@@
 		(company "ProComm")
 		(comment 1 "Top sheet is the electrical system interconnect; nested roots expose all detailed circuits")
-		(comment 2 "PWR-SELECT, CM5-CARRIER, and AUDIO-8X8 are authoritative physical PCB netlists")
+		(comment 2 "PWR-SELECT, CM5-CARRIER, AUDIO-8X8, and SIM-SERVICE are authoritative physical PCB netlists")
 		(comment 3 "System connector representations are excluded from BOM and board update")
 		(comment 4 "ENGINEERING PCB LAYOUT AUTHORIZED; FABRICATION RELEASE HELD")
@@
 		)
 	)
-	(label "SIM1_RST"
+	(label "SIM1_RESET"
 		(at 579.12 547.37 0.0000)
 		(effects
@@
 		)
 	)
-	(label "SIM1_IO"
+	(label "SIM1_DATA"
 		(at 579.12 552.45 0.0000)
 		(effects
@@
 		)
 	)
-	(label "SIM1_DET"
+	(label "CHASSIS_GND"
 		(at 579.12 557.53 0.0000)
 		(effects
@@
 		)
 	)
-	(label "SIM2_RST"
+	(label "SIM2_RESET"
 		(at 698.5 547.37 0.0000)
 		(effects
@@
 		)
 	)
-	(label "SIM2_IO"
+	(label "SIM2_DATA"
 		(at 698.5 552.45 0.0000)
 		(effects
@@
 		)
 	)
-	(label "SIM2_DET"
+	(label "CHASSIS_GND"
 		(at 698.5 557.53 0.0000)
 		(effects
@@
 		)
 	)
-	(text "Page 1 shows system harness interconnects. The three physical board roots contain the complete connected component-level circuits."
+	(text "Page 1 shows system harness interconnects. The four physical board roots contain the complete connected component-level circuits."
 		(exclude_from_sim no)
 		(at 400 38 0.0000)
@@
 				)
 			)
+		)
+	)
+	(sheet
+		(at 895 700)
+		(size 245 20)
+		(exclude_from_sim yes)
+		(in_bom no)
+		(on_board no)
+		(dnp no)
+		(fields_autoplaced yes)
+		(stroke
+			(width 0.3)
+			(type solid)
+		)
+		(fill
+			(color 0 0 0 0.0000)
+		)
+		(property "Sheetname" "SIM-SERVICE Connected Root"
+			(at 895 699.2884 0)
+			(effects
+				(font
+					(size 1.27 1.27)
+				)
+				(justify left bottom)
+			)
+		)
+		(property "Sheetfile" "../SIM-SERVICE/Sim-Service.kicad_sch"
+			(at 895 720.5846 0)
+			(effects
+				(font
+					(size 1.27 1.27)
+				)
+				(justify left top)
+			)
+		)
+		(instances
+			(project "Radxa-CM5-ProComm-System"
+				(path "/8ee1d215-def5-50f5-8d2f-a9585b61ca2c"
+					(page "18")
+				)
+			)
